Commit message: appended the meldog_ros2_control urdf file

File: src/meldog_description/description/ros2_control/meldog_ros2_control.urdf.xacro (robot description, xacro)
@@ -1,3 +1,28 @@
 <?xml version="1.0"?>
 <robot xmlns:xacro="http://www.ros.org/wiki/xacro">
+    <ros2_control name="GazeboSimSystem" type="system">
+        <hardware>
+          <plugin>gz_ros2_control/GazeboSimSystem</plugin>
+        </hardware>
+        <joint name="slider_to_cart">
+          <command_interface name="effort">
+            <param name="min">-1000</param>
+            <param name="max">1000</param>
+          </command_interface>
+          <state_interface name="position">
+            <param name="initial_value">1.0</param>
+          </state_interface>
+          <state_interface name="velocity"/>
+          <state_interface name="effort"/>
+        </joint>
+      </ros2_control>
+    <gazebo>
+        <plugin filename="libgz_ros2_control-system.so" name="gz_ros2_control::GazeboSimROS2ControlPlugin">
+            <robot_param>robot_description</robot_param>
+            <robot_param_node>robot_state_publisher</robot_param_node>
+            <parameters>$(find meldog_description)/controllers/meldog_controllers.yaml</parameters>
+            <hold_joints>true</hold_joints>
+            <controller_manager_name>controller_manager</controller_manager_name>
+        </plugin>
+    </gazebo>
 </robot>
