Commit message: added joints and transmissions in ros2 control

File: src/meldog_description/description/ros2_control/meldog_gazebo_ros2_control.urdf.xacro (robot description, xacro)
@@ -7,6 +7,31 @@
           <plugin>gz_ros2_control/GazeboSimSystem</plugin>
         </hardware>
-        <xacro:ros2_control_joint_macro name="lf_hip_upper_limb_joint" pos_min="${hip_upper_limb_lower_limit}" pos_max="${hip_upper_limb_upper_limit}" />
-      </ros2_control>
+        <!-- joints -->
+        <xacro:ros2_control_joint_macro name="LFT" pos_min="${hip_upper_limb_lower_limit}" pos_max="${hip_upper_limb_upper_limit}" />
+        <xacro:ros2_control_joint_macro name="LFH" pos_min="${hip_upper_limb_lower_limit}" pos_max="${hip_upper_limb_upper_limit}" />
+        <xacro:ros2_control_joint_macro name="LFK" pos_min="${hip_upper_limb_lower_limit}" pos_max="${hip_upper_limb_upper_limit}" />
+        <xacro:ros2_control_joint_macro name="RFT" pos_min="${hip_upper_limb_lower_limit}" pos_max="${hip_upper_limb_upper_limit}" />
+        <xacro:ros2_control_joint_macro name="RFH" pos_min="${hip_upper_limb_lower_limit}" pos_max="${hip_upper_limb_upper_limit}" />
+        <xacro:ros2_control_joint_macro name="RFK" pos_min="${hip_upper_limb_lower_limit}" pos_max="${hip_upper_limb_upper_limit}" />
+        <xacro:ros2_control_joint_macro name="LRT" pos_min="${hip_upper_limb_lower_limit}" pos_max="${hip_upper_limb_upper_limit}" />
+        <xacro:ros2_control_joint_macro name="LRH" pos_min="${hip_upper_limb_lower_limit}" pos_max="${hip_upper_limb_upper_limit}" />
+        <xacro:ros2_control_joint_macro name="LRK" pos_min="${hip_upper_limb_lower_limit}" pos_max="${hip_upper_limb_upper_limit}" />
+        <xacro:ros2_control_joint_macro name="RRT" pos_min="${hip_upper_limb_lower_limit}" pos_max="${hip_upper_limb_upper_limit}" />
+        <xacro:ros2_control_joint_macro name="RRH" pos_min="${hip_upper_limb_lower_limit}" pos_max="${hip_upper_limb_upper_limit}" />
+        <xacro:ros2_control_joint_macro name="RRK" pos_min="${hip_upper_limb_lower_limit}" pos_max="${hip_upper_limb_upper_limit}" />
+        <!-- transmission -->
+        <xacro:simple_transmission joint="LFT" reduction="1" offset="0.0" />
+        <xacro:simple_transmission joint="LFH" reduction="1" offset="0.0" />
+        <xacro:simple_transmission joint="LFK" reduction="1" offset="0.0" />
+        <xacro:simple_transmission joint="RFT" reduction="1" offset="0.0" />
+        <xacro:simple_transmission joint="RFH" reduction="1" offset="0.0" />
+        <xacro:simple_transmission joint="RFK" reduction="1" offset="0.0" />
+        <xacro:simple_transmission joint="LRT" reduction="1" offset="0.0" />
+        <xacro:simple_transmission joint="LRH" reduction="1" offset="0.0" />
+        <xacro:simple_transmission joint="LRK" reduction="1" offset="0.0" />
+        <xacro:simple_transmission joint="RRT" reduction="1" offset="0.0" />
+        <xacro:simple_transmission joint="RRH" reduction="1" offset="0.0" />
+        <xacro:simple_transmission joint="RRK" reduction="1" offset="0.0" />
+    </ros2_control>
     <gazebo>
         <plugin filename="libgz_ros2_control-system.so" name="gz_ros2_control::GazeboSimROS2ControlPlugin">

File: src/meldog_description/description/ros2_control/ros2_control_macros.urdf.xacro (robot description, xacro)
@@ -20,3 +20,12 @@
           </joint>
     </xacro:macro>
+    <xacro:macro name="simple_transmission" params="joint reduction offset">
+      <transmission name="${name}_transmission">
+        <plugin>transmission_interface/SimpleTransmission</plugin>
+        <joint name="${name}_joint" role="joint1">
+            <mechanical_reduction>${reduction}</mechanical_reduction>
+            <offset>${offset}</offset>
+        </joint>
+      </transmission>
+    </xacro:macro>
 </robot>

Commit message: switched joint command interface to effort, added hardware properties, modified ros2_control joints and transmissions

File: src/meldog_description/description/ros2_control/meldog_gazebo_ros2_control.urdf.xacro (robot description, xacro)
@@ -2,4 +2,5 @@
 <robot xmlns:xacro="http://www.ros.org/wiki/xacro">
     <xacro:include filename="ros2_control_macros.urdf.xacro" />
+    <xacro:include filename="hardware_properties.urdf.xacro" />
     <xacro:include filename="../joints/properties/H_joint_properties.urdf.xacro" />
     <xacro:include filename="../joints/properties/K_joint_properties.urdf.xacro" />
@@ -10,29 +11,29 @@
         </hardware>
         <!-- joints -->
-        <xacro:ros2_control_joint_macro name="LFT" pos_min="${T_lower_limit}" pos_max="${T_upper_limit}" />
-        <xacro:ros2_control_joint_macro name="LFH" pos_min="${H_lower_limit}" pos_max="${H_upper_limit}" />
-        <xacro:ros2_control_joint_macro name="LFK" pos_min="${K_lower_limit}" pos_max="${K_upper_limit}" />
-        <xacro:ros2_control_joint_macro name="RFT" pos_min="${T_lower_limit}" pos_max="${T_upper_limit}" />
-        <xacro:ros2_control_joint_macro name="RFH" pos_min="${H_lower_limit}" pos_max="${H_upper_limit}" />
-        <xacro:ros2_control_joint_macro name="RFK" pos_min="${K_lower_limit}" pos_max="${K_upper_limit}" />
-        <xacro:ros2_control_joint_macro name="LRT" pos_min="${T_lower_limit}" pos_max="${T_upper_limit}" />
-        <xacro:ros2_control_joint_macro name="LRH" pos_min="${H_lower_limit}" pos_max="${H_upper_limit}" />
-        <xacro:ros2_control_joint_macro name="LRK" pos_min="${K_lower_limit}" pos_max="${K_upper_limit}" />
-        <xacro:ros2_control_joint_macro name="RRT" pos_min="${T_lower_limit}" pos_max="${T_upper_limit}" />
-        <xacro:ros2_control_joint_macro name="RRH" pos_min="${H_lower_limit}" pos_max="${H_upper_limit}" />
-        <xacro:ros2_control_joint_macro name="RRK" pos_min="${K_lower_limit}" pos_max="${K_upper_limit}" />
+        <xacro:ros2_control_joint_macro name="LFT" pos_min="${T_lower_limit}" pos_max="${T_upper_limit}" vel_max="${motor_max_vel}" eff_max="${motor_max_eff}"/>
+        <xacro:ros2_control_joint_macro name="LFH" pos_min="${H_lower_limit}" pos_max="${H_upper_limit}" vel_max="${motor_max_vel}" eff_max="${motor_max_eff}"/>
+        <xacro:ros2_control_joint_macro name="LFK" pos_min="${K_lower_limit}" pos_max="${K_upper_limit}" vel_max="${motor_max_vel}" eff_max="${motor_max_eff}"/>
+        <xacro:ros2_control_joint_macro name="RFT" pos_min="${T_lower_limit}" pos_max="${T_upper_limit}" vel_max="${motor_max_vel}" eff_max="${motor_max_eff}"/>
+        <xacro:ros2_control_joint_macro name="RFH" pos_min="${H_lower_limit}" pos_max="${H_upper_limit}" vel_max="${motor_max_vel}" eff_max="${motor_max_eff}"/>
+        <xacro:ros2_control_joint_macro name="RFK" pos_min="${K_lower_limit}" pos_max="${K_upper_limit}" vel_max="${motor_max_vel}" eff_max="${motor_max_eff}"/>
+        <xacro:ros2_control_joint_macro name="LRT" pos_min="${T_lower_limit}" pos_max="${T_upper_limit}" vel_max="${motor_max_vel}" eff_max="${motor_max_eff}"/>
+        <xacro:ros2_control_joint_macro name="LRH" pos_min="${H_lower_limit}" pos_max="${H_upper_limit}" vel_max="${motor_max_vel}" eff_max="${motor_max_eff}"/>
+        <xacro:ros2_control_joint_macro name="LRK" pos_min="${K_lower_limit}" pos_max="${K_upper_limit}" vel_max="${motor_max_vel}" eff_max="${motor_max_eff}"/>
+        <xacro:ros2_control_joint_macro name="RRT" pos_min="${T_lower_limit}" pos_max="${T_upper_limit}" vel_max="${motor_max_vel}" eff_max="${motor_max_eff}"/>
+        <xacro:ros2_control_joint_macro name="RRH" pos_min="${H_lower_limit}" pos_max="${H_upper_limit}" vel_max="${motor_max_vel}" eff_max="${motor_max_eff}"/>
+        <xacro:ros2_control_joint_macro name="RRK" pos_min="${K_lower_limit}" pos_max="${K_upper_limit}" vel_max="${motor_max_vel}" eff_max="${motor_max_eff}"/>
         <!-- transmission -->
-        <xacro:simple_transmission joint="LFT" reduction="10" offset="0.0" />
-        <xacro:simple_transmission joint="LFH" reduction="10" offset="0.0" />
-        <xacro:simple_transmission joint="LFK" reduction="1" offset="0.0" />
-        <xacro:simple_transmission joint="RFT" reduction="10" offset="0.0" />
-        <xacro:simple_transmission joint="RFH" reduction="10" offset="0.0" />
-        <xacro:simple_transmission joint="RFK" reduction="10" offset="0.0" />
-        <xacro:simple_transmission joint="LRT" reduction="10" offset="0.0" />
-        <xacro:simple_transmission joint="LRH" reduction="10" offset="0.0" />
-        <xacro:simple_transmission joint="LRK" reduction="10" offset="0.0" />
-        <xacro:simple_transmission joint="RRT" reduction="10" offset="0.0" />
-        <xacro:simple_transmission joint="RRH" reduction="10" offset="0.0" />
-        <xacro:simple_transmission joint="RRK" reduction="10" offset="0.0" />
+        <xacro:simple_transmission joint="LFT" reduction="${actuator_reduction}" offset="0.0" />
+        <xacro:simple_transmission joint="LFH" reduction="${actuator_reduction}" offset="0.0" />
+        <xacro:simple_transmission joint="LFK" reduction="${actuator_reduction}" offset="0.0" />
+        <xacro:simple_transmission joint="RFT" reduction="${actuator_reduction}" offset="0.0" />
+        <xacro:simple_transmission joint="RFH" reduction="${actuator_reduction}" offset="0.0" />
+        <xacro:simple_transmission joint="RFK" reduction="${actuator_reduction}" offset="0.0" />
+        <xacro:simple_transmission joint="LRT" reduction="${actuator_reduction}" offset="0.0" />
+        <xacro:simple_transmission joint="LRH" reduction="${actuator_reduction}" offset="0.0" />
+        <xacro:simple_transmission joint="LRK" reduction="${actuator_reduction}" offset="0.0" />
+        <xacro:simple_transmission joint="RRT" reduction="${actuator_reduction}" offset="0.0" />
+        <xacro:simple_transmission joint="RRH" reduction="${actuator_reduction}" offset="0.0" />
+        <xacro:simple_transmission joint="RRK" reduction="${actuator_reduction}" offset="0.0" />
     </ros2_control>
     <gazebo>

File: src/meldog_description/description/ros2_control/ros2_control_macros.urdf.xacro (robot description, xacro)
@@ -1,18 +1,19 @@
 <?xml version="1.0"?>
 <robot xmlns:xacro="http://www.ros.org/wiki/xacro">
-    <xacro:macro name="ros2_control_joint_macro" params="name pos_min pos_max">
+    <xacro:macro name="ros2_control_joint_macro" params="name pos_min pos_max vel_max eff_max">
         <joint name="${name}_joint">
+          <!-- co jesli joint continuous? -->
             <command_interface name="position">
               <param name="min">${pos_min}</param>
               <param name="max">${pos_max}</param>
             </command_interface>
-            <!-- <command_interface name="velocity" >
-              <param name="min">-1000</param>
-              <param name="max">1000</param>
-            </command_interface> -->
-            <!-- <command_interface name="effort">
-              <param name="min">-1000</param>
-              <param name="max">1000</param>
-            </command_interface> -->
+            <command_interface name="velocity" >
+              <param name="min">${-vel_max/60.0*2*pi}</param>
+              <param name="max">${vel_max/60.0*2*pi}</param>
+            </command_interface>
+            <command_interface name="effort">
+              <param name="min">${-eff_max/actuator_reduction}</param>
+              <param name="max">${eff_max/actuator_reduction}</param>
+            </command_interface>
             <state_interface name="position" />
             <state_interface name="velocity"/>
