Commit message: moved link properties from base_prroperties to separate files for each link type

File: src/meldog_description/description/links/lower_limb/LL_properties.urdf.xacro (robot description, xacro)
@@ -4,4 +4,6 @@
     <xacro:property name="lower_limb_vis_stl_name" value="lower_limb_test.stl" />
     <xacro:property name="lower_limb_coll_stl_name" value="lower_limb_collision.stl" />
+    <!-- Limb dimensions -->
+    <xacro:property name="lower_limb_length_to_foot" value="0.25" />
     <!-- inertial properties -->
         <!-- mass -->

File: src/meldog_description/description/links/upper_limb/UL_properties.urdf.xacro (robot description, xacro)
@@ -4,4 +4,6 @@
     <xacro:property name="upper_limb_vis_stl_name" value="upper_limb_test.stl" />
     <xacro:property name="upper_limb_coll_stl_name" value="upper_limb_collision.stl" />
+    <!-- limb dimensions -->
+    <xacro:property name="upper_limb_length" value="0.25" />
     <!-- inertial properties -->
         <!-- mass -->
