Commit message: removed temmporary joints ffolder

File: src/meldog_description/description/base_properties.urdf.xacro (robot description, xacro)
@@ -80,3 +80,5 @@
         <xacro:property name="upper_limb_lower_limb_velocity" value="100.0" />
         <xacro:property name="trunk_hip_velocity" value="100.0" />
+        <xacro:property name="test_damping" value="0"/>
+        <xacro:property name="test_friction" value="0"/>
 </robot>

File: src/meldog_description/description/meldog_core.urdf.xacro (robot description, xacro)
@@ -53,4 +53,5 @@
                velocity="${hip_upper_limb_velocity}" />
         <axis xyz="0 1 0" />
+        <dynamics damping="${test_damping}" friction="${test_friction}" />
     </joint>
     <joint name="lf_upper_limb_lower_limb_joint" type="revolute">
@@ -63,4 +64,5 @@
                velocity="${upper_limb_lower_limb_velocity}" />
         <axis xyz="0 1 0" />
+        <dynamics damping="${test_damping}" friction="${test_friction}" />
     </joint>
     <joint name="lf_lower_limb_foot_joint" type="fixed">
@@ -78,4 +80,5 @@
                velocity="${trunk_hip_velocity}" />
         <axis xyz="1 0 0" />
+        <dynamics damping="${test_damping}" friction="${test_friction}" />
     </joint>
     <!-- Right front leg joints -->
@@ -89,4 +92,5 @@
                velocity="${trunk_hip_velocity}" />
         <axis xyz="-1 0 0" />
+        <dynamics damping="${test_damping}" friction="${test_friction}" />
     </joint>
     <joint name="rf_hip_upper_limb_joint" type="revolute">
@@ -102,4 +106,5 @@
                velocity="${hip_upper_limb_velocity}" />
         <axis xyz="0 1 0" />
+        <dynamics damping="${test_damping}" friction="${test_friction}" />
     </joint>
     <joint name="rf_upper_limb_lower_limb_joint" type="revolute">
@@ -112,4 +117,5 @@
                velocity="${upper_limb_lower_limb_velocity}" />
         <axis xyz="0 1 0" />
+        <dynamics damping="${test_damping}" friction="${test_friction}" />
     </joint>
     <joint name="rf_lower_limb_foot_joint" type="fixed">
@@ -131,4 +137,5 @@
                velocity="${hip_upper_limb_velocity}" />
         <axis xyz="0 1 0" />
+        <dynamics damping="${test_damping}" friction="${test_friction}" />
     </joint>
     <joint name="lr_upper_limb_lower_limb_joint" type="revolute">
@@ -141,4 +148,5 @@
                velocity="${upper_limb_lower_limb_velocity}" />
         <axis xyz="0 1 0" />
+        <dynamics damping="${test_damping}" friction="${test_friction}" />
     </joint>
     <joint name="lr_lower_limb_foot_joint" type="fixed">
@@ -156,4 +164,5 @@
                velocity="${trunk_hip_velocity}" />
         <axis xyz="1 0 0" />
+        <dynamics damping="${test_damping}" friction="${test_friction}" />
     </joint>
     <!-- Right rear leg joints -->
@@ -167,4 +176,5 @@
                velocity="${trunk_hip_velocity}" />
         <axis xyz="-1 0 0" />
+        <dynamics damping="${test_damping}" friction="${test_friction}" />
     </joint>
     <joint name="rr_hip_upper_limb_joint" type="revolute">
@@ -180,4 +190,5 @@
                velocity="${hip_upper_limb_velocity}" />
         <axis xyz="0 1 0" />
+        <dynamics damping="${test_damping}" friction="${test_friction}" />
     </joint>
     <joint name="rr_upper_limb_lower_limb_joint" type="revolute">
@@ -190,4 +201,5 @@
                velocity="${upper_limb_lower_limb_velocity}" />
         <axis xyz="0 1 0" />
+        <dynamics damping="${test_damping}" friction="${test_friction}" />
     </joint>
     <joint name="rr_lower_limb_foot_joint" type="fixed">

Commit message: included link properties in main urdf, created base link and base joint

File: src/meldog_description/description/base_properties.urdf.xacro (robot description, xacro)
@@ -1,59 +1,4 @@
 <?xml version="1.0"?>
 <robot xmlns:xacro="http://www.ros.org/wiki/xacro">
-    <!-- stl mesh names for each link in leg -->
-        <!-- visual tag meshes -->
-        <xacro:property name="hip_vis_stl_name" value="hip_test.stl" />
-        <xacro:property name="upper_limb_vis_stl_name" value="upper_limb_test.stl" />
-        <xacro:property name="lower_limb_vis_stl_name" value="lower_limb_test.stl" />
-        <!-- collision tag meshes -->
-        <xacro:property name="hip_coll_stl_name" value="hip_collision.stl" />
-        <xacro:property name="upper_limb_coll_stl_name" value="upper_limb_collision.stl" />
-        <xacro:property name="lower_limb_coll_stl_name" value="lower_limb_collision.stl" />
-    <!-- limb dimensions -->
-    <xacro:property name="upper_limb_length" value="0.25" />
-    <xacro:property name="lower_limb_length_to_foot" value="0.25" />
-    <!-- inertial properties for each link in left front leg-->
-        <!-- hip link -->
-            <!-- mass -->
-            <xacro:property name="hip_mass" value="3.607"/>
-            <!-- center of mass -->
-            <xacro:property name="hip_cm_x" value="125.497"/>
-            <xacro:property name="hip_cm_y" value="20.770"/>
-            <xacro:property name="hip_cm_z" value="0.248"/>
-            <!-- moments of inertia -->
-            <xacro:property name="hip_ixx" value="4660.408"/>
-            <xacro:property name="hip_ixy" value="-338.226"/>
-            <xacro:property name="hip_ixz" value="0.847"/>
-            <xacro:property name="hip_iyy" value="14607.423"/>
-            <xacro:property name="hip_iyz" value="49.927"/>
-            <xacro:property name="hip_izz" value="13707.172"/>
-        <!-- upper limb link -->
-            <!-- mass -->
-            <xacro:property name="upper_limb_mass" value="0.474"/>
-            <!-- center of mass -->
-            <xacro:property name="upper_limb_cm_x" value="-1.185"/>
-            <xacro:property name="upper_limb_cm_y" value="-4.308"/>
-            <xacro:property name="upper_limb_cm_z" value="-94.203"/>
-            <!-- moments of inertia -->
-            <xacro:property name="upper_limb_ixx" value="4064.505"/>
-            <xacro:property name="upper_limb_ixy" value="1.241"/>
-            <xacro:property name="upper_limb_ixz" value="19.989"/>
-            <xacro:property name="upper_limb_iyy" value="4150.05"/>
-            <xacro:property name="upper_limb_iyz" value="235.648"/>
-            <xacro:property name="upper_limb_izz" value="424.555"/>
-        <!-- lower limb link -->
-            <!-- mass -->
-            <xacro:property name="lower_limb_mass" value="0.116"/>
-            <!-- center of mass -->
-            <xacro:property name="lower_limb_cm_x" value="0.546"/>
-            <xacro:property name="lower_limb_cm_y" value="0"/>
-            <xacro:property name="lower_limb_cm_z" value="-177.643"/>
-            <!-- moments of inertia -->
-            <xacro:property name="lower_limb_ixx" value="967.349"/>
-            <xacro:property name="lower_limb_ixy" value="0"/>
-            <xacro:property name="lower_limb_ixz" value="-4.842"/>
-            <xacro:property name="lower_limb_iyy" value="982.604"/>
-            <xacro:property name="lower_limb_iyz" value="-0.001"/>
-            <xacro:property name="lower_limb_izz" value="37.177"/>
     <!-- joint properties -->
         <!-- body to limb Joint positions -->

File: src/meldog_description/description/meldog_core.urdf.xacro (robot description, xacro)
@@ -3,5 +3,12 @@
     <xacro:include filename="base_properties.urdf.xacro" />
     <xacro:include filename="macros/macros.urdf.xacro" />
+    <!-- Link properties -->
+    <xacro:include filename="links/foot/F_properties.urdf.xacro"/>
+    <xacro:include filename="links/hip/H_properties.urdf.xacro"/>
+    <xacro:include filename="links/lower_limb/LL_properties.urdf.xacro"/>
+    <xacro:include filename="links/upper_limb/UL_properties.urdf.xacro"/>
     <!-- LINKS -->
+        <!-- Base link -->
+        <link name="base_link" />
         <!-- Trunk link -->
         <xacro:include filename="links/trunk.urdf.xacro" />
@@ -43,4 +50,10 @@
             <xacro:include filename="links/foot/RRF_link.urdf.xacro"/>
     <!-- JOINTS -->
+        <!-- Base joint -->
+        <joint name="base_joint" type="fixed">
+            <parent link="base_link" />
+            <child link="trunk_link" />
+            <origin xyz="0 0 0.55" rpy="0 0 0" />
+        </joint>
         <!-- Left front leg joints -->
             <!-- Left front trunk joint -->
