Commit message: renamed joints, renamed ros2_control file

File: src/meldog_description/description/meldog_core.urdf.xacro (robot description, xacro)
@@ -41,5 +41,5 @@
         <xacro:include filename="links/foot/RRF_link.urdf.xacro"/>
     <!-- left front leg joints -->
-    <joint name="lf_hip_upper_limb_joint" type="revolute">
+    <joint name="LFH_joint" type="revolute">
         <parent link="LFH_link" />
         <child link="LFUL_link" />
@@ -54,5 +54,5 @@
         <axis xyz="0 1 0" />
     </joint>
-    <joint name="lf_upper_limb_lower_limb_joint" type="revolute">
+    <joint name="LFK_joint" type="revolute">
         <parent link="LFUL_link" />
         <child link="LFLL_link" />
@@ -64,10 +64,10 @@
         <axis xyz="0 1 0" />
     </joint>
-    <joint name="lf_lower_limb_foot_joint" type="fixed">
+    <joint name="LFF_joint" type="fixed">
         <parent link="LFLL_link" />
         <child link="LFF_link" />
         <origin xyz="0 0 ${-lower_limb_length_to_foot}" rpy="0 0 0" />
     </joint>
-    <joint name="lf_trunk_hip_joint" type="revolute">
+    <joint name="LFT_joint" type="revolute">
         <parent link="trunk_link" />
         <child link="LFH_link" />
@@ -80,5 +80,5 @@
     </joint>
     <!-- Right front leg joints -->
-    <joint name="rf_trunk_hip_joint" type="revolute">
+    <joint name="RFT_joint" type="revolute">
         <parent link="trunk_link" />
         <child link="RFH_link" />
@@ -90,5 +90,5 @@
         <axis xyz="-1 0 0" />
     </joint>
-    <joint name="rf_hip_upper_limb_joint" type="revolute">
+    <joint name="RFH_joint" type="revolute">
         <parent link="RFH_link" />
         <child link="RFUL_link" />
@@ -103,5 +103,5 @@
         <axis xyz="0 1 0" />
     </joint>
-    <joint name="rf_upper_limb_lower_limb_joint" type="revolute">
+    <joint name="RFK_joint" type="revolute">
         <parent link="RFUL_link" />
         <child link="RFLL_link" />
@@ -119,5 +119,5 @@
     </joint>
     <!-- Left rear leg joints -->
-    <joint name="lr_hip_upper_limb_joint" type="revolute">
+    <joint name="LRH_joint" type="revolute">
         <parent link="LRH_link" />
         <child link="LRUL_link" />
@@ -132,5 +132,5 @@
         <axis xyz="0 1 0" />
     </joint>
-    <joint name="lr_upper_limb_lower_limb_joint" type="revolute">
+    <joint name="LRK_joint" type="revolute">
         <parent link="LRUL_link" />
         <child link="LRLL_link" />
@@ -142,10 +142,10 @@
         <axis xyz="0 1 0" />
     </joint>
-    <joint name="lr_lower_limb_foot_joint" type="fixed">
+    <joint name="LRF_joint" type="fixed">
         <parent link="LRLL_link" />
         <child link="LRF_link" />
         <origin xyz="0 0 ${-lower_limb_length_to_foot}" rpy="0 0 0" />
     </joint>
-    <joint name="lr_trunk_hip_joint" type="revolute">
+    <joint name="LRT_joint" type="revolute">
         <parent link="trunk_link" />
         <child link="LRH_link" />
@@ -158,5 +158,5 @@
     </joint>
     <!-- Right rear leg joints -->
-    <joint name="rr_trunk_hip_joint" type="revolute">
+    <joint name="RRT_joint" type="revolute">
         <parent link="trunk_link" />
         <child link="RRH_link" />
@@ -168,5 +168,5 @@
         <axis xyz="-1 0 0" />
     </joint>
-    <joint name="rr_hip_upper_limb_joint" type="revolute">
+    <joint name="RRH_joint" type="revolute">
         <parent link="RRH_link" />
         <child link="RRUL_link" />
@@ -181,5 +181,5 @@
         <axis xyz="0 1 0" />
     </joint>
-    <joint name="rr_upper_limb_lower_limb_joint" type="revolute">
+    <joint name="RRK_joint" type="revolute">
         <parent link="RRUL_link" />
         <child link="RRLL_link" />
@@ -191,5 +191,5 @@
         <axis xyz="0 1 0" />
     </joint>
-    <joint name="rr_lower_limb_foot_joint" type="fixed">
+    <joint name="RRF_joint" type="fixed">
         <parent link="RRLL_link" />
         <child link="RRF_link" />

File: src/meldog_description/description/ros2_control/meldog_gazebo_ros2_control.urdf.xacro (robot description, xacro)
@@ -1,19 +1,11 @@
 <?xml version="1.0"?>
 <robot xmlns:xacro="http://www.ros.org/wiki/xacro">
+    <xacro:include filename="ros2_control_macros.urdf.xacro" />
+    <xacro:include filename="../base_properties.urdf.xacro" />
     <ros2_control name="GazeboSimSystem" type="system">
         <hardware>
           <plugin>gz_ros2_control/GazeboSimSystem</plugin>
         </hardware>
-        <joint name="slider_to_cart">
-          <command_interface name="effort">
-            <param name="min">-1000</param>
-            <param name="max">1000</param>
-          </command_interface>
-          <state_interface name="position">
-            <param name="initial_value">1.0</param>
-          </state_interface>
-          <state_interface name="velocity"/>
-          <state_interface name="effort"/>
-        </joint>
+        <xacro:ros2_control_joint_macro name="lf_hip_upper_limb_joint" pos_min="${hip_upper_limb_lower_limit}" pos_max="${hip_upper_limb_upper_limit}" />
       </ros2_control>
     <gazebo>

Commit message: renamed joints for better readability

File: src/meldog_description/description/meldog_core.urdf.xacro (robot description, xacro)
@@ -41,5 +41,5 @@
         <xacro:include filename="links/foot/RRF_link.urdf.xacro"/>
     <!-- left front leg joints -->
-    <joint name="lf_hip_upper_limb_joint" type="revolute">
+    <joint name="LFH_joint" type="revolute">
         <parent link="LFH_link" />
         <child link="LFUL_link" />
@@ -53,7 +53,6 @@
                velocity="${hip_upper_limb_velocity}" />
         <axis xyz="0 1 0" />
-        <dynamics damping="${test_damping}" friction="${test_friction}" />
     </joint>
-    <joint name="lf_upper_limb_lower_limb_joint" type="revolute">
+    <joint name="LFK_joint" type="revolute">
         <parent link="LFUL_link" />
         <child link="LFLL_link" />
@@ -64,12 +63,11 @@
                velocity="${upper_limb_lower_limb_velocity}" />
         <axis xyz="0 1 0" />
-        <dynamics damping="${test_damping}" friction="${test_friction}" />
     </joint>
-    <joint name="lf_lower_limb_foot_joint" type="fixed">
+    <joint name="LFF_joint" type="fixed">
         <parent link="LFLL_link" />
         <child link="LFF_link" />
         <origin xyz="0 0 ${-lower_limb_length_to_foot}" rpy="0 0 0" />
     </joint>
-    <joint name="lf_trunk_hip_joint" type="revolute">
+    <joint name="LFT_joint" type="revolute">
         <parent link="trunk_link" />
         <child link="LFH_link" />
@@ -80,8 +78,7 @@
                velocity="${trunk_hip_velocity}" />
         <axis xyz="1 0 0" />
-        <dynamics damping="${test_damping}" friction="${test_friction}" />
     </joint>
     <!-- Right front leg joints -->
-    <joint name="rf_trunk_hip_joint" type="revolute">
+    <joint name="RFT_joint" type="revolute">
         <parent link="trunk_link" />
         <child link="RFH_link" />
@@ -92,7 +89,6 @@
                velocity="${trunk_hip_velocity}" />
         <axis xyz="-1 0 0" />
-        <dynamics damping="${test_damping}" friction="${test_friction}" />
     </joint>
-    <joint name="rf_hip_upper_limb_joint" type="revolute">
+    <joint name="RFH_joint" type="revolute">
         <parent link="RFH_link" />
         <child link="RFUL_link" />
@@ -106,7 +102,6 @@
                velocity="${hip_upper_limb_velocity}" />
         <axis xyz="0 1 0" />
-        <dynamics damping="${test_damping}" friction="${test_friction}" />
     </joint>
-    <joint name="rf_upper_limb_lower_limb_joint" type="revolute">
+    <joint name="RFK_joint" type="revolute">
         <parent link="RFUL_link" />
         <child link="RFLL_link" />
@@ -117,5 +112,4 @@
                velocity="${upper_limb_lower_limb_velocity}" />
         <axis xyz="0 1 0" />
-        <dynamics damping="${test_damping}" friction="${test_friction}" />
     </joint>
     <joint name="rf_lower_limb_foot_joint" type="fixed">
@@ -125,5 +119,5 @@
     </joint>
     <!-- Left rear leg joints -->
-    <joint name="lr_hip_upper_limb_joint" type="revolute">
+    <joint name="LRH_joint" type="revolute">
         <parent link="LRH_link" />
         <child link="LRUL_link" />
@@ -137,7 +131,6 @@
                velocity="${hip_upper_limb_velocity}" />
         <axis xyz="0 1 0" />
-        <dynamics damping="${test_damping}" friction="${test_friction}" />
     </joint>
-    <joint name="lr_upper_limb_lower_limb_joint" type="revolute">
+    <joint name="LRK_joint" type="revolute">
         <parent link="LRUL_link" />
         <child link="LRLL_link" />
@@ -148,12 +141,11 @@
                velocity="${upper_limb_lower_limb_velocity}" />
         <axis xyz="0 1 0" />
-        <dynamics damping="${test_damping}" friction="${test_friction}" />
     </joint>
-    <joint name="lr_lower_limb_foot_joint" type="fixed">
+    <joint name="LRF_joint" type="fixed">
         <parent link="LRLL_link" />
         <child link="LRF_link" />
         <origin xyz="0 0 ${-lower_limb_length_to_foot}" rpy="0 0 0" />
     </joint>
-    <joint name="lr_trunk_hip_joint" type="revolute">
+    <joint name="LRT_joint" type="revolute">
         <parent link="trunk_link" />
         <child link="LRH_link" />
@@ -164,8 +156,7 @@
                velocity="${trunk_hip_velocity}" />
         <axis xyz="1 0 0" />
-        <dynamics damping="${test_damping}" friction="${test_friction}" />
     </joint>
     <!-- Right rear leg joints -->
-    <joint name="rr_trunk_hip_joint" type="revolute">
+    <joint name="RRT_joint" type="revolute">
         <parent link="trunk_link" />
         <child link="RRH_link" />
@@ -176,7 +167,6 @@
                velocity="${trunk_hip_velocity}" />
         <axis xyz="-1 0 0" />
-        <dynamics damping="${test_damping}" friction="${test_friction}" />
     </joint>
-    <joint name="rr_hip_upper_limb_joint" type="revolute">
+    <joint name="RRH_joint" type="revolute">
         <parent link="RRH_link" />
         <child link="RRUL_link" />
@@ -190,7 +180,6 @@
                velocity="${hip_upper_limb_velocity}" />
         <axis xyz="0 1 0" />
-        <dynamics damping="${test_damping}" friction="${test_friction}" />
     </joint>
-    <joint name="rr_upper_limb_lower_limb_joint" type="revolute">
+    <joint name="RRK_joint" type="revolute">
         <parent link="RRUL_link" />
         <child link="RRLL_link" />
@@ -201,7 +190,6 @@
                velocity="${upper_limb_lower_limb_velocity}" />
         <axis xyz="0 1 0" />
-        <dynamics damping="${test_damping}" friction="${test_friction}" />
     </joint>
-    <joint name="rr_lower_limb_foot_joint" type="fixed">
+    <joint name="RRF_joint" type="fixed">
         <parent link="RRLL_link" />
         <child link="RRF_link" />
