Commit message: moved joints to separate files in joints folder

File: src/meldog_description/description/meldog_core.urdf.xacro (robot description, xacro)
@@ -4,159 +4,80 @@
     <xacro:include filename="macros/macros.urdf.xacro" />
     <xacro:include filename="links/trunk.urdf.xacro" />
-    <!-- Left front leg links -->
-        <!-- Left front hip link -->
-        <xacro:include filename="links/hip/LFH_link.urdf.xacro"/>
-        <!-- Left front upper limb link -->
-        <xacro:include filename="links/upper_limb/LFUL_link.urdf.xacro"/>
-        <!-- Left front lower limb link -->
-        <xacro:include filename="links/lower_limb/LFLL_link.urdf.xacro"/>
-        <!-- Left front foot link -->
-        <xacro:include filename="links/foot/LFF_link.urdf.xacro"/>
-    <!-- Right front leg links -->
-        <!-- Right front hip link -->
-        <xacro:include filename="links/hip/RFH_link.urdf.xacro"/>
-        <!-- Right front upper limb link -->
-        <xacro:include filename="links/upper_limb/RFUL_link.urdf.xacro"/>
-        <!-- Right front lower limb link -->
-        <xacro:include filename="links/lower_limb/RFLL_link.urdf.xacro"/>
-        <!-- Right front foot link -->
-        <xacro:include filename="links/foot/RFF_link.urdf.xacro"/>
-    <!-- Left rear leg links -->
-        <!-- Left rear hip link -->
-        <xacro:include filename="links/hip/LRH_link.urdf.xacro"/>
-        <!-- Left rear upper limb link -->
-        <xacro:include filename="links/upper_limb/LRUL_link.urdf.xacro"/>
-        <!-- Left rear lower limb link -->
-        <xacro:include filename="links/lower_limb/LRLL_link.urdf.xacro"/>
-        <!-- Left rear foot link -->
-        <xacro:include filename="links/foot/LRF_link.urdf.xacro"/>
-    <!-- Right rear leg links -->
-        <!-- Right rear hip link -->
-        <xacro:include filename="links/hip/RRH_link.urdf.xacro"/>
-        <!-- Right rear upper limb link -->
-        <xacro:include filename="links/upper_limb/RRUL_link.urdf.xacro"/>
-        <!-- Right rear lower limb link -->
-        <xacro:include filename="links/lower_limb/RRLL_link.urdf.xacro"/>
-        <!-- Right rear foot link -->
-        <xacro:include filename="links/foot/RRF_link.urdf.xacro"/>
-    <!-- left front leg joints -->
-    <joint name="LFH_joint" type="revolute">
-        <parent link="LFH_link" />
-        <child link="LFUL_link" />
-        <origin xyz="${hip_upper_limb_x}
-                     ${hip_upper_limb_y}
-                     ${hip_upper_limb_z}"
-                rpy="0 0 0" />
-        <limit lower="${hip_upper_limb_lower_limit/180.0*pi}"
-               upper="${hip_upper_limb_upper_limit/180.0*pi}"
-               effort="${hip_upper_limb_effort}"
-               velocity="${hip_upper_limb_velocity}" />
-        <axis xyz="0 1 0" />
-    </joint>
-    <joint name="LFK_joint" type="revolute">
-        <parent link="LFUL_link" />
-        <child link="LFLL_link" />
-        <origin xyz="0 0 ${-upper_limb_length}" rpy="0 0 0" />
-        <limit lower="${upper_limb_lower_limb_lower_limit/180.0*pi}"
-               upper="${upper_limb_lower_limb_upper_limit/180.0*pi}"
-               effort="${upper_limb_lower_limb_effort}"
-               velocity="${upper_limb_lower_limb_velocity}" />
-        <axis xyz="0 1 0" />
-    </joint>
-    <joint name="LFF_joint" type="fixed">
-        <parent link="LFLL_link" />
-        <child link="LFF_link" />
-        <origin xyz="0 0 ${-lower_limb_length_to_foot}" rpy="0 0 0" />
-    </joint>
-    <joint name="LFT_joint" type="revolute">
-        <parent link="trunk_link" />
-        <child link="LFH_link" />
-        <origin xyz="${trunk_actuators_length/2.0} ${(trunk_base_width+trunk_actuators_width)/2.0} 0" rpy="0 0 0" />
-        <limit lower="${trunk_hip_lower_limit/180.0*pi}"
-               upper="${trunk_hip_upper_limit/180.0*pi}"
-               effort="${trunk_hip_effort}"
-               velocity="${trunk_hip_velocity}" />
-        <axis xyz="1 0 0" />
-    </joint>
-    <!-- Right front leg joints -->
-    <joint name="RFT_joint" type="revolute">
-        <parent link="trunk_link" />
-        <child link="RFH_link" />
-        <origin xyz="${trunk_actuators_length/2.0} ${-(trunk_base_width+trunk_actuators_width)/2.0} 0" rpy="0 0 0" />
-        <limit lower="${trunk_hip_lower_limit/180.0*pi}"
-               upper="${trunk_hip_upper_limit/180.0*pi}"
-               effort="${trunk_hip_effort}"
-               velocity="${trunk_hip_velocity}" />
-        <axis xyz="-1 0 0" />
-    </joint>
-    <joint name="RFH_joint" type="revolute">
-        <parent link="RFH_link" />
-        <child link="RFUL_link" />
-        <origin xyz="${hip_upper_limb_x}
-                     ${-hip_upper_limb_y}
-                     ${hip_upper_limb_z}"
-                rpy="0 0 0" />
-        <limit lower="${hip_upper_limb_lower_limit/180.0*pi}"
-               upper="${hip_upper_limb_upper_limit/180.0*pi}"
-               effort="${hip_upper_limb_effort}"
-               velocity="${hip_upper_limb_velocity}" />
-        <axis xyz="0 1 0" />
-    </joint>
-    <joint name="RFK_joint" type="revolute">
-        <parent link="RFUL_link" />
-        <child link="RFLL_link" />
-        <origin xyz="0 0 ${-upper_limb_length}" rpy="0 0 0" />
-        <limit lower="${upper_limb_lower_limb_lower_limit/180.0*pi}"
-               upper="${upper_limb_lower_limb_upper_limit/180.0*pi}"
-               effort="${upper_limb_lower_limb_effort}"
-               velocity="${upper_limb_lower_limb_velocity}" />
-        <axis xyz="0 1 0" />
-    </joint>
-    <joint name="rf_lower_limb_foot_joint" type="fixed">
-        <parent link="RFLL_link" />
-        <child link="RFF_link" />
-        <origin xyz="0 0 ${-lower_limb_length_to_foot}" rpy="0 0 0" />
-    </joint>
-    <!-- Left rear leg joints -->
-    <joint name="LRH_joint" type="revolute">
-        <parent link="LRH_link" />
-        <child link="LRUL_link" />
-        <origin xyz="${-hip_upper_limb_x}
-                     ${hip_upper_limb_y}
-                     ${hip_upper_limb_z}"
-                rpy="0 0 0" />
-        <limit lower="${hip_upper_limb_lower_limit/180.0*pi}"
-               upper="${hip_upper_limb_upper_limit/180.0*pi}"
-               effort="${hip_upper_limb_effort}"
-               velocity="${hip_upper_limb_velocity}" />
-        <axis xyz="0 1 0" />
-    </joint>
-    <joint name="LRK_joint" type="revolute">
-        <parent link="LRUL_link" />
-        <child link="LRLL_link" />
-        <origin xyz="0 0 ${-upper_limb_length}" rpy="0 0 0" />
-        <limit lower="${upper_limb_lower_limb_lower_limit/180.0*pi}"
-               upper="${upper_limb_lower_limb_upper_limit/180.0*pi}"
-               effort="${upper_limb_lower_limb_effort}"
-               velocity="${upper_limb_lower_limb_velocity}" />
-        <axis xyz="0 1 0" />
-    </joint>
-    <joint name="LRF_joint" type="fixed">
-        <parent link="LRLL_link" />
-        <child link="LRF_link" />
-        <origin xyz="0 0 ${-lower_limb_length_to_foot}" rpy="0 0 0" />
-    </joint>
-    <joint name="LRT_joint" type="revolute">
-        <parent link="trunk_link" />
-        <child link="LRH_link" />
-        <origin xyz="${-trunk_actuators_length/2.0} ${(trunk_base_width+trunk_actuators_width)/2.0} 0" rpy="0 0 0" />
-        <limit lower="${trunk_hip_lower_limit/180.0*pi}"
-               upper="${trunk_hip_upper_limit/180.0*pi}"
-               effort="${trunk_hip_effort}"
-               velocity="${trunk_hip_velocity}" />
-        <axis xyz="1 0 0" />
-    </joint>
+    <!-- LINKS -->
+        <!-- Left front leg links -->
+            <!-- Left front hip link -->
+            <xacro:include filename="links/hip/LFH_link.urdf.xacro"/>
+            <!-- Left front upper limb link -->
+            <xacro:include filename="links/upper_limb/LFUL_link.urdf.xacro"/>
+            <!-- Left front lower limb link -->
+            <xacro:include filename="links/lower_limb/LFLL_link.urdf.xacro"/>
+            <!-- Left front foot link -->
+            <xacro:include filename="links/foot/LFF_link.urdf.xacro"/>
+        <!-- Right front leg links -->
+            <!-- Right front hip link -->
+            <xacro:include filename="links/hip/RFH_link.urdf.xacro"/>
+            <!-- Right front upper limb link -->
+            <xacro:include filename="links/upper_limb/RFUL_link.urdf.xacro"/>
+            <!-- Right front lower limb link -->
+            <xacro:include filename="links/lower_limb/RFLL_link.urdf.xacro"/>
+            <!-- Right front foot link -->
+            <xacro:include filename="links/foot/RFF_link.urdf.xacro"/>
+        <!-- Left rear leg links -->
+            <!-- Left rear hip link -->
+            <xacro:include filename="links/hip/LRH_link.urdf.xacro"/>
+            <!-- Left rear upper limb link -->
+            <xacro:include filename="links/upper_limb/LRUL_link.urdf.xacro"/>
+            <!-- Left rear lower limb link -->
+            <xacro:include filename="links/lower_limb/LRLL_link.urdf.xacro"/>
+            <!-- Left rear foot link -->
+            <xacro:include filename="links/foot/LRF_link.urdf.xacro"/>
+        <!-- Right rear leg links -->
+            <!-- Right rear hip link -->
+            <xacro:include filename="links/hip/RRH_link.urdf.xacro"/>
+            <!-- Right rear upper limb link -->
+            <xacro:include filename="links/upper_limb/RRUL_link.urdf.xacro"/>
+            <!-- Right rear lower limb link -->
+            <xacro:include filename="links/lower_limb/RRLL_link.urdf.xacro"/>
+            <!-- Right rear foot link -->
+            <xacro:include filename="links/foot/RRF_link.urdf.xacro"/>
+    <!-- JOINTS -->
+        <!-- Left front leg joints -->
+            <!-- Left front trunk joint -->
+            <xacro:include filename="joints/trunk/LFT_joint.urdf.xacro"/>
+            <!-- Left front hip joint -->
+            <xacro:include filename="joints/hip/LFH_joint.urdf.xacro"/>
+            <!-- Left front knee joint -->
+            <xacro:include filename="joints/knee/LFK_joint.urdf.xacro"/>
+            <!-- Left front foot joint -->
+            <xacro:include filename="joints/foot/LFF_joint.urdf.xacro"/>
+        <!-- Right front leg joints -->
+            <!-- Right front trunk joint -->
+            <xacro:include filename="joints/trunk/RFT_joint.urdf.xacro"/>
+            <!-- Right front hip joint -->
+            <xacro:include filename="joints/hip/RFH_joint.urdf.xacro"/>
+            <!-- Right front knee joint -->
+            <xacro:include filename="joints/knee/RFK_joint.urdf.xacro"/>
+            <!-- Right front foot joint -->
+            <xacro:include filename="joints/foot/RFF_joint.urdf.xacro"/>
+        <!-- Left rear leg joints -->
+            <!-- Left rear trunk joint -->
+            <xacro:include filename="joints/trunk/LRT_joint.urdf.xacro"/>
+            <!-- Left rear hip joint -->
+            <xacro:include filename="joints/hip/LRH_joint.urdf.xacro"/>
+            <!-- Left rear knee joint -->
+            <xacro:include filename="joints/knee/LRK_joint.urdf.xacro"/>
+            <!-- Left rear foot joint -->
+            <xacro:include filename="joints/foot/LRF_joint.urdf.xacro"/>
+        <!-- Right rear leg joints -->
+            <!-- Right rear trunk joint -->
+            <xacro:include filename="joints/trunk/RRT_joint.urdf.xacro"/>
+            <!-- Right rear hip joint -->
+            <xacro:include filename="joints/hip/RRH_joint.urdf.xacro"/>
+            <!-- Right rear knee joint -->
+            <xacro:include filename="joints/knee/RRK_joint.urdf.xacro"/>
+            <!-- Right rear foot joint -->
+            <xacro:include filename="joints/foot/RRF_joint.urdf.xacro"/>
     <!-- Right rear leg joints -->
-    <joint name="RRT_joint" type="revolute">
+    <!-- <joint name="RRT_joint" type="revolute">
         <parent link="trunk_link" />
         <child link="RRH_link" />
@@ -167,6 +88,6 @@
                velocity="${trunk_hip_velocity}" />
         <axis xyz="-1 0 0" />
-    </joint>
-    <joint name="RRH_joint" type="revolute">
+    </joint> -->
+    <!-- <joint name="RRH_joint" type="revolute">
         <parent link="RRH_link" />
         <child link="RRUL_link" />
@@ -180,6 +101,6 @@
                velocity="${hip_upper_limb_velocity}" />
         <axis xyz="0 1 0" />
-    </joint>
-    <joint name="RRK_joint" type="revolute">
+    </joint> -->
+    <!-- <joint name="RRK_joint" type="revolute">
         <parent link="RRUL_link" />
         <child link="RRLL_link" />
@@ -190,9 +111,9 @@
                velocity="${upper_limb_lower_limb_velocity}" />
         <axis xyz="0 1 0" />
-    </joint>
-    <joint name="RRF_joint" type="fixed">
+    </joint> -->
+    <!-- <joint name="RRF_joint" type="fixed">
         <parent link="RRLL_link" />
         <child link="RRF_link" />
         <origin xyz="0 0 ${-lower_limb_length_to_foot}" rpy="0 0 0" />
-    </joint>
+    </joint> -->
 </robot>

Commit message: added simple joint trajectory controller

File: src/meldog_description/description/meldog_core.urdf.xacro (robot description, xacro)
@@ -4,5 +4,7 @@
     <xacro:include filename="macros/macros.urdf.xacro" />
     <xacro:include filename="links/trunk.urdf.xacro" />
+    <xacro:include filename="ros2_control/meldog_gazebo_ros2_control.urdf.xacro"/>
     <!-- LINKS -->
+        <link name="base_link" />
         <!-- Left front leg links -->
             <!-- Left front hip link -->
@@ -42,4 +44,9 @@
             <xacro:include filename="links/foot/RRF_link.urdf.xacro"/>
     <!-- JOINTS -->
+        <joint name="base_joint" type="fixed">
+            <parent link="base_link" />
+            <child link="trunk_link" />
+            <origin xyz="0 0 0.55" rpy="0 0 0" />
+        </joint>
         <!-- Left front leg joints -->
             <!-- Left front trunk joint -->

File: src/meldog_description/description/ros2_control/meldog_gazebo_ros2_control.urdf.xacro (robot description, xacro)
@@ -3,7 +3,7 @@
     <xacro:include filename="ros2_control_macros.urdf.xacro" />
     <xacro:include filename="../base_properties.urdf.xacro" />
-    <ros2_control name="GazeboSimSystem" type="system">
+    <ros2_control name="IgnitionSystem" type="system">
         <hardware>
-          <plugin>gz_ros2_control/GazeboSimSystem</plugin>
+          <plugin>ign_ros2_control/IgnitionSystem</plugin>
         </hardware>
         <!-- joints -->
@@ -21,19 +21,27 @@
         <xacro:ros2_control_joint_macro name="RRK" pos_min="${hip_upper_limb_lower_limit}" pos_max="${hip_upper_limb_upper_limit}" />
         <!-- transmission -->
-        <xacro:simple_transmission joint="LFT" reduction="1" offset="0.0" />
-        <xacro:simple_transmission joint="LFH" reduction="1" offset="0.0" />
+        <xacro:simple_transmission joint="LFT" reduction="10" offset="0.0" />
+        <xacro:simple_transmission joint="LFH" reduction="10" offset="0.0" />
         <xacro:simple_transmission joint="LFK" reduction="1" offset="0.0" />
-        <xacro:simple_transmission joint="RFT" reduction="1" offset="0.0" />
-        <xacro:simple_transmission joint="RFH" reduction="1" offset="0.0" />
-        <xacro:simple_transmission joint="RFK" reduction="1" offset="0.0" />
-        <xacro:simple_transmission joint="LRT" reduction="1" offset="0.0" />
-        <xacro:simple_transmission joint="LRH" reduction="1" offset="0.0" />
-        <xacro:simple_transmission joint="LRK" reduction="1" offset="0.0" />
-        <xacro:simple_transmission joint="RRT" reduction="1" offset="0.0" />
-        <xacro:simple_transmission joint="RRH" reduction="1" offset="0.0" />
-        <xacro:simple_transmission joint="RRK" reduction="1" offset="0.0" />
+        <xacro:simple_transmission joint="RFT" reduction="10" offset="0.0" />
+        <xacro:simple_transmission joint="RFH" reduction="10" offset="0.0" />
+        <xacro:simple_transmission joint="RFK" reduction="10" offset="0.0" />
+        <xacro:simple_transmission joint="LRT" reduction="10" offset="0.0" />
+        <xacro:simple_transmission joint="LRH" reduction="10" offset="0.0" />
+        <xacro:simple_transmission joint="LRK" reduction="10" offset="0.0" />
+        <xacro:simple_transmission joint="RRT" reduction="10" offset="0.0" />
+        <xacro:simple_transmission joint="RRH" reduction="10" offset="0.0" />
+        <xacro:simple_transmission joint="RRK" reduction="10" offset="0.0" />
     </ros2_control>
     <gazebo>
-        <plugin filename="libgz_ros2_control-system.so" name="gz_ros2_control::GazeboSimROS2ControlPlugin">
+        <plugin filename="ign_ros2_control-system" name="ign_ros2_control::IgnitionROS2ControlPlugin">
+          <robot_param>robot_description</robot_param>
+          <robot_param_node>robot_state_publisher</robot_param_node>
+          <parameters>$(find meldog_description)/controllers/meldog_controllers.yaml</parameters>
+          <hold_joints>true</hold_joints>
+        </plugin>
+      </gazebo>
+    <!-- <gazebo>
+        <plugin filename="ign_ros2_control-system" name="ign_ros2_control::IgnitionROS2ControlPlugin">
             <robot_param>robot_description</robot_param>
             <robot_param_node>robot_state_publisher</robot_param_node>
@@ -42,4 +50,4 @@
             <controller_manager_name>controller_manager</controller_manager_name>
         </plugin>
-    </gazebo>
+    </gazebo> -->
 </robot>

File: src/meldog_description/description/ros2_control/ros2_control_macros.urdf.xacro (robot description, xacro)
@@ -3,15 +3,15 @@
     <xacro:macro name="ros2_control_joint_macro" params="name pos_min pos_max">
         <joint name="${name}_joint">
-            <command_interface name="position">
+            <!-- <command_interface name="position">
               <param name="min">${pos_min}</param>
               <param name="max">${pos_max}</param>
-            </command_interface>
-            <command_interface name="velocity" >
-              <param name="min">-100</param>
-              <param name="max">100</param>
-            </command_interface>
+            </command_interface> -->
+            <!-- <command_interface name="velocity" >
+              <param name="min">-1000</param>
+              <param name="max">1000</param>
+            </command_interface> -->
             <command_interface name="effort">
-              <param name="min">-100</param>
-              <param name="max">100</param>
+              <param name="min">-1000</param>
+              <param name="max">1000</param>
             </command_interface>
             <state_interface name="position" />
@@ -21,7 +21,7 @@
     </xacro:macro>
     <xacro:macro name="simple_transmission" params="joint reduction offset">
-      <transmission name="${name}_transmission">
+      <transmission name="${joint}_transmission">
         <plugin>transmission_interface/SimpleTransmission</plugin>
-        <joint name="${name}_joint" role="joint1">
+        <joint name="${joint}_joint" role="joint1">
             <mechanical_reduction>${reduction}</mechanical_reduction>
             <offset>${offset}</offset>
