Commit message: removed commented code in main urdf

File: src/meldog_description/description/meldog_core.urdf.xacro (robot description, xacro)
@@ -28,25 +28,4 @@
             <!-- Left front foot link -->
             <xacro:include filename="links/foot/LFF_link.urdf.xacro"/>
-            <!-- <link name="LFF_link">
-                <visual>
-                    <geometry>
-                        <sphere radius="0.035" />
-                    </geometry>
-                    <origin xyz="0 0 0" rpy="0 0 0" />
-                </visual>
-                <collision>
-                    <geometry>
-                        <sphere radius="0.035" />
-                    </geometry>
-                    <origin xyz="0 0 0" rpy="0 0 0" />
-                </collision>
-                <inertial>
-                    <mass value="${foot_mass}" />
-                    <origin xyz="${foot_cm_x*0.001} ${foot_cm_y*0.001} ${foot_cm_z*0.001}" rpy="0 0 0" />
-                    <inertia ixx="${foot_ixx*0.000001}" ixy="${foot_ixy*0.000001}" ixz="${foot_ixz*0.000001}"
-                                               iyy="${foot_iyy*0.000001}" iyz="${foot_iyz*0.000001}"
-                                                                     izz="${foot_izz*0.000001}" />
-                </inertial>
-            </link> -->
         <!-- Right front leg links -->
             <!-- Right front hip link -->
@@ -58,25 +37,4 @@
             <!-- Right front foot link -->
             <xacro:include filename="links/foot/RFF_link.urdf.xacro"/>
-            <!-- <link name="RFF_link">
-                <visual>
-                    <geometry>
-                        <sphere radius="0.035" />
-                    </geometry>
-                    <origin xyz="0 0 0" rpy="0 0 0" />
-                </visual>
-                <collision>
-                    <geometry>
-                        <sphere radius="0.035" />
-                    </geometry>
-                    <origin xyz="0 0 0" rpy="0 0 0" />
-                </collision>
-                <inertial>
-                    <mass value="${foot_mass}" />
-                    <origin xyz="${foot_cm_x*0.001} ${foot_cm_y*0.001} ${foot_cm_z*0.001}" rpy="0 0 0" />
-                    <inertia ixx="${foot_ixx*0.000001}" ixy="${foot_ixy*0.000001}" ixz="${foot_ixz*0.000001}"
-                                               iyy="${foot_iyy*0.000001}" iyz="${foot_iyz*0.000001}"
-                                                                     izz="${foot_izz*0.000001}" />
-                </inertial>
-            </link> -->
         <!-- Left rear leg links -->
             <!-- Left rear hip link -->
@@ -88,25 +46,4 @@
             <!-- Left rear foot link -->
             <xacro:include filename="links/foot/LRF_link.urdf.xacro"/>
-            <!-- <link name="LRF_link">
-                <visual>
-                    <geometry>
-                        <sphere radius="0.035" />
-                    </geometry>
-                    <origin xyz="0 0 0" rpy="0 0 0" />
-                </visual>
-                <collision>
-                    <geometry>
-                        <sphere radius="0.035" />
-                    </geometry>
-                    <origin xyz="0 0 0" rpy="0 0 0" />
-                </collision>
-                <inertial>
-                    <mass value="${foot_mass}" />
-                    <origin xyz="${foot_cm_x*0.001} ${foot_cm_y*0.001} ${foot_cm_z*0.001}" rpy="0 0 0" />
-                    <inertia ixx="${foot_ixx*0.000001}" ixy="${foot_ixy*0.000001}" ixz="${foot_ixz*0.000001}"
-                                               iyy="${foot_iyy*0.000001}" iyz="${foot_iyz*0.000001}"
-                                                                     izz="${foot_izz*0.000001}" />
-                </inertial>
-            </link> -->
         <!-- Right rear leg links -->
             <!-- Right rear hip link -->
@@ -118,25 +55,4 @@
             <!-- Right rear foot link -->
             <xacro:include filename="links/foot/RRF_link.urdf.xacro"/>
-            <!-- <link name="RRF_link">
-                <visual>
-                    <geometry>
-                        <sphere radius="0.035" />
-                    </geometry>
-                    <origin xyz="0 0 0" rpy="0 0 0" />
-                </visual>
-                <collision>
-                    <geometry>
-                        <sphere radius="0.035" />
-                    </geometry>
-                    <origin xyz="0 0 0" rpy="0 0 0" />
-                </collision>
-                <inertial>
-                    <mass value="${foot_mass}" />
-                    <origin xyz="${foot_cm_x*0.001} ${foot_cm_y*0.001} ${foot_cm_z*0.001}" rpy="0 0 0" />
-                    <inertia ixx="${foot_ixx*0.000001}" ixy="${foot_ixy*0.000001}" ixz="${foot_ixz*0.000001}"
-                                               iyy="${foot_iyy*0.000001}" iyz="${foot_iyz*0.000001}"
-                                                                     izz="${foot_izz*0.000001}" />
-                </inertial>
-            </link> -->
     <!-- JOINTS -->
         <joint name="base_joint" type="fixed">
