Commit message: added separate property files for each type of link and joint

File: src/meldog_description/description/links/foot/LFF_link.urdf.xacro (robot description, xacro)
@@ -1,6 +1,4 @@
 <?xml version="1.0"?>
 <robot xmlns:xacro="http://www.ros.org/wiki/xacro">
-    <xacro:include filename="../../base_properties.urdf.xacro" />
-    <xacro:include filename="../../macros/macros.urdf.xacro"/>
     <link name="LFF_link" />
 </robot>

File: src/meldog_description/description/links/foot/LRF_link.urdf.xacro (robot description, xacro)
@@ -1,6 +1,4 @@
 <?xml version="1.0"?>
 <robot xmlns:xacro="http://www.ros.org/wiki/xacro">
-    <xacro:include filename="../../base_properties.urdf.xacro" />
-    <xacro:include filename="../../macros/macros.urdf.xacro"/>
     <link name="LRF_link" />
 </robot>

File: src/meldog_description/description/links/foot/RFF_link.urdf.xacro (robot description, xacro)
@@ -1,6 +1,4 @@
 <?xml version="1.0"?>
 <robot xmlns:xacro="http://www.ros.org/wiki/xacro">
-    <xacro:include filename="../../base_properties.urdf.xacro" />
-    <xacro:include filename="../../macros/macros.urdf.xacro"/>
     <link name="RFF_link" />
 </robot>

File: src/meldog_description/description/links/foot/properties.urdf.xacro (robot description, xacro)
@@ -1,4 +1,3 @@
 <?xml version="1.0"?>
 <robot xmlns:xacro="http://www.ros.org/wiki/xacro">
-    <link name="RRF_link" />
 </robot>

File: src/meldog_description/description/links/hip/LFH_link.urdf.xacro (robot description, xacro)
@@ -1,6 +1,4 @@
 <?xml version="1.0"?>
 <robot xmlns:xacro="http://www.ros.org/wiki/xacro">
-    <xacro:include filename="../../base_properties.urdf.xacro" />
-    <xacro:include filename="../../macros/macros.urdf.xacro"/>
     <xacro:link_macro
         name="LFH_link"

File: src/meldog_description/description/links/hip/LRH_link.urdf.xacro (robot description, xacro)
@@ -1,6 +1,4 @@
 <?xml version="1.0"?>
 <robot xmlns:xacro="http://www.ros.org/wiki/xacro">
-    <xacro:include filename="../../base_properties.urdf.xacro" />
-    <xacro:include filename="../../macros/macros.urdf.xacro"/>
     <xacro:link_macro
         name="LRH_link"

File: src/meldog_description/description/links/hip/RFH_link.urdf.xacro (robot description, xacro)
@@ -1,6 +1,4 @@
 <?xml version="1.0"?>
 <robot xmlns:xacro="http://www.ros.org/wiki/xacro">
-    <xacro:include filename="../../base_properties.urdf.xacro" />
-    <xacro:include filename="../../macros/macros.urdf.xacro"/>
     <xacro:link_macro
         name="RFH_link"

File: src/meldog_description/description/links/hip/RRH_link.urdf.xacro (robot description, xacro)
@@ -1,6 +1,4 @@
 <?xml version="1.0"?>
 <robot xmlns:xacro="http://www.ros.org/wiki/xacro">
-    <xacro:include filename="../../base_properties.urdf.xacro" />
-    <xacro:include filename="../../macros/macros.urdf.xacro"/>
     <xacro:link_macro
         name="RRH_link"

File: src/meldog_description/description/links/lower_limb/LFLL_link.urdf.xacro (robot description, xacro)
@@ -1,6 +1,4 @@
 <?xml version="1.0"?>
 <robot xmlns:xacro="http://www.ros.org/wiki/xacro">
-    <xacro:include filename="../../base_properties.urdf.xacro" />
-    <xacro:include filename="../../macros/macros.urdf.xacro"/>
     <xacro:link_macro
         name="LFLL_link"

File: src/meldog_description/description/links/lower_limb/LRLL_link.urdf.xacro (robot description, xacro)
@@ -1,6 +1,4 @@
 <?xml version="1.0"?>
 <robot xmlns:xacro="http://www.ros.org/wiki/xacro">
-    <xacro:include filename="../../base_properties.urdf.xacro" />
-    <xacro:include filename="../../macros/macros.urdf.xacro"/>
     <xacro:link_macro
         name="LRLL_link"

File: src/meldog_description/description/links/lower_limb/RFLL_link.urdf.xacro (robot description, xacro)
@@ -1,6 +1,4 @@
 <?xml version="1.0"?>
 <robot xmlns:xacro="http://www.ros.org/wiki/xacro">
-    <xacro:include filename="../../base_properties.urdf.xacro" />
-    <xacro:include filename="../../macros/macros.urdf.xacro"/>
     <xacro:link_macro
     name="RFLL_link"

File: src/meldog_description/description/links/lower_limb/RRLL_link.urdf.xacro (robot description, xacro)
@@ -1,6 +1,4 @@
 <?xml version="1.0"?>
 <robot xmlns:xacro="http://www.ros.org/wiki/xacro">
-    <xacro:include filename="../../base_properties.urdf.xacro" />
-    <xacro:include filename="../../macros/macros.urdf.xacro"/>
     <xacro:link_macro
     name="RRLL_link"

File: src/meldog_description/description/links/upper_limb/LFUL_link.urdf.xacro (robot description, xacro)
@@ -1,6 +1,4 @@
 <?xml version="1.0"?>
 <robot xmlns:xacro="http://www.ros.org/wiki/xacro">
-    <xacro:include filename="../../base_properties.urdf.xacro" />
-    <xacro:include filename="../../macros/macros.urdf.xacro"/>
     <xacro:link_macro
         name="LFUL_link"

File: src/meldog_description/description/links/upper_limb/LRUL_link.urdf.xacro (robot description, xacro)
@@ -1,6 +1,4 @@
 <?xml version="1.0"?>
 <robot xmlns:xacro="http://www.ros.org/wiki/xacro">
-    <xacro:include filename="../../base_properties.urdf.xacro" />
-    <xacro:include filename="../../macros/macros.urdf.xacro"/>
     <xacro:link_macro
         name="LRUL_link"

File: src/meldog_description/description/links/upper_limb/RFUL_link.urdf.xacro (robot description, xacro)
@@ -1,6 +1,4 @@
 <?xml version="1.0"?>
 <robot xmlns:xacro="http://www.ros.org/wiki/xacro">
-    <xacro:include filename="../../base_properties.urdf.xacro" />
-    <xacro:include filename="../../macros/macros.urdf.xacro"/>
     <xacro:link_macro
         name="RFUL_link"

File: src/meldog_description/description/links/upper_limb/RRUL_link.urdf.xacro (robot description, xacro)
@@ -1,6 +1,4 @@
 <?xml version="1.0"?>
 <robot xmlns:xacro="http://www.ros.org/wiki/xacro">
-    <xacro:include filename="../../base_properties.urdf.xacro" />
-    <xacro:include filename="../../macros/macros.urdf.xacro"/>
     <xacro:link_macro
         name="RRUL_link"

File: src/meldog_description/description/meldog_core.urdf.xacro (robot description, xacro)
@@ -3,6 +3,7 @@
     <xacro:include filename="base_properties.urdf.xacro" />
     <xacro:include filename="macros/macros.urdf.xacro" />
-    <xacro:include filename="links/trunk.urdf.xacro" />
     <!-- LINKS -->
+        <!-- Trunk link -->
+        <xacro:include filename="links/trunk.urdf.xacro" />
         <!-- Left front leg links -->
             <!-- Left front hip link -->
@@ -78,42 +79,3 @@
             <!-- Right rear foot joint -->
             <xacro:include filename="joints/foot/RRF_joint.urdf.xacro"/>
-    <!-- Right rear leg joints -->
-    <!-- <joint name="RRT_joint" type="revolute">
-        <parent link="trunk_link" />
-        <child link="RRH_link" />
-        <origin xyz="${-trunk_actuators_length/2.0} ${-(trunk_base_width+trunk_actuators_width)/2.0} 0" rpy="0 0 0" />
-        <limit lower="${trunk_hip_lower_limit/180.0*pi}"
-               upper="${trunk_hip_upper_limit/180.0*pi}"
-               effort="${trunk_hip_effort}"
-               velocity="${trunk_hip_velocity}" />
-        <axis xyz="-1 0 0" />
-    </joint> -->
-    <!-- <joint name="RRH_joint" type="revolute">
-        <parent link="RRH_link" />
-        <child link="RRUL_link" />
-        <origin xyz="${-hip_upper_limb_x}
-                     ${-hip_upper_limb_y}
-                     ${hip_upper_limb_z}"
-                rpy="0 0 0" />
-        <limit lower="${hip_upper_limb_lower_limit/180.0*pi}"
-               upper="${hip_upper_limb_upper_limit/180.0*pi}"
-               effort="${hip_upper_limb_effort}"
-               velocity="${hip_upper_limb_velocity}" />
-        <axis xyz="0 1 0" />
-    </joint> -->
-    <!-- <joint name="RRK_joint" type="revolute">
-        <parent link="RRUL_link" />
-        <child link="RRLL_link" />
-        <origin xyz="0 0 ${-upper_limb_length}" rpy="0 0 0" />
-        <limit lower="${upper_limb_lower_limb_lower_limit/180.0*pi}"
-               upper="${upper_limb_lower_limb_upper_limit/180.0*pi}"
-               effort="${upper_limb_lower_limb_effort}"
-               velocity="${upper_limb_lower_limb_velocity}" />
-        <axis xyz="0 1 0" />
-    </joint> -->
-    <!-- <joint name="RRF_joint" type="fixed">
-        <parent link="RRLL_link" />
-        <child link="RRF_link" />
-        <origin xyz="0 0 ${-lower_limb_length_to_foot}" rpy="0 0 0" />
-    </joint> -->
 </robot>

Commit message: added separate foot joints and updated lower limb vis and coll models

File: src/meldog_description/description/links/foot/LFF_link.urdf.xacro (robot description, xacro)
@@ -1,4 +1,14 @@
 <?xml version="1.0"?>
 <robot xmlns:xacro="http://www.ros.org/wiki/xacro">
-    <link name="LFF_link" />
+    <xacro:link_macro
+        name="LFF_link"
+        vis_name="${foot_vis_stl_name}"
+        coll_name="${foot_coll_stl_name}"
+        m="${foot_mass}"
+        cm_x="${foot_cm_x}"
+        cm_y="${foot_cm_y}"
+        cm_z="${foot_cm_z}"
+        ixx="${foot_ixx}" ixy="${foot_ixy}" ixz="${foot_ixz}"
+                          iyy="${foot_iyy}" iyz="${foot_iyz}"
+                                            izz="${foot_izz}"/>
 </robot>

File: src/meldog_description/description/links/foot/LRF_link.urdf.xacro (robot description, xacro)
@@ -1,4 +1,14 @@
 <?xml version="1.0"?>
 <robot xmlns:xacro="http://www.ros.org/wiki/xacro">
-    <link name="LRF_link" />
+    <xacro:link_macro
+        name="LRF_link"
+        vis_name="${foot_vis_stl_name}"
+        coll_name="${foot_coll_stl_name}"
+        m="${foot_mass}"
+        cm_x="${-foot_cm_x}"
+        cm_y="${foot_cm_y}"
+        cm_z="${foot_cm_z}"
+        ixx="${foot_ixx}" ixy="${-foot_ixy}" ixz="${-foot_ixz}"
+                         iyy="${foot_iyy}" iyz="${foot_iyz}"
+                                          izz="${foot_izz}"/>
 </robot>

File: src/meldog_description/description/links/foot/RFF_link.urdf.xacro (robot description, xacro)
@@ -1,4 +1,14 @@
 <?xml version="1.0"?>
 <robot xmlns:xacro="http://www.ros.org/wiki/xacro">
-    <link name="RFF_link" />
+    <xacro:link_macro
+        name="RFF_link"
+        vis_name="${foot_vis_stl_name}"
+        coll_name="${foot_coll_stl_name}"
+        m="${foot_mass}"
+        cm_x="${foot_cm_x}"
+        cm_y="${-foot_cm_y}"
+        cm_z="${foot_cm_z}"
+        ixx="${foot_ixx}" ixy="${-foot_ixy}" ixz="${foot_ixz}"
+                         iyy="${foot_iyy}" iyz="${-foot_iyz}"
+                                          izz="${foot_izz}"/>
 </robot>

File: src/meldog_description/description/links/foot/RRF_link.urdf.xacro (robot description, xacro)
@@ -1,4 +1,14 @@
 <?xml version="1.0"?>
 <robot xmlns:xacro="http://www.ros.org/wiki/xacro">
-    <link name="RRF_link" />
+    <xacro:link_macro
+        name="RRF_link"
+        vis_name="${foot_vis_stl_name}"
+        coll_name="${foot_coll_stl_name}"
+        m="${foot_mass}"
+        cm_x="${-foot_cm_x}"
+        cm_y="${-foot_cm_y}"
+        cm_z="${foot_cm_z}"
+        ixx="${foot_ixx}" ixy="${foot_ixy}" ixz="${-foot_ixz}"
+                         iyy="${foot_iyy}" iyz="${-foot_iyz}"
+                                          izz="${foot_izz}"/>
 </robot>

File: src/meldog_description/description/links/hip/LRH_link.urdf.xacro (robot description, xacro)
@@ -10,5 +10,5 @@
         cm_z="${hip_cm_z}"
         ixx="${hip_ixx}" ixy="${-hip_ixy}" ixz="${-hip_ixz}"
-                         iyy="${hip_iyy}" iyz="${hip_iyz}"
-                                          izz="${hip_izz}"/>
+                         iyy="${hip_iyy}"  iyz="${hip_iyz}"
+                                           izz="${hip_izz}"/>
 </robot>

File: src/meldog_description/description/links/properties/F_properties.urdf.xacro (robot description, xacro)
@@ -1,3 +1,20 @@
 <?xml version="1.0"?>
 <robot xmlns:xacro="http://www.ros.org/wiki/xacro">
+    <!-- meshes -->
+    <xacro:property name="foot_vis_stl_name" value="foot_vis.stl" />
+    <xacro:property name="foot_coll_stl_name" value="foot_collision.stl" />
+    <!-- inertial properties -->
+        <!-- mass -->
+        <xacro:property name="foot_mass" value="0.037"/>
+        <!-- center of mass -->
+        <xacro:property name="foot_cm_x" value="0.0"/>
+        <xacro:property name="foot_cm_y" value="0.0"/>
+        <xacro:property name="foot_cm_z" value="-8.417"/>
+        <!-- tensor of inertia -->
+        <xacro:property name="foot_ixx" value="14.919"/>
+        <xacro:property name="foot_ixy" value="0.0"/>
+        <xacro:property name="foot_ixz" value="0.0"/>
+        <xacro:property name="foot_iyy" value="25.291"/>
+        <xacro:property name="foot_iyz" value="0.0"/>
+        <xacro:property name="foot_izz" value="23.390"/>
 </robot>

File: src/meldog_description/description/links/properties/LL_properties.urdf.xacro (robot description, xacro)
@@ -2,5 +2,5 @@
 <robot xmlns:xacro="http://www.ros.org/wiki/xacro">
     <!-- meshes -->
-    <xacro:property name="lower_limb_vis_stl_name" value="lower_limb_test.stl" />
+    <xacro:property name="lower_limb_vis_stl_name" value="LL_vis_v2.stl" />
     <xacro:property name="lower_limb_coll_stl_name" value="lower_limb_collision.stl" />
     <!-- Limb dimensions -->
@@ -8,15 +8,15 @@
     <!-- inertial properties -->
         <!-- mass -->
-        <xacro:property name="lower_limb_mass" value="0.116"/>
+        <xacro:property name="lower_limb_mass" value="0.079"/>
         <!-- center of mass -->
-        <xacro:property name="lower_limb_cm_x" value="0.546"/>
+        <xacro:property name="lower_limb_cm_x" value="0.801"/>
         <xacro:property name="lower_limb_cm_y" value="0"/>
-        <xacro:property name="lower_limb_cm_z" value="-177.643"/>
+        <xacro:property name="lower_limb_cm_z" value="-139.836"/>
         <!-- moments of inertia -->
-        <xacro:property name="lower_limb_ixx" value="967.349"/>
-        <xacro:property name="lower_limb_ixy" value="0"/>
-        <xacro:property name="lower_limb_ixz" value="-4.842"/>
-        <xacro:property name="lower_limb_iyy" value="982.604"/>
-        <xacro:property name="lower_limb_iyz" value="-0.001"/>
-        <xacro:property name="lower_limb_izz" value="37.177"/>
+        <xacro:property name="lower_limb_ixx" value="598.222"/>
+        <xacro:property name="lower_limb_ixy" value="0.0"/>
+        <xacro:property name="lower_limb_ixz" value="-2.447"/>
+        <xacro:property name="lower_limb_iyy" value="603.088"/>
+        <xacro:property name="lower_limb_iyz" value="0.0"/>
+        <xacro:property name="lower_limb_izz" value="13.771"/>
 </robot>
