Commit message: fixed issue with foot collision causing low RTF, modified link macro

File: src/meldog_description/description/links/foot/LFF_link.urdf.xacro (robot description, xacro)
@@ -3,6 +3,7 @@
     <xacro:link_macro
         name="LFF_link"
+        is_foot="1"
         vis_name="${foot_vis_stl_name}"
-        coll_name="${foot_coll_stl_name}"
+        coll_name="empty"
         m="${foot_mass}"
         cm_x="${foot_cm_x}"

File: src/meldog_description/description/links/foot/LRF_link.urdf.xacro (robot description, xacro)
@@ -3,6 +3,7 @@
     <xacro:link_macro
         name="LRF_link"
+        is_foot="1"
         vis_name="${foot_vis_stl_name}"
-        coll_name="${foot_coll_stl_name}"
+        coll_name="empty"
         m="${foot_mass}"
         cm_x="${-foot_cm_x}"

File: src/meldog_description/description/links/foot/RFF_link.urdf.xacro (robot description, xacro)
@@ -3,6 +3,7 @@
     <xacro:link_macro
         name="RFF_link"
+        is_foot="1"
         vis_name="${foot_vis_stl_name}"
-        coll_name="${foot_coll_stl_name}"
+        coll_name="empty"
         m="${foot_mass}"
         cm_x="${foot_cm_x}"

File: src/meldog_description/description/links/foot/RRF_link.urdf.xacro (robot description, xacro)
@@ -3,6 +3,7 @@
     <xacro:link_macro
         name="RRF_link"
+        is_foot="1"
         vis_name="${foot_vis_stl_name}"
-        coll_name="${foot_coll_stl_name}"
+        coll_name="empty"
         m="${foot_mass}"
         cm_x="${-foot_cm_x}"

File: src/meldog_description/description/links/hip/LFH_link.urdf.xacro (robot description, xacro)
@@ -3,4 +3,5 @@
     <xacro:link_macro
         name="LFH_link"
+        is_foot="0"
         vis_name="${hip_vis_stl_name}"
         coll_name="${hip_coll_stl_name}"

File: src/meldog_description/description/links/hip/LRH_link.urdf.xacro (robot description, xacro)
@@ -3,4 +3,5 @@
     <xacro:link_macro
         name="LRH_link"
+        is_foot="0"
         vis_name="rear_left_hip.stl"
         coll_name="rear_left_hip_collision.stl"

File: src/meldog_description/description/links/hip/RFH_link.urdf.xacro (robot description, xacro)
@@ -3,4 +3,5 @@
     <xacro:link_macro
         name="RFH_link"
+        is_foot="0"
         vis_name="front_right_hip.stl"
         coll_name="front_right_hip_collision.stl"

File: src/meldog_description/description/links/hip/RRH_link.urdf.xacro (robot description, xacro)
@@ -3,4 +3,5 @@
     <xacro:link_macro
         name="RRH_link"
+        is_foot="0"
         vis_name="rear_right_hip.stl"
         coll_name="rear_right_hip_collision.stl"

File: src/meldog_description/description/links/lower_limb/LFLL_link.urdf.xacro (robot description, xacro)
@@ -3,4 +3,5 @@
     <xacro:link_macro
         name="LFLL_link"
+        is_foot="0"
         vis_name="${lower_limb_vis_stl_name}"
         coll_name="${lower_limb_coll_stl_name}"

File: src/meldog_description/description/links/lower_limb/LRLL_link.urdf.xacro (robot description, xacro)
@@ -3,4 +3,5 @@
     <xacro:link_macro
         name="LRLL_link"
+        is_foot="0"
         vis_name="${lower_limb_vis_stl_name}"
         coll_name="${lower_limb_coll_stl_name}"

File: src/meldog_description/description/links/lower_limb/RFLL_link.urdf.xacro (robot description, xacro)
@@ -2,13 +2,14 @@
 <robot xmlns:xacro="http://www.ros.org/wiki/xacro">
     <xacro:link_macro
-    name="RFLL_link"
-    vis_name="${lower_limb_vis_stl_name}"
-    coll_name="${lower_limb_coll_stl_name}"
-    m="${lower_limb_mass}"
-    cm_x="${lower_limb_cm_x}"
-    cm_y="${-lower_limb_cm_y}"
-    cm_z="${lower_limb_cm_z}"
-    ixx="${lower_limb_ixx}" ixy="${-lower_limb_ixy}" ixz="${lower_limb_ixz}"
-                            iyy="${lower_limb_iyy}" iyz="${-lower_limb_iyz}"
-                                                    izz="${lower_limb_izz}"/>
+        name="RFLL_link"
+        is_foot="0"
+        vis_name="${lower_limb_vis_stl_name}"
+        coll_name="${lower_limb_coll_stl_name}"
+        m="${lower_limb_mass}"
+        cm_x="${lower_limb_cm_x}"
+        cm_y="${-lower_limb_cm_y}"
+        cm_z="${lower_limb_cm_z}"
+        ixx="${lower_limb_ixx}" ixy="${-lower_limb_ixy}" ixz="${lower_limb_ixz}"
+                                iyy="${lower_limb_iyy}" iyz="${-lower_limb_iyz}"
+                                                        izz="${lower_limb_izz}"/>
 </robot>

File: src/meldog_description/description/links/lower_limb/RRLL_link.urdf.xacro (robot description, xacro)
@@ -2,13 +2,14 @@
 <robot xmlns:xacro="http://www.ros.org/wiki/xacro">
     <xacro:link_macro
-    name="RRLL_link"
-    vis_name="${lower_limb_vis_stl_name}"
-    coll_name="${lower_limb_coll_stl_name}"
-    m="${lower_limb_mass}"
-    cm_x="${-lower_limb_cm_x}"
-    cm_y="${-lower_limb_cm_y}"
-    cm_z="${lower_limb_cm_z}"
-    ixx="${lower_limb_ixx}" ixy="${lower_limb_ixy}" ixz="${-lower_limb_ixz}"
-                            iyy="${lower_limb_iyy}" iyz="${-lower_limb_iyz}"
-                                                    izz="${lower_limb_izz}"/>
+        name="RRLL_link"
+        is_foot="0"
+        vis_name="${lower_limb_vis_stl_name}"
+        coll_name="${lower_limb_coll_stl_name}"
+        m="${lower_limb_mass}"
+        cm_x="${-lower_limb_cm_x}"
+        cm_y="${-lower_limb_cm_y}"
+        cm_z="${lower_limb_cm_z}"
+        ixx="${lower_limb_ixx}" ixy="${lower_limb_ixy}" ixz="${-lower_limb_ixz}"
+                                iyy="${lower_limb_iyy}" iyz="${-lower_limb_iyz}"
+                                                        izz="${lower_limb_izz}"/>
 </robot>

File: src/meldog_description/description/links/properties/F_properties.urdf.xacro (robot description, xacro)
@@ -1,4 +1,6 @@
 <?xml version="1.0"?>
 <robot xmlns:xacro="http://www.ros.org/wiki/xacro">
+    <!-- foot radius -->
+    <xacro:property name="foot_radius" value="0.035" />
     <!-- meshes -->
     <xacro:property name="foot_vis_stl_name" value="foot_vis.stl" />

File: src/meldog_description/description/links/upper_limb/LFUL_link.urdf.xacro (robot description, xacro)
@@ -3,4 +3,5 @@
     <xacro:link_macro
         name="LFUL_link"
+        is_foot="0"
         vis_name="${upper_limb_vis_stl_name}"
         coll_name="${upper_limb_coll_stl_name}"

File: src/meldog_description/description/links/upper_limb/LRUL_link.urdf.xacro (robot description, xacro)
@@ -3,4 +3,5 @@
     <xacro:link_macro
         name="LRUL_link"
+        is_foot="0"
         vis_name="upper_limb_test.stl"
         coll_name="upper_limb_collision.stl"

File: src/meldog_description/description/links/upper_limb/RFUL_link.urdf.xacro (robot description, xacro)
@@ -3,4 +3,5 @@
     <xacro:link_macro
         name="RFUL_link"
+        is_foot="0"
         vis_name="r_upper_limb_vis.stl"
         coll_name="upper_limb_collision.stl"

File: src/meldog_description/description/links/upper_limb/RRUL_link.urdf.xacro (robot description, xacro)
@@ -3,4 +3,5 @@
     <xacro:link_macro
         name="RRUL_link"
+        is_foot="0"
         vis_name="r_upper_limb_vis.stl"
         coll_name="upper_limb_collision.stl"

File: src/meldog_description/description/macros/link_macro.urdf.xacro (robot description, xacro)
@@ -4,5 +4,5 @@
     the visual and collision models coordinate
     systems are placed in joints -->
-    <xacro:macro name="link_macro" params="name vis_name coll_name m cm_x cm_y cm_z ixx ixy ixz iyy iyz izz">
+    <xacro:macro name="link_macro" params="name is_foot vis_name coll_name m cm_x cm_y cm_z ixx ixy ixz iyy iyz izz">
         <link name="${name}">
             <visual>
@@ -13,11 +13,21 @@
                 <origin xyz="0 0 0" rpy="0 0 0"/>
             </visual>
-            <collision>
-                <geometry>
-                    <mesh filename="package://meldog_description/meshes/collision/${coll_name}"
-                          scale="0.001 0.001 0.001" />
-                </geometry>
-                <origin xyz="0 0 0" rpy="0 0 0" />
-            </collision>
+            <xacro:if value="${is_foot == 1}">
+                <collision>
+                    <geometry>
+                        <sphere radius="${foot_radius}" />
+                    </geometry>
+                    <origin xyz="0 0 0" rpy="0 0 0" />
+                </collision>
+            </xacro:if>
+            <xacro:if value="${is_foot == 0}">
+                <collision>
+                    <geometry>
+                        <mesh filename="package://meldog_description/meshes/collision/${coll_name}"
+                            scale="0.001 0.001 0.001" />
+                    </geometry>
+                    <origin xyz="0 0 0" rpy="0 0 0" />
+                </collision>
+            </xacro:if>
             <inertial>
                 <mass value="${m}" />

File: src/meldog_description/description/meldog_core.urdf.xacro (robot description, xacro)
@@ -28,4 +28,25 @@
             <!-- Left front foot link -->
             <xacro:include filename="links/foot/LFF_link.urdf.xacro"/>
+            <!-- <link name="LFF_link">
+                <visual>
+                    <geometry>
+                        <sphere radius="0.035" />
+                    </geometry>
+                    <origin xyz="0 0 0" rpy="0 0 0" />
+                </visual>
+                <collision>
+                    <geometry>
+                        <sphere radius="0.035" />
+                    </geometry>
+                    <origin xyz="0 0 0" rpy="0 0 0" />
+                </collision>
+                <inertial>
+                    <mass value="${foot_mass}" />
+                    <origin xyz="${foot_cm_x*0.001} ${foot_cm_y*0.001} ${foot_cm_z*0.001}" rpy="0 0 0" />
+                    <inertia ixx="${foot_ixx*0.000001}" ixy="${foot_ixy*0.000001}" ixz="${foot_ixz*0.000001}"
+                                               iyy="${foot_iyy*0.000001}" iyz="${foot_iyz*0.000001}"
+                                                                     izz="${foot_izz*0.000001}" />
+                </inertial>
+            </link> -->
         <!-- Right front leg links -->
             <!-- Right front hip link -->
@@ -37,4 +58,25 @@
             <!-- Right front foot link -->
             <xacro:include filename="links/foot/RFF_link.urdf.xacro"/>
+            <!-- <link name="RFF_link">
+                <visual>
+                    <geometry>
+                        <sphere radius="0.035" />
+                    </geometry>
+                    <origin xyz="0 0 0" rpy="0 0 0" />
+                </visual>
+                <collision>
+                    <geometry>
+                        <sphere radius="0.035" />
+                    </geometry>
+                    <origin xyz="0 0 0" rpy="0 0 0" />
+                </collision>
+                <inertial>
+                    <mass value="${foot_mass}" />
+                    <origin xyz="${foot_cm_x*0.001} ${foot_cm_y*0.001} ${foot_cm_z*0.001}" rpy="0 0 0" />
+                    <inertia ixx="${foot_ixx*0.000001}" ixy="${foot_ixy*0.000001}" ixz="${foot_ixz*0.000001}"
+                                               iyy="${foot_iyy*0.000001}" iyz="${foot_iyz*0.000001}"
+                                                                     izz="${foot_izz*0.000001}" />
+                </inertial>
+            </link> -->
         <!-- Left rear leg links -->
             <!-- Left rear hip link -->
@@ -46,4 +88,25 @@
             <!-- Left rear foot link -->
             <xacro:include filename="links/foot/LRF_link.urdf.xacro"/>
+            <!-- <link name="LRF_link">
+                <visual>
+                    <geometry>
+                        <sphere radius="0.035" />
+                    </geometry>
+                    <origin xyz="0 0 0" rpy="0 0 0" />
+                </visual>
+                <collision>
+                    <geometry>
+                        <sphere radius="0.035" />
+                    </geometry>
+                    <origin xyz="0 0 0" rpy="0 0 0" />
+                </collision>
+                <inertial>
+                    <mass value="${foot_mass}" />
+                    <origin xyz="${foot_cm_x*0.001} ${foot_cm_y*0.001} ${foot_cm_z*0.001}" rpy="0 0 0" />
+                    <inertia ixx="${foot_ixx*0.000001}" ixy="${foot_ixy*0.000001}" ixz="${foot_ixz*0.000001}"
+                                               iyy="${foot_iyy*0.000001}" iyz="${foot_iyz*0.000001}"
+                                                                     izz="${foot_izz*0.000001}" />
+                </inertial>
+            </link> -->
         <!-- Right rear leg links -->
             <!-- Right rear hip link -->
@@ -55,4 +118,25 @@
             <!-- Right rear foot link -->
             <xacro:include filename="links/foot/RRF_link.urdf.xacro"/>
+            <!-- <link name="RRF_link">
+                <visual>
+                    <geometry>
+                        <sphere radius="0.035" />
+                    </geometry>
+                    <origin xyz="0 0 0" rpy="0 0 0" />
+                </visual>
+                <collision>
+                    <geometry>
+                        <sphere radius="0.035" />
+                    </geometry>
+                    <origin xyz="0 0 0" rpy="0 0 0" />
+                </collision>
+                <inertial>
+                    <mass value="${foot_mass}" />
+                    <origin xyz="${foot_cm_x*0.001} ${foot_cm_y*0.001} ${foot_cm_z*0.001}" rpy="0 0 0" />
+                    <inertia ixx="${foot_ixx*0.000001}" ixy="${foot_ixy*0.000001}" ixz="${foot_ixz*0.000001}"
+                                               iyy="${foot_iyy*0.000001}" iyz="${foot_iyz*0.000001}"
+                                                                     izz="${foot_izz*0.000001}" />
+                </inertial>
+            </link> -->
     <!-- JOINTS -->
         <joint name="base_joint" type="fixed">
