Commit message: added joint controller

File: src/meldog_description/description/gazebo/meldog_gazebo.urdf.xacro (robot description, xacro)
@@ -1,3 +1,13 @@
 <?xml version="1.0"?>
 <robot xmlns:xacro="http://www.ros.org/wiki/xacro">
+    <xacro:macro name="gz_joint" params="name mu1 mu2 kp kd maxVel dampingFactor">
+        <gazebo reference="${name}_link">
+            <mu1 value="${mu1}"/>
+            <mu2 value="${mu2}"/>
+            <kp value="${kp_}" />
+            <kd value="${kd}" />
+            <maxVel value="${maxVel}"/>
+            <dampingFactor value="${dampingFactor}"/>
+        </gazebo>
+    </xacro:macro>
 </robot>

File: src/meldog_description/description/joints/hip/LFH_joint.urdf.xacro (robot description, xacro)
@@ -1,13 +1,12 @@
 <?xml version="1.0"?>
 <robot xmlns:xacro="http://www.ros.org/wiki/xacro">
-    <joint name="LFH_joint" type="continuous">
+    <joint name="LFH_joint" type="revolute">
         <parent link="LFH_link" />
         <child link="LFUL_link" />
         <origin xyz="${H_x}
                      ${H_y}
-                     ${H_z}"
-                rpy="0 0 0" />
-        <limit effort="${H_effort}"
-               velocity="${H_velocity}" />
+                     ${H_z}" rpy="0 0 0" />
+        <limit lower="${H_lower_limit}" upper="${H_upper_limit}"
+               effort="${H_effort}" velocity="${H_velocity}" />
         <axis xyz="0 -1 0" />
     </joint>

File: src/meldog_description/description/joints/hip/LRH_joint.urdf.xacro (robot description, xacro)
@@ -1,5 +1,5 @@
 <?xml version="1.0"?>
 <robot xmlns:xacro="http://www.ros.org/wiki/xacro">
-    <joint name="LRH_joint" type="continuous">
+    <joint name="LRH_joint" type="revolute">
         <parent link="LRH_link" />
         <child link="LRUL_link" />
@@ -8,6 +8,6 @@
                      ${H_z}"
                 rpy="0 0 0" />
-        <limit effort="${H_effort}"
-               velocity="${H_velocity}" />
+        <limit lower="${H_lower_limit}" upper="${H_upper_limit}"
+               effort="${H_effort}" velocity="${H_velocity}" />
         <axis xyz="0 -1 0" />
     </joint>

File: src/meldog_description/description/joints/hip/RFH_joint.urdf.xacro (robot description, xacro)
@@ -1,5 +1,5 @@
 <?xml version="1.0"?>
 <robot xmlns:xacro="http://www.ros.org/wiki/xacro">
-    <joint name="RFH_joint" type="continuous">
+    <joint name="RFH_joint" type="revolute">
         <parent link="RFH_link" />
         <child link="RFUL_link" />
@@ -8,6 +8,6 @@
                      ${H_z}"
                 rpy="0 0 0" />
-        <limit effort="${H_effort}"
-               velocity="${H_velocity}" />
+        <limit lower="${H_lower_limit}" upper="${H_upper_limit}"
+               effort="${H_effort}" velocity="${H_velocity}" />
         <axis xyz="0 -1 0" />
     </joint>

File: src/meldog_description/description/joints/hip/RRH_joint.urdf.xacro (robot description, xacro)
@@ -1,5 +1,5 @@
 <?xml version="1.0"?>
 <robot xmlns:xacro="http://www.ros.org/wiki/xacro">
-    <joint name="RRH_joint" type="continuous">
+    <joint name="RRH_joint" type="revolute">
         <parent link="RRH_link" />
         <child link="RRUL_link" />
@@ -8,6 +8,6 @@
                      ${H_z}"
                 rpy="0 0 0" />
-        <limit effort="${H_effort}"
-               velocity="${H_velocity}" />
+        <limit lower="${H_lower_limit}" upper="${H_upper_limit}"
+               effort="${H_effort}" velocity="${H_velocity}" />
         <axis xyz="0 -1 0" />
     </joint>

File: src/meldog_description/description/joints/properties/H_joint_properties.urdf.xacro (robot description, xacro)
@@ -9,6 +9,6 @@
     <xacro:property name="H_upper_limit" value="120" />
     <!-- Hip joint effort and velocity limits -->
-    <xacro:property name="H_effort" value="100.0" />
-    <xacro:property name="H_velocity" value="100.0" />
+    <xacro:property name="H_effort" value="${motor_max_eff*actuator_reduction}" />
+    <xacro:property name="H_velocity" value="${motor_max_vel*pi/30.0/actuator_reduction}" />
     <!-- Hip joint friction and damping -->
     <xacro:property name="H_damping" value="0"/>

File: src/meldog_description/description/joints/properties/K_joint_properties.urdf.xacro (robot description, xacro)
@@ -5,6 +5,6 @@
     <xacro:property name="K_upper_limit" value="160" />
     <!-- Knee joint effort and velocity limits -->
-    <xacro:property name="K_effort" value="100.0" />
-    <xacro:property name="K_velocity" value="100.0" />
+    <xacro:property name="K_effort" value="${motor_max_eff*actuator_reduction}" />
+    <xacro:property name="K_velocity" value="${motor_max_vel*pi/30.0/actuator_reduction}" />
     <!-- Knee joint friction and damping -->
     <xacro:property name="K_damping" value="0"/>

File: src/meldog_description/description/joints/properties/T_joint_properties.urdf.xacro (robot description, xacro)
@@ -5,6 +5,6 @@
     <xacro:property name="T_upper_limit" value="45" />
     <!-- Trunk joint effort and velocity limits -->
-    <xacro:property name="T_effort" value="100.0" />
-    <xacro:property name="T_velocity" value="100.0" />
+    <xacro:property name="T_effort" value="${motor_max_eff*actuator_reduction}" />
+    <xacro:property name="T_velocity" value="${motor_max_vel*pi/30.0/actuator_reduction}" />
     <!-- Trunk joint friction and damping -->
     <xacro:property name="T_damping" value="0"/>

File: src/meldog_description/description/ros2_control/hardware_properties.urdf.xacro (robot description, xacro)
@@ -3,4 +3,4 @@
     <xacro:property name="motor_max_eff" value="3.5" />
     <xacro:property name="motor_max_vel" value="1800" />
-    <xacro:property name="actuator_reduction" value="0.0625" />
+    <xacro:property name="actuator_reduction" value="9.97" />
 </robot>

File: src/meldog_description/description/ros2_control/meldog_gazebo_ros2_control.urdf.xacro (robot description, xacro)
@@ -11,18 +11,18 @@
         </hardware>
         <!-- joints -->
-        <xacro:ros2_control_joint_macro name="LFT" pos_min="${T_lower_limit}" pos_max="${T_upper_limit}" vel_max="${motor_max_vel}" eff_max="${motor_max_eff}"/>
-        <xacro:ros2_control_joint_macro name="LFH" pos_min="${H_lower_limit}" pos_max="${H_upper_limit}" vel_max="${motor_max_vel}" eff_max="${motor_max_eff}"/>
-        <xacro:ros2_control_joint_macro name="LFK" pos_min="${K_lower_limit}" pos_max="${K_upper_limit}" vel_max="${motor_max_vel}" eff_max="${motor_max_eff}"/>
-        <xacro:ros2_control_joint_macro name="RFT" pos_min="${T_lower_limit}" pos_max="${T_upper_limit}" vel_max="${motor_max_vel}" eff_max="${motor_max_eff}"/>
-        <xacro:ros2_control_joint_macro name="RFH" pos_min="${H_lower_limit}" pos_max="${H_upper_limit}" vel_max="${motor_max_vel}" eff_max="${motor_max_eff}"/>
-        <xacro:ros2_control_joint_macro name="RFK" pos_min="${K_lower_limit}" pos_max="${K_upper_limit}" vel_max="${motor_max_vel}" eff_max="${motor_max_eff}"/>
-        <xacro:ros2_control_joint_macro name="LRT" pos_min="${T_lower_limit}" pos_max="${T_upper_limit}" vel_max="${motor_max_vel}" eff_max="${motor_max_eff}"/>
-        <xacro:ros2_control_joint_macro name="LRH" pos_min="${H_lower_limit}" pos_max="${H_upper_limit}" vel_max="${motor_max_vel}" eff_max="${motor_max_eff}"/>
-        <xacro:ros2_control_joint_macro name="LRK" pos_min="${K_lower_limit}" pos_max="${K_upper_limit}" vel_max="${motor_max_vel}" eff_max="${motor_max_eff}"/>
-        <xacro:ros2_control_joint_macro name="RRT" pos_min="${T_lower_limit}" pos_max="${T_upper_limit}" vel_max="${motor_max_vel}" eff_max="${motor_max_eff}"/>
-        <xacro:ros2_control_joint_macro name="RRH" pos_min="${H_lower_limit}" pos_max="${H_upper_limit}" vel_max="${motor_max_vel}" eff_max="${motor_max_eff}"/>
-        <xacro:ros2_control_joint_macro name="RRK" pos_min="${K_lower_limit}" pos_max="${K_upper_limit}" vel_max="${motor_max_vel}" eff_max="${motor_max_eff}"/>
+        <xacro:ros2_control_joint_macro name="LFT" pos_min="${T_lower_limit}" pos_max="${T_upper_limit}" vel_max="${T_velocity}" eff_max="${T_effort}"/>
+        <xacro:ros2_control_joint_macro name="LFH" pos_min="${H_lower_limit}" pos_max="${H_upper_limit}" vel_max="${H_velocity}" eff_max="${H_effort}"/>
+        <xacro:ros2_control_joint_macro name="LFK" pos_min="${K_lower_limit}" pos_max="${K_upper_limit}" vel_max="${K_velocity}" eff_max="${K_effort}"/>
+        <xacro:ros2_control_joint_macro name="RFT" pos_min="${T_lower_limit}" pos_max="${T_upper_limit}" vel_max="${T_velocity}" eff_max="${T_effort}"/>
+        <xacro:ros2_control_joint_macro name="RFH" pos_min="${H_lower_limit}" pos_max="${H_upper_limit}" vel_max="${H_velocity}" eff_max="${H_effort}"/>
+        <xacro:ros2_control_joint_macro name="RFK" pos_min="${K_lower_limit}" pos_max="${K_upper_limit}" vel_max="${K_velocity}" eff_max="${K_effort}"/>
+        <xacro:ros2_control_joint_macro name="LRT" pos_min="${T_lower_limit}" pos_max="${T_upper_limit}" vel_max="${T_velocity}" eff_max="${T_effort}"/>
+        <xacro:ros2_control_joint_macro name="LRH" pos_min="${H_lower_limit}" pos_max="${H_upper_limit}" vel_max="${H_velocity}" eff_max="${H_effort}"/>
+        <xacro:ros2_control_joint_macro name="LRK" pos_min="${K_lower_limit}" pos_max="${K_upper_limit}" vel_max="${K_velocity}" eff_max="${K_effort}"/>
+        <xacro:ros2_control_joint_macro name="RRT" pos_min="${T_lower_limit}" pos_max="${T_upper_limit}" vel_max="${T_velocity}" eff_max="${T_effort}"/>
+        <xacro:ros2_control_joint_macro name="RRH" pos_min="${H_lower_limit}" pos_max="${H_upper_limit}" vel_max="${H_velocity}" eff_max="${H_effort}"/>
+        <xacro:ros2_control_joint_macro name="RRK" pos_min="${K_lower_limit}" pos_max="${K_upper_limit}" vel_max="${K_velocity}" eff_max="${K_effort}"/>
         <!-- transmission -->
-        <xacro:simple_transmission joint="LFT" reduction="${actuator_reduction}" offset="0.0" />
+        <!-- <xacro:simple_transmission joint="LFT" reduction="${actuator_reduction}" offset="0.0" />
         <xacro:simple_transmission joint="LFH" reduction="${actuator_reduction}" offset="0.0" />
         <xacro:simple_transmission joint="LFK" reduction="${actuator_reduction}" offset="0.0" />
@@ -35,12 +35,16 @@
         <xacro:simple_transmission joint="RRT" reduction="${actuator_reduction}" offset="0.0" />
         <xacro:simple_transmission joint="RRH" reduction="${actuator_reduction}" offset="0.0" />
-        <xacro:simple_transmission joint="RRK" reduction="${actuator_reduction}" offset="0.0" />
+        <xacro:simple_transmission joint="RRK" reduction="${actuator_reduction}" offset="0.0" /> -->
+        <xacro:FourBarLinkageTransmission first_joint_name="LFH" second_joint_name="LFK" />
+        <xacro:FourBarLinkageTransmission first_joint_name="RFH" second_joint_name="RFK" />
+        <xacro:FourBarLinkageTransmission first_joint_name="LRH" second_joint_name="LRK" />
+        <xacro:FourBarLinkageTransmission first_joint_name="RRH" second_joint_name="RRK" />
     </ros2_control>
     <gazebo>
         <plugin filename="ign_ros2_control-system" name="ign_ros2_control::IgnitionROS2ControlPlugin">
-          <robot_param>robot_description</robot_param>
-          <robot_param_node>robot_state_publisher</robot_param_node>
-          <parameters>$(find meldog_description)/controllers/meldog_controllers.yaml</parameters>
-          <hold_joints>true</hold_joints>
+          <!-- <robot_param>robot_description</robot_param>
+          <robot_param_node>robot_state_publisher</robot_param_node> -->
+          <parameters>$(find meldog_description)/controllers/joint_controller.yaml</parameters>
+          <!-- <hold_joints>true</hold_joints> -->
         </plugin>
       </gazebo>

File: src/meldog_description/description/ros2_control/ros2_control_macros.urdf.xacro (robot description, xacro)
@@ -9,10 +9,10 @@
             </command_interface>
             <command_interface name="velocity" >
-              <param name="min">${-vel_max/60.0*2*pi}</param>
-              <param name="max">${vel_max/60.0*2*pi}</param>
+              <param name="min">${-vel_max}</param>
+              <param name="max">${vel_max}</param>
             </command_interface>
             <command_interface name="effort">
-              <param name="min">${-eff_max/actuator_reduction}</param>
-              <param name="max">${eff_max/actuator_reduction}</param>
+              <param name="min">${-eff_max}</param>
+              <param name="max">${eff_max}</param>
             </command_interface>
             <state_interface name="position" />
@@ -30,3 +30,22 @@
       </transmission>
     </xacro:macro>
+    <xacro:macro name="FourBarLinkageTransmission" params="first_joint_name second_joint_name">
+        <transmission name="FourBarLinkageTransmission_${first_joint_name}_${second_joint_name}">
+            <plugin>transmission_interface/FourBarLinkageTransmission</plugin>
+            <!-- <actuator name="${first_joint_name}_actuator" role="actuator1">
+                <mechanical_reduction>${reduction}</mechanical_reduction>
+            </actuator>
+            <actuator name="${second_joint_name}_actuator" role="actuator2">
+                <mechanical_reduction>${reduction}</mechanical_reduction>
+            </actuator> -->
+            <joint name="${first_joint_name}_joint" role="joint1">
+                <mechanical_reduction>1.0</mechanical_reduction>
+                <offset>0.0</offset>
+            </joint>
+            <joint name="${second_joint_name}_joint" role="joint2">
+                <mechanical_reduction>1.0</mechanical_reduction>
+                <offset>0.0</offset>
+            </joint>
+        </transmission>
+    </xacro:macro>
 </robot>
