Commit message: added gazebo properties and macros

File: src/meldog_description/description/gazebo/meldog_gazebo.urdf.xacro (robot description, xacro)
@@ -1,9 +1,14 @@
 <?xml version="1.0"?>
 <robot xmlns:xacro="http://www.ros.org/wiki/xacro">
-    <xacro:macro name="gz_joint" params="name mu1 mu2 kp kd maxVel dampingFactor">
+    <xacro:macro name="gz_link" params="name mu1 mu2 kp kd maxVel dampingFactor">
         <gazebo reference="${name}_link">
+            <visual>
+                <material>
+                    <diffuse>0 0 1 1 </diffuse>
+                </material>
+            </visual>
             <mu1 value="${mu1}"/>
             <mu2 value="${mu2}"/>
-            <kp value="${kp_}" />
+            <kp value="${kp}" />
             <kd value="${kd}" />
             <maxVel value="${maxVel}"/>
@@ -11,3 +16,114 @@
         </gazebo>
     </xacro:macro>
+    <xacro:macro name="gz_joint" params="name isd s_stiff s_ref stopErp stopCfm">
+        <gazebo reference="${name}_joint">
+            <implicitSpringDamper>${isd}</implicitSpringDamper>
+            <springStiffness>${s_stiff}</springStiffness>
+            <springReference>${s_ref}</springReference>
+            <stopErp>${stopErp}</stopErp>
+            <stopCfm>${stopCfm}</stopCfm>
+        </gazebo>
+    </xacro:macro>
+    <!-- If using gazebo link parameters -->
+    <xacro:if value="${use_gz_links==1}">
+        <!-- Trunk link -->
+        <xacro:gz_link name="trunk" mu1="${mu1_value}" mu2="${mu2_value}"
+                       kp="${kp_value}" kd="${kd_value}"
+                       maxVel="${maxVel_value}" dampingFactor="${dampingFactor_value}" />
+        <!-- Left front leg -->
+        <xacro:gz_link name="LFH" mu1="${mu1_value}" mu2="${mu2_value}"
+                       kp="${kp_value}" kd="${kd_value}"
+                       maxVel="${maxVel_value}" dampingFactor="${dampingFactor_value}" />
+        <xacro:gz_link name="LFUL" mu1="${mu1_value}" mu2="${mu2_value}"
+                       kp="${kp_value}" kd="${kd_value}"
+                       maxVel="${maxVel_value}" dampingFactor="${dampingFactor_value}" />
+        <xacro:gz_link name="LFLL" mu1="${mu1_value}" mu2="${mu2_value}"
+                       kp="${kp_value}" kd="${kd_value}"
+                       maxVel="${maxVel_value}" dampingFactor="${dampingFactor_value}" />
+        <xacro:gz_link name="LFF" mu1="${mu1_value_foot}" mu2="${mu2_value_foot}"
+                       kp="${kp_value_foot}" kd="${kd_value_foot}"
+                       maxVel="${maxVel_value_foot}" dampingFactor="${dampingFactor_value_foot}" />
+        <!-- Right front leg -->
+        <xacro:gz_link name="RFH" mu1="${mu1_value}" mu2="${mu2_value}"
+                       kp="${kp_value}" kd="${kd_value}"
+                       maxVel="${maxVel_value}" dampingFactor="${dampingFactor_value}" />
+        <xacro:gz_link name="RFUL" mu1="${mu1_value}" mu2="${mu2_value}"
+                       kp="${kp_value}" kd="${kd_value}"
+                       maxVel="${maxVel_value}" dampingFactor="${dampingFactor_value}" />
+        <xacro:gz_link name="RFLL" mu1="${mu1_value}" mu2="${mu2_value}"
+                       kp="${kp_value}" kd="${kd_value}"
+                       maxVel="${maxVel_value}" dampingFactor="${dampingFactor_value}" />
+        <xacro:gz_link name="RFF" mu1="${mu1_value_foot}" mu2="${mu2_value_foot}"
+                       kp="${kp_value_foot}" kd="${kd_value_foot}"
+                       maxVel="${maxVel_value_foot}" dampingFactor="${dampingFactor_value_foot}" />
+        <!-- Left rear leg -->
+        <xacro:gz_link name="LRH" mu1="${mu1_value}" mu2="${mu2_value}"
+                       kp="${kp_value}" kd="${kd_value}"
+                       maxVel="${maxVel_value}" dampingFactor="${dampingFactor_value}" />
+        <xacro:gz_link name="LRUL" mu1="${mu1_value}" mu2="${mu2_value}"
+                       kp="${kp_value}" kd="${kd_value}"
+                       maxVel="${maxVel_value}" dampingFactor="${dampingFactor_value}" />
+        <xacro:gz_link name="LRLL" mu1="${mu1_value}" mu2="${mu2_value}"
+                       kp="${kp_value}" kd="${kd_value}"
+                       maxVel="${maxVel_value}" dampingFactor="${dampingFactor_value}" />
+        <xacro:gz_link name="LRF" mu1="${mu1_value_foot}" mu2="${mu2_value_foot}"
+                       kp="${kp_value_foot}" kd="${kd_value_foot}"
+                       maxVel="${maxVel_value_foot}" dampingFactor="${dampingFactor_value_foot}" />
+        <!-- Right rear leg -->
+        <xacro:gz_link name="RRH" mu1="${mu1_value}" mu2="${mu2_value}"
+                       kp="${kp_value}" kd="${kd_value}"
+                       maxVel="${maxVel_value}" dampingFactor="${dampingFactor_value}" />
+        <xacro:gz_link name="RRUL" mu1="${mu1_value}" mu2="${mu2_value}"
+                       kp="${kp_value}" kd="${kd_value}"
+                       maxVel="${maxVel_value}" dampingFactor="${dampingFactor_value}" />
+        <xacro:gz_link name="RRLL" mu1="${mu1_value}" mu2="${mu2_value}"
+                       kp="${kp_value}" kd="${kd_value}"
+                       maxVel="${maxVel_value}" dampingFactor="${dampingFactor_value}" />
+        <xacro:gz_link name="RRF" mu1="${mu1_value_foot}" mu2="${mu2_value_foot}"
+                       kp="${kp_value_foot}" kd="${kd_value_foot}"
+                       maxVel="${maxVel_value_foot}" dampingFactor="${dampingFactor_value_foot}" />
+    </xacro:if>
+    <!-- if using gazebo joint parameters -->
+    <xacro:if value="${use_gz_joints==1}">
+        <!-- Left front leg -->
+        <xacro:gz_joint name="LFT" isd="${implicitSpringDamper_value}"
+                       s_stiff="${springStiffness_value}" s_ref="${springReference_value}"
+                       stopErp="${stopErp_value}" stopCfm="${stopCfm_value}" />
+        <xacro:gz_joint name="LFH" isd="${implicitSpringDamper_value}"
+                       s_stiff="${springStiffness_value}" s_ref="${springReference_value}"
+                       stopErp="${stopErp_value}" stopCfm="${stopCfm_value}" />
+        <xacro:gz_joint name="LFK" isd="${implicitSpringDamper_value}"
+                       s_stiff="${springStiffness_value}" s_ref="${springReference_value}"
+                       stopErp="${stopErp_value}" stopCfm="${stopCfm_value}" />
+        <!-- Right front leg -->
+        <xacro:gz_joint name="RFT" isd="${implicitSpringDamper_value}"
+                       s_stiff="${springStiffness_value}" s_ref="${springReference_value}"
+                       stopErp="${stopErp_value}" stopCfm="${stopCfm_value}" />
+        <xacro:gz_joint name="RFH" isd="${implicitSpringDamper_value}"
+                       s_stiff="${springStiffness_value}" s_ref="${springReference_value}"
+                       stopErp="${stopErp_value}" stopCfm="${stopCfm_value}" />
+        <xacro:gz_joint name="RFK" isd="${implicitSpringDamper_value}"
+                       s_stiff="${springStiffness_value}" s_ref="${springReference_value}"
+                       stopErp="${stopErp_value}" stopCfm="${stopCfm_value}" />
+        <!-- Left rear leg -->
+        <xacro:gz_joint name="LRT" isd="${implicitSpringDamper_value}"
+                       s_stiff="${springStiffness_value}" s_ref="${springReference_value}"
+                       stopErp="${stopErp_value}" stopCfm="${stopCfm_value}" />
+        <xacro:gz_joint name="LRH" isd="${implicitSpringDamper_value}"
+                       s_stiff="${springStiffness_value}" s_ref="${springReference_value}"
+                       stopErp="${stopErp_value}" stopCfm="${stopCfm_value}" />
+        <xacro:gz_joint name="LRK" isd="${implicitSpringDamper_value}"
+                       s_stiff="${springStiffness_value}" s_ref="${springReference_value}"
+                       stopErp="${stopErp_value}" stopCfm="${stopCfm_value}" />
+        <!-- Right rear leg -->
+        <xacro:gz_joint name="RRT" isd="${implicitSpringDamper_value}"
+                       s_stiff="${springStiffness_value}" s_ref="${springReference_value}"
+                       stopErp="${stopErp_value}" stopCfm="${stopCfm_value}" />
+        <xacro:gz_joint name="RRH" isd="${implicitSpringDamper_value}"
+                       s_stiff="${springStiffness_value}" s_ref="${springReference_value}"
+                       stopErp="${stopErp_value}" stopCfm="${stopCfm_value}" />
+        <xacro:gz_joint name="RRK" isd="${implicitSpringDamper_value}"
+                       s_stiff="${springStiffness_value}" s_ref="${springReference_value}"
+                       stopErp="${stopErp_value}" stopCfm="${stopCfm_value}" />
+    </xacro:if>
 </robot>

File: src/meldog_description/description/links/trunk.urdf.xacro (robot description, xacro)
@@ -20,7 +20,4 @@
                 <box size="${trunk_base_length} ${trunk_base_width} ${trunk_base_height}"/>
             </geometry>
-            <material name="">
-                <color rgba="0.0 0.0 1.0 1.0"/>
-            </material>
         </visual>
         <visual name="trunk_actuators_left_visual">
@@ -29,7 +26,4 @@
                 <box size="${trunk_actuators_length} ${trunk_actuators_width} ${trunk_actuators_height}"/>
             </geometry>
-            <material name="">
-                <color rgba="0.0 1.0 0.0 1.0"/>
-            </material>
         </visual>
         <visual name="trunk_actuators_right_visual">
@@ -38,7 +32,4 @@
                 <box size="${trunk_actuators_length} ${trunk_actuators_width} ${trunk_actuators_height}"/>
             </geometry>
-            <material name="">
-                <color rgba="1.0 0.0 0.0 1.0"/>
-            </material>
         </visual>
          <collision name="trunk_base_collision">

File: src/meldog_description/description/meldog_core.urdf.xacro (robot description, xacro)
@@ -12,4 +12,7 @@
     <xacro:include filename="joints/properties/H_joint_properties.urdf.xacro"/>
     <xacro:include filename="joints/properties/K_joint_properties.urdf.xacro"/>
+    <!-- Gazebo -->
+    <xacro:include filename="gazebo/gazebo_properties.urdf.xacro" />
+    <xacro:include filename="gazebo/meldog_gazebo.urdf.xacro" />
     <!-- ROS2 Control -->
     <xacro:include filename="ros2_control/meldog_gazebo_ros2_control.urdf.xacro"/>
