Commit message: small changes in urdf and yaml config

File: src/meldog_description/description/gazebo/gazebo_properties.urdf.xacro (robot description, xacro)
@@ -6,5 +6,5 @@
     <xacro:property name="use_gz_joints" value="1" />
     <!-- Gazebo joint parameters -->
-    <xacro:property name="implicitSpringDamper_value" value="0" />
+    <xacro:property name="implicitSpringDamper_value" value="1" />
     <xacro:property name="springStiffness_value" value="0" />
     <xacro:property name="springReference_value" value="0" />

File: src/meldog_description/description/ros2_control/meldog_gazebo_ros2_control.urdf.xacro (robot description, xacro)
@@ -36,15 +36,15 @@
         <xacro:simple_transmission joint="RRH" reduction="${actuator_reduction}" offset="0.0" />
         <xacro:simple_transmission joint="RRK" reduction="${actuator_reduction}" offset="0.0" /> -->
-        <xacro:FourBarLinkageTransmission first_joint_name="LFH" second_joint_name="LFK" />
+        <!-- <xacro:FourBarLinkageTransmission first_joint_name="LFH" second_joint_name="LFK" />
         <xacro:FourBarLinkageTransmission first_joint_name="RFH" second_joint_name="RFK" />
         <xacro:FourBarLinkageTransmission first_joint_name="LRH" second_joint_name="LRK" />
-        <xacro:FourBarLinkageTransmission first_joint_name="RRH" second_joint_name="RRK" />
+        <xacro:FourBarLinkageTransmission first_joint_name="RRH" second_joint_name="RRK" /> -->
     </ros2_control>
     <gazebo>
         <plugin filename="ign_ros2_control-system" name="ign_ros2_control::IgnitionROS2ControlPlugin">
-          <!-- <robot_param>robot_description</robot_param>
-          <robot_param_node>robot_state_publisher</robot_param_node> -->
-          <parameters>$(find meldog_description)/controllers/joint_controller.yaml</parameters>
-          <!-- <hold_joints>true</hold_joints> -->
+          <robot_param>robot_description</robot_param>
+          <robot_param_node>robot_state_publisher</robot_param_node>
+          <parameters>$(find meldog_description)/controllers/meldog_controllers.yaml</parameters>
+          <hold_joints>true</hold_joints>
         </plugin>
       </gazebo>

File: src/meldog_description/description/ros2_control/ros2_control_macros.urdf.xacro (robot description, xacro)
@@ -8,5 +8,5 @@
               <param name="max">${pos_max}</param>
             </command_interface>
-            <command_interface name="velocity" >
+            <!-- <command_interface name="velocity" >
               <param name="min">${-vel_max}</param>
               <param name="max">${vel_max}</param>
@@ -15,5 +15,5 @@
               <param name="min">${-eff_max}</param>
               <param name="max">${eff_max}</param>
-            </command_interface>
+            </command_interface> -->
             <state_interface name="position" />
             <state_interface name="velocity"/>

Commit message: Poprawiony model nogi w gazebo

File: src/meldog_description/description/gazebo/gazebo_properties.urdf.xacro (robot description, xacro)
@@ -6,5 +6,5 @@
     <xacro:property name="use_gz_joints" value="1" />
     <!-- Gazebo joint parameters -->
-    <xacro:property name="implicitSpringDamper_value" value="1" />
+    <xacro:property name="implicitSpringDamper_value" value="0" />
     <xacro:property name="springStiffness_value" value="0" />
     <xacro:property name="springReference_value" value="0" />

File: src/meldog_description/description/joints/hip/LFH_joint.urdf.xacro (robot description, xacro)
@@ -9,5 +9,4 @@
         <limit lower="${H_lower_limit}" upper="${H_upper_limit}"
                effort="${H_effort}" velocity="${H_velocity}" />
-        <dynamics friction="${H_friction}" damping="${H_damping}" />
         <axis xyz="0 -1 0" />
     </joint>

File: src/meldog_description/description/joints/hip/LRH_joint.urdf.xacro (robot description, xacro)
@@ -10,5 +10,4 @@
         <limit lower="${H_lower_limit}" upper="${H_upper_limit}"
                effort="${H_effort}" velocity="${H_velocity}" />
-        <dynamics friction="${H_friction}" damping="${H_damping}" />
         <axis xyz="0 -1 0" />
     </joint>

File: src/meldog_description/description/joints/hip/RFH_joint.urdf.xacro (robot description, xacro)
@@ -10,5 +10,4 @@
         <limit lower="${H_lower_limit}" upper="${H_upper_limit}"
                effort="${H_effort}" velocity="${H_velocity}" />
-        <dynamics friction="${H_friction}" damping="${H_damping}" />
         <axis xyz="0 -1 0" />
     </joint>

File: src/meldog_description/description/joints/hip/RRH_joint.urdf.xacro (robot description, xacro)
@@ -10,5 +10,4 @@
         <limit lower="${H_lower_limit}" upper="${H_upper_limit}"
                effort="${H_effort}" velocity="${H_velocity}" />
-        <dynamics friction="${H_friction}" damping="${H_damping}" />
         <axis xyz="0 -1 0" />
     </joint>

File: src/meldog_description/description/joints/knee/LFK_joint.urdf.xacro (robot description, xacro)
@@ -9,5 +9,4 @@
             effort="${K_effort}"
             velocity="${K_velocity}" />
-        <dynamics friction="${K_friction}" damping="${K_damping}" />
         <axis xyz="0 -1 0" />
     </joint>

File: src/meldog_description/description/joints/knee/LRK_joint.urdf.xacro (robot description, xacro)
@@ -9,5 +9,4 @@
                effort="${K_effort}"
                velocity="${K_velocity}" />
-        <dynamics friction="${K_friction}" damping="${K_damping}" />
         <axis xyz="0 -1 0" />
     </joint>

File: src/meldog_description/description/joints/knee/RFK_joint.urdf.xacro (robot description, xacro)
@@ -9,5 +9,4 @@
                effort="${K_effort}"
                velocity="${K_velocity}" />
-        <dynamics friction="${K_friction}" damping="${K_damping}" />
         <axis xyz="0 -1 0" />
     </joint>

File: src/meldog_description/description/joints/knee/RRK_joint.urdf.xacro (robot description, xacro)
@@ -9,5 +9,4 @@
                effort="${K_effort}"
                velocity="${K_velocity}" />
-        <dynamics friction="${K_friction}" damping="${K_damping}" />
         <axis xyz="0 -1 0" />
     </joint>

File: src/meldog_description/description/joints/properties/H_joint_properties.urdf.xacro (robot description, xacro)
@@ -13,4 +13,4 @@
     <!-- Hip joint friction and damping -->
     <xacro:property name="H_damping" value="0"/>
-    <xacro:property name="H_friction" value="0.0312"/>
+    <xacro:property name="H_friction" value="0"/>
 </robot>

File: src/meldog_description/description/joints/properties/K_joint_properties.urdf.xacro (robot description, xacro)
@@ -9,4 +9,4 @@
     <!-- Knee joint friction and damping -->
     <xacro:property name="K_damping" value="0"/>
-    <xacro:property name="K_friction" value="0.0312"/>
+    <xacro:property name="K_friction" value="0"/>
 </robot>

File: src/meldog_description/description/joints/properties/T_joint_properties.urdf.xacro (robot description, xacro)
@@ -9,4 +9,4 @@
     <!-- Trunk joint friction and damping -->
     <xacro:property name="T_damping" value="0"/>
-    <xacro:property name="T_friction" value="0.0312"/>
+    <xacro:property name="T_friction" value="0"/>
 </robot>

File: src/meldog_description/description/joints/trunk/LFT_joint.urdf.xacro (robot description, xacro)
@@ -9,5 +9,4 @@
                effort="${T_effort}"
                velocity="${T_velocity}" />
-        <dynamics friction="${T_friction}" damping="${T_damping}" />
         <axis xyz="1 0 0" />
     </joint>

File: src/meldog_description/description/joints/trunk/LRT_joint.urdf.xacro (robot description, xacro)
@@ -9,5 +9,4 @@
                effort="${T_effort}"
                velocity="${T_velocity}" />
-        <dynamics friction="${T_friction}" damping="${T_damping}" />
         <axis xyz="1 0 0" />
     </joint>

File: src/meldog_description/description/joints/trunk/RFT_joint.urdf.xacro (robot description, xacro)
@@ -9,5 +9,4 @@
                effort="${T_effort}"
                velocity="${T_velocity}" />
-        <dynamics friction="${T_friction}" damping="${T_damping}" />
         <axis xyz="-1 0 0" />
     </joint>

File: src/meldog_description/description/joints/trunk/RRT_joint.urdf.xacro (robot description, xacro)
@@ -9,5 +9,4 @@
                effort="${T_effort}"
                velocity="${T_velocity}" />
-        <dynamics friction="${T_friction}" damping="${T_damping}" />
         <axis xyz="-1 0 0" />
     </joint>

File: src/meldog_description/description/ros2_control/meldog_gazebo_ros2_control.urdf.xacro (robot description, xacro)
@@ -36,15 +36,15 @@
         <xacro:simple_transmission joint="RRH" reduction="${actuator_reduction}" offset="0.0" />
         <xacro:simple_transmission joint="RRK" reduction="${actuator_reduction}" offset="0.0" /> -->
-        <!-- <xacro:FourBarLinkageTransmission first_joint_name="LFH" second_joint_name="LFK" />
+        <xacro:FourBarLinkageTransmission first_joint_name="LFH" second_joint_name="LFK" />
         <xacro:FourBarLinkageTransmission first_joint_name="RFH" second_joint_name="RFK" />
         <xacro:FourBarLinkageTransmission first_joint_name="LRH" second_joint_name="LRK" />
-        <xacro:FourBarLinkageTransmission first_joint_name="RRH" second_joint_name="RRK" /> -->
+        <xacro:FourBarLinkageTransmission first_joint_name="RRH" second_joint_name="RRK" />
     </ros2_control>
     <gazebo>
         <plugin filename="ign_ros2_control-system" name="ign_ros2_control::IgnitionROS2ControlPlugin">
-          <robot_param>robot_description</robot_param>
-          <robot_param_node>robot_state_publisher</robot_param_node>
-          <parameters>$(find meldog_description)/controllers/meldog_controllers.yaml</parameters>
-          <hold_joints>true</hold_joints>
+          <!-- <robot_param>robot_description</robot_param>
+          <robot_param_node>robot_state_publisher</robot_param_node> -->
+          <parameters>$(find meldog_description)/controllers/joint_controller.yaml</parameters>
+          <!-- <hold_joints>true</hold_joints> -->
         </plugin>
       </gazebo>

File: src/meldog_description/description/ros2_control/ros2_control_macros.urdf.xacro (robot description, xacro)
@@ -8,5 +8,5 @@
               <param name="max">${pos_max}</param>
             </command_interface>
-            <!-- <command_interface name="velocity" >
+            <command_interface name="velocity" >
               <param name="min">${-vel_max}</param>
               <param name="max">${vel_max}</param>
@@ -15,5 +15,5 @@
               <param name="min">${-eff_max}</param>
               <param name="max">${eff_max}</param>
-            </command_interface> -->
+            </command_interface>
             <state_interface name="position" />
             <state_interface name="velocity"/>

File: src/meldog_leg_description/description/links/trunk.urdf.xacro (robot description, xacro)
@@ -1,5 +1,5 @@
 <?xml version="1.0"?>
 <robot xmlns:xacro="http://www.ros.org/wiki/xacro">
-    <xacro:property name="trunk_mass" value="0.001"/>
+    <xacro:property name="trunk_mass" value="0.1"/>
     <link name="trunk_link">
         <inertial>
@@ -20,4 +20,7 @@
             </geometry>
         </collision>
+        <gazebo reference="trunk_link">
+            <kinematic>false</kinematic>
+        </gazebo>
     </link>
 </robot>

File: src/meldog_leg_description/description/meldog_core.urdf.xacro (robot description, xacro)
@@ -18,8 +18,14 @@
     <xacro:include filename="ros2_control/meldog_gazebo_ros2_control.urdf.xacro"/>
     <!-- LINKS -->
+        <link name="world"/>
+        <joint name="world_joint" type="fixed">
+            <parent link="world"/>
+            <child link="base_link"/>
+            <origin xyz="0 0 0" rpy="0 0 0"/>
+        </joint>
         <!-- Base link -->
-        <link name="base_link" />
-        <!-- Trunk link -->
-        <xacro:include filename="links/trunk.urdf.xacro" />
+            <link name="base_link"/>
+            <!-- Trunk link -->
+            <xacro:include filename="links/trunk.urdf.xacro" />
         <!-- Left rear leg links -->
             <!-- Left rear hip link -->
@@ -35,5 +41,5 @@
             <parent link="base_link" />
             <child link="trunk_link" />
-            <origin xyz="0 0 0.55" rpy="0 0 0" />
+            <origin xyz="0 0 0.6" rpy="0 0 0" />
         </joint>
         <!-- Left rear leg joints -->
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