Commit message: added properties folders for links and joints, moved link and joint properties to the newly created folders

File: src/meldog_description/description/joints/hip/LFH_joint.urdf.xacro (robot description, xacro)
@@ -4,12 +4,12 @@
         <parent link="LFH_link" />
         <child link="LFUL_link" />
-        <origin xyz="${hip_upper_limb_x}
-                     ${hip_upper_limb_y}
-                     ${hip_upper_limb_z}"
+        <origin xyz="${H_x}
+                     ${H_y}
+                     ${H_z}"
                 rpy="0 0 0" />
-        <limit lower="${hip_upper_limb_lower_limit/180.0*pi}"
-               upper="${hip_upper_limb_upper_limit/180.0*pi}"
-               effort="${hip_upper_limb_effort}"
-               velocity="${hip_upper_limb_velocity}" />
+        <limit lower="${H_lower_limit/180.0*pi}"
+               upper="${H_upper_limit/180.0*pi}"
+               effort="${H_effort}"
+               velocity="${H_velocity}" />
         <axis xyz="0 1 0" />
     </joint>

File: src/meldog_description/description/joints/hip/LRH_joint.urdf.xacro (robot description, xacro)
@@ -4,12 +4,12 @@
         <parent link="LRH_link" />
         <child link="LRUL_link" />
-        <origin xyz="${-hip_upper_limb_x}
-                     ${hip_upper_limb_y}
-                     ${hip_upper_limb_z}"
+        <origin xyz="${-H_x}
+                     ${H_y}
+                     ${H_z}"
                 rpy="0 0 0" />
-        <limit lower="${hip_upper_limb_lower_limit/180.0*pi}"
-               upper="${hip_upper_limb_upper_limit/180.0*pi}"
-               effort="${hip_upper_limb_effort}"
-               velocity="${hip_upper_limb_velocity}" />
+        <limit lower="${H_lower_limit/180.0*pi}"
+               upper="${H_upper_limit/180.0*pi}"
+               effort="${H_effort}"
+               velocity="${H_velocity}" />
         <axis xyz="0 1 0" />
     </joint>

File: src/meldog_description/description/joints/hip/RFH_joint.urdf.xacro (robot description, xacro)
@@ -4,12 +4,12 @@
         <parent link="RFH_link" />
         <child link="RFUL_link" />
-        <origin xyz="${hip_upper_limb_x}
-                     ${-hip_upper_limb_y}
-                     ${hip_upper_limb_z}"
+        <origin xyz="${H_x}
+                     ${-H_y}
+                     ${H_z}"
                 rpy="0 0 0" />
-        <limit lower="${hip_upper_limb_lower_limit/180.0*pi}"
-               upper="${hip_upper_limb_upper_limit/180.0*pi}"
-               effort="${hip_upper_limb_effort}"
-               velocity="${hip_upper_limb_velocity}" />
+        <limit lower="${H_lower_limit/180.0*pi}"
+               upper="${H_upper_limit/180.0*pi}"
+               effort="${H_effort}"
+               velocity="${H_velocity}" />
         <axis xyz="0 1 0" />
     </joint>

File: src/meldog_description/description/joints/hip/RRH_joint.urdf.xacro (robot description, xacro)
@@ -4,12 +4,12 @@
         <parent link="RRH_link" />
         <child link="RRUL_link" />
-        <origin xyz="${-hip_upper_limb_x}
-                     ${-hip_upper_limb_y}
-                     ${hip_upper_limb_z}"
+        <origin xyz="${-H_x}
+                     ${-H_y}
+                     ${H_z}"
                 rpy="0 0 0" />
-        <limit lower="${hip_upper_limb_lower_limit/180.0*pi}"
-               upper="${hip_upper_limb_upper_limit/180.0*pi}"
-               effort="${hip_upper_limb_effort}"
-               velocity="${hip_upper_limb_velocity}" />
+        <limit lower="${H_lower_limit/180.0*pi}"
+               upper="${H_upper_limit/180.0*pi}"
+               effort="${H_effort}"
+               velocity="${H_velocity}" />
         <axis xyz="0 1 0" />
     </joint>

File: src/meldog_description/description/joints/knee/LFK_joint.urdf.xacro (robot description, xacro)
@@ -5,8 +5,8 @@
         <child link="LFLL_link" />
         <origin xyz="0 0 ${-upper_limb_length}" rpy="0 0 0" />
-        <limit lower="${upper_limb_lower_limb_lower_limit/180.0*pi}"
-            upper="${upper_limb_lower_limb_upper_limit/180.0*pi}"
-            effort="${upper_limb_lower_limb_effort}"
-            velocity="${upper_limb_lower_limb_velocity}" />
+        <limit lower="${K_lower_limit/180.0*pi}"
+            upper="${K_upper_limit/180.0*pi}"
+            effort="${K_effort}"
+            velocity="${K_velocity}" />
         <axis xyz="0 1 0" />
     </joint>

File: src/meldog_description/description/joints/knee/LRK_joint.urdf.xacro (robot description, xacro)
@@ -5,8 +5,8 @@
         <child link="LRLL_link" />
         <origin xyz="0 0 ${-upper_limb_length}" rpy="0 0 0" />
-        <limit lower="${upper_limb_lower_limb_lower_limit/180.0*pi}"
-               upper="${upper_limb_lower_limb_upper_limit/180.0*pi}"
-               effort="${upper_limb_lower_limb_effort}"
-               velocity="${upper_limb_lower_limb_velocity}" />
+        <limit lower="${K_lower_limit/180.0*pi}"
+               upper="${K_upper_limit/180.0*pi}"
+               effort="${K_effort}"
+               velocity="${K_velocity}" />
         <axis xyz="0 1 0" />
     </joint>

File: src/meldog_description/description/joints/knee/RFK_joint.urdf.xacro (robot description, xacro)
@@ -5,8 +5,8 @@
         <child link="RFLL_link" />
         <origin xyz="0 0 ${-upper_limb_length}" rpy="0 0 0" />
-        <limit lower="${upper_limb_lower_limb_lower_limit/180.0*pi}"
-               upper="${upper_limb_lower_limb_upper_limit/180.0*pi}"
-               effort="${upper_limb_lower_limb_effort}"
-               velocity="${upper_limb_lower_limb_velocity}" />
+        <limit lower="${K_lower_limit/180.0*pi}"
+               upper="${K_upper_limit/180.0*pi}"
+               effort="${K_effort}"
+               velocity="${K_velocity}" />
         <axis xyz="0 1 0" />
     </joint>

File: src/meldog_description/description/joints/knee/RRK_joint.urdf.xacro (robot description, xacro)
@@ -5,8 +5,8 @@
         <child link="RRLL_link" />
         <origin xyz="0 0 ${-upper_limb_length}" rpy="0 0 0" />
-        <limit lower="${upper_limb_lower_limb_lower_limit/180.0*pi}"
-               upper="${upper_limb_lower_limb_upper_limit/180.0*pi}"
-               effort="${upper_limb_lower_limb_effort}"
-               velocity="${upper_limb_lower_limb_velocity}" />
+        <limit lower="${K_lower_limit/180.0*pi}"
+               upper="${K_upper_limit/180.0*pi}"
+               effort="${K_effort}"
+               velocity="${K_velocity}" />
         <axis xyz="0 1 0" />
     </joint>

File: src/meldog_description/description/joints/trunk/LFT_joint.urdf.xacro (robot description, xacro)
@@ -5,8 +5,8 @@
         <child link="LFH_link" />
         <origin xyz="${trunk_actuators_length/2.0} ${(trunk_base_width+trunk_actuators_width)/2.0} 0" rpy="0 0 0" />
-        <limit lower="${trunk_hip_lower_limit/180.0*pi}"
-               upper="${trunk_hip_upper_limit/180.0*pi}"
-               effort="${trunk_hip_effort}"
-               velocity="${trunk_hip_velocity}" />
+        <limit lower="${T_lower_limit/180.0*pi}"
+               upper="${T_upper_limit/180.0*pi}"
+               effort="${T_effort}"
+               velocity="${T_velocity}" />
         <axis xyz="1 0 0" />
     </joint>

File: src/meldog_description/description/joints/trunk/LRT_joint.urdf.xacro (robot description, xacro)
@@ -5,8 +5,8 @@
         <child link="LRH_link" />
         <origin xyz="${-trunk_actuators_length/2.0} ${(trunk_base_width+trunk_actuators_width)/2.0} 0" rpy="0 0 0" />
-        <limit lower="${trunk_hip_lower_limit/180.0*pi}"
-               upper="${trunk_hip_upper_limit/180.0*pi}"
-               effort="${trunk_hip_effort}"
-               velocity="${trunk_hip_velocity}" />
+        <limit lower="${T_lower_limit/180.0*pi}"
+               upper="${T_upper_limit/180.0*pi}"
+               effort="${T_effort}"
+               velocity="${T_velocity}" />
         <axis xyz="1 0 0" />
     </joint>

File: src/meldog_description/description/joints/trunk/RFT_joint.urdf.xacro (robot description, xacro)
@@ -5,8 +5,8 @@
         <child link="RFH_link" />
         <origin xyz="${trunk_actuators_length/2.0} ${-(trunk_base_width+trunk_actuators_width)/2.0} 0" rpy="0 0 0" />
-        <limit lower="${trunk_hip_lower_limit/180.0*pi}"
-               upper="${trunk_hip_upper_limit/180.0*pi}"
-               effort="${trunk_hip_effort}"
-               velocity="${trunk_hip_velocity}" />
+        <limit lower="${T_lower_limit/180.0*pi}"
+               upper="${T_upper_limit/180.0*pi}"
+               effort="${T_effort}"
+               velocity="${T_velocity}" />
         <axis xyz="-1 0 0" />
     </joint>

File: src/meldog_description/description/joints/trunk/RRT_joint.urdf.xacro (robot description, xacro)
@@ -5,8 +5,8 @@
         <child link="RRH_link" />
         <origin xyz="${-trunk_actuators_length/2.0} ${-(trunk_base_width+trunk_actuators_width)/2.0} 0" rpy="0 0 0" />
-        <limit lower="${trunk_hip_lower_limit/180.0*pi}"
-               upper="${trunk_hip_upper_limit/180.0*pi}"
-               effort="${trunk_hip_effort}"
-               velocity="${trunk_hip_velocity}" />
+        <limit lower="${T_lower_limit/180.0*pi}"
+               upper="${T_upper_limit/180.0*pi}"
+               effort="${T_effort}"
+               velocity="${T_velocity}" />
         <axis xyz="-1 0 0" />
     </joint>

File: src/meldog_description/description/meldog_core.urdf.xacro (robot description, xacro)
@@ -1,11 +1,15 @@
 <?xml version="1.0"?>
 <robot name="meldog_core" xmlns:xacro="http://www.ros.org/wiki/xacro">
-    <xacro:include filename="base_properties.urdf.xacro" />
+    <!-- <xacro:include filename="base_properties.urdf.xacro" /> -->
     <xacro:include filename="macros/macros.urdf.xacro" />
     <!-- Link properties -->
-    <xacro:include filename="links/foot/F_properties.urdf.xacro"/>
-    <xacro:include filename="links/hip/H_properties.urdf.xacro"/>
-    <xacro:include filename="links/lower_limb/LL_properties.urdf.xacro"/>
-    <xacro:include filename="links/upper_limb/UL_properties.urdf.xacro"/>
+    <xacro:include filename="links/properties/F_properties.urdf.xacro"/>
+    <xacro:include filename="links/properties/H_properties.urdf.xacro"/>
+    <xacro:include filename="links/properties/LL_properties.urdf.xacro"/>
+    <xacro:include filename="links/properties/UL_properties.urdf.xacro"/>
+    <!-- Joint properties -->
+    <xacro:include filename="joints/properties/T_joint_properties.urdf.xacro"/>
+    <xacro:include filename="joints/properties/H_joint_properties.urdf.xacro"/>
+    <xacro:include filename="joints/properties/K_joint_properties.urdf.xacro"/>
     <!-- LINKS -->
         <!-- Base link -->

Commit message: corrected the orientation for joint axes

File: src/meldog_description/description/joints/hip/LFH_joint.urdf.xacro (robot description, xacro)
@@ -12,5 +12,5 @@
                effort="${hip_upper_limb_effort}"
                velocity="${hip_upper_limb_velocity}" />
-        <axis xyz="0 1 0" />
+        <axis xyz="0 -1 0" />
     </joint>
 </robot>

File: src/meldog_description/description/joints/hip/LRH_joint.urdf.xacro (robot description, xacro)
@@ -12,5 +12,5 @@
                effort="${hip_upper_limb_effort}"
                velocity="${hip_upper_limb_velocity}" />
-        <axis xyz="0 1 0" />
+        <axis xyz="0 -1 0" />
     </joint>
 </robot>

File: src/meldog_description/description/joints/hip/RFH_joint.urdf.xacro (robot description, xacro)
@@ -12,5 +12,5 @@
                effort="${hip_upper_limb_effort}"
                velocity="${hip_upper_limb_velocity}" />
-        <axis xyz="0 1 0" />
+        <axis xyz="0 -1 0" />
     </joint>
 </robot>

File: src/meldog_description/description/joints/hip/RRH_joint.urdf.xacro (robot description, xacro)
@@ -12,5 +12,5 @@
                effort="${hip_upper_limb_effort}"
                velocity="${hip_upper_limb_velocity}" />
-        <axis xyz="0 1 0" />
+        <axis xyz="0 -1 0" />
     </joint>
 </robot>

File: src/meldog_description/description/joints/knee/LFK_joint.urdf.xacro (robot description, xacro)
@@ -9,5 +9,5 @@
             effort="${upper_limb_lower_limb_effort}"
             velocity="${upper_limb_lower_limb_velocity}" />
-        <axis xyz="0 1 0" />
+        <axis xyz="0 -1 0" />
     </joint>
 </robot>

File: src/meldog_description/description/joints/knee/LRK_joint.urdf.xacro (robot description, xacro)
@@ -9,5 +9,5 @@
                effort="${upper_limb_lower_limb_effort}"
                velocity="${upper_limb_lower_limb_velocity}" />
-        <axis xyz="0 1 0" />
+        <axis xyz="0 -1 0" />
     </joint>
 </robot>

File: src/meldog_description/description/joints/knee/RFK_joint.urdf.xacro (robot description, xacro)
@@ -9,5 +9,5 @@
                effort="${upper_limb_lower_limb_effort}"
                velocity="${upper_limb_lower_limb_velocity}" />
-        <axis xyz="0 1 0" />
+        <axis xyz="0 -1 0" />
     </joint>
 </robot>

File: src/meldog_description/description/joints/knee/RRK_joint.urdf.xacro (robot description, xacro)
@@ -9,5 +9,5 @@
                effort="${upper_limb_lower_limb_effort}"
                velocity="${upper_limb_lower_limb_velocity}" />
-        <axis xyz="0 1 0" />
+        <axis xyz="0 -1 0" />
     </joint>
 </robot>

Commit message: fixced joint axes orientation

File: src/meldog_description/description/joints/hip/LFH_joint.urdf.xacro (robot description, xacro)
@@ -12,5 +12,5 @@
                effort="${H_effort}"
                velocity="${H_velocity}" />
-        <axis xyz="0 1 0" />
+        <axis xyz="0 -1 0" />
     </joint>
 </robot>

File: src/meldog_description/description/joints/hip/LRH_joint.urdf.xacro (robot description, xacro)
@@ -12,5 +12,5 @@
                effort="${H_effort}"
                velocity="${H_velocity}" />
-        <axis xyz="0 1 0" />
+        <axis xyz="0 -1 0" />
     </joint>
 </robot>

File: src/meldog_description/description/joints/hip/RFH_joint.urdf.xacro (robot description, xacro)
@@ -12,5 +12,5 @@
                effort="${H_effort}"
                velocity="${H_velocity}" />
-        <axis xyz="0 1 0" />
+        <axis xyz="0 -1 0" />
     </joint>
 </robot>

File: src/meldog_description/description/joints/hip/RRH_joint.urdf.xacro (robot description, xacro)
@@ -12,5 +12,5 @@
                effort="${H_effort}"
                velocity="${H_velocity}" />
-        <axis xyz="0 1 0" />
+        <axis xyz="0 -1 0" />
     </joint>
 </robot>

File: src/meldog_description/description/joints/knee/LFK_joint.urdf.xacro (robot description, xacro)
@@ -9,5 +9,5 @@
             effort="${K_effort}"
             velocity="${K_velocity}" />
-        <axis xyz="0 1 0" />
+        <axis xyz="0 -1 0" />
     </joint>
 </robot>

File: src/meldog_description/description/joints/knee/LRK_joint.urdf.xacro (robot description, xacro)
@@ -9,5 +9,5 @@
                effort="${K_effort}"
                velocity="${K_velocity}" />
-        <axis xyz="0 1 0" />
+        <axis xyz="0 -1 0" />
     </joint>
 </robot>

File: src/meldog_description/description/joints/knee/RFK_joint.urdf.xacro (robot description, xacro)
@@ -9,5 +9,5 @@
                effort="${K_effort}"
                velocity="${K_velocity}" />
-        <axis xyz="0 1 0" />
+        <axis xyz="0 -1 0" />
     </joint>
 </robot>

File: src/meldog_description/description/joints/knee/RRK_joint.urdf.xacro (robot description, xacro)
@@ -9,5 +9,5 @@
                effort="${K_effort}"
                velocity="${K_velocity}" />
-        <axis xyz="0 1 0" />
+        <axis xyz="0 -1 0" />
     </joint>
 </robot>

Commit message: changed hip joint type to continous

File: src/meldog_description/description/joints/hip/LFH_joint.urdf.xacro (robot description, xacro)
@@ -1,5 +1,5 @@
 <?xml version="1.0"?>
 <robot xmlns:xacro="http://www.ros.org/wiki/xacro">
-    <joint name="LFH_joint" type="revolute">
+    <joint name="LFH_joint" type="continuous">
         <parent link="LFH_link" />
         <child link="LFUL_link" />
@@ -8,7 +8,5 @@
                      ${H_z}"
                 rpy="0 0 0" />
-        <limit lower="${H_lower_limit/180.0*pi}"
-               upper="${H_upper_limit/180.0*pi}"
-               effort="${H_effort}"
+        <limit effort="${H_effort}"
                velocity="${H_velocity}" />
         <axis xyz="0 -1 0" />

File: src/meldog_description/description/joints/hip/LRH_joint.urdf.xacro (robot description, xacro)
@@ -1,5 +1,5 @@
 <?xml version="1.0"?>
 <robot xmlns:xacro="http://www.ros.org/wiki/xacro">
-    <joint name="LRH_joint" type="revolute">
+    <joint name="LRH_joint" type="continuous">
         <parent link="LRH_link" />
         <child link="LRUL_link" />
@@ -8,7 +8,5 @@
                      ${H_z}"
                 rpy="0 0 0" />
-        <limit lower="${H_lower_limit/180.0*pi}"
-               upper="${H_upper_limit/180.0*pi}"
-               effort="${H_effort}"
+        <limit effort="${H_effort}"
                velocity="${H_velocity}" />
         <axis xyz="0 -1 0" />

File: src/meldog_description/description/joints/hip/RFH_joint.urdf.xacro (robot description, xacro)
@@ -1,5 +1,5 @@
 <?xml version="1.0"?>
 <robot xmlns:xacro="http://www.ros.org/wiki/xacro">
-    <joint name="RFH_joint" type="revolute">
+    <joint name="RFH_joint" type="continuous">
         <parent link="RFH_link" />
         <child link="RFUL_link" />
@@ -8,7 +8,5 @@
                      ${H_z}"
                 rpy="0 0 0" />
-        <limit lower="${H_lower_limit/180.0*pi}"
-               upper="${H_upper_limit/180.0*pi}"
-               effort="${H_effort}"
+        <limit effort="${H_effort}"
                velocity="${H_velocity}" />
         <axis xyz="0 -1 0" />

File: src/meldog_description/description/joints/hip/RRH_joint.urdf.xacro (robot description, xacro)
@@ -1,5 +1,5 @@
 <?xml version="1.0"?>
 <robot xmlns:xacro="http://www.ros.org/wiki/xacro">
-    <joint name="RRH_joint" type="revolute">
+    <joint name="RRH_joint" type="continuous">
         <parent link="RRH_link" />
         <child link="RRUL_link" />
@@ -8,7 +8,5 @@
                      ${H_z}"
                 rpy="0 0 0" />
-        <limit lower="${H_lower_limit/180.0*pi}"
-               upper="${H_upper_limit/180.0*pi}"
-               effort="${H_effort}"
+        <limit effort="${H_effort}"
                velocity="${H_velocity}" />
         <axis xyz="0 -1 0" />

File: src/meldog_description/description/ros2_control/meldog_gazebo_ros2_control.urdf.xacro (robot description, xacro)
@@ -44,12 +44,3 @@
         </plugin>
       </gazebo>
-    <!-- <gazebo>
-        <plugin filename="ign_ros2_control-system" name="ign_ros2_control::IgnitionROS2ControlPlugin">
-            <robot_param>robot_description</robot_param>
-            <robot_param_node>robot_state_publisher</robot_param_node>
-            <parameters>$(find meldog_description)/controllers/meldog_controllers.yaml</parameters>
-            <hold_joints>true</hold_joints>
-            <controller_manager_name>controller_manager</controller_manager_name>
-        </plugin>
-    </gazebo> -->
 </robot>
