Commit message: added missing dynamics tags in joints

File: src/meldog_description/description/joints/hip/LFH_joint.urdf.xacro (robot description, xacro)
@@ -9,4 +9,5 @@
         <limit lower="${H_lower_limit}" upper="${H_upper_limit}"
                effort="${H_effort}" velocity="${H_velocity}" />
+        <dynamics friction="${H_friction}" damping="${H_damping}" />
         <axis xyz="0 -1 0" />
     </joint>

File: src/meldog_description/description/joints/hip/LRH_joint.urdf.xacro (robot description, xacro)
@@ -10,4 +10,5 @@
         <limit lower="${H_lower_limit}" upper="${H_upper_limit}"
                effort="${H_effort}" velocity="${H_velocity}" />
+        <dynamics friction="${H_friction}" damping="${H_damping}" />
         <axis xyz="0 -1 0" />
     </joint>

File: src/meldog_description/description/joints/hip/RFH_joint.urdf.xacro (robot description, xacro)
@@ -10,4 +10,5 @@
         <limit lower="${H_lower_limit}" upper="${H_upper_limit}"
                effort="${H_effort}" velocity="${H_velocity}" />
+        <dynamics friction="${H_friction}" damping="${H_damping}" />
         <axis xyz="0 -1 0" />
     </joint>

File: src/meldog_description/description/joints/hip/RRH_joint.urdf.xacro (robot description, xacro)
@@ -10,4 +10,5 @@
         <limit lower="${H_lower_limit}" upper="${H_upper_limit}"
                effort="${H_effort}" velocity="${H_velocity}" />
+        <dynamics friction="${H_friction}" damping="${H_damping}" />
         <axis xyz="0 -1 0" />
     </joint>

File: src/meldog_description/description/joints/knee/LFK_joint.urdf.xacro (robot description, xacro)
@@ -9,4 +9,5 @@
             effort="${K_effort}"
             velocity="${K_velocity}" />
+        <dynamics friction="${K_friction}" damping="${K_damping}" />
         <axis xyz="0 -1 0" />
     </joint>

File: src/meldog_description/description/joints/knee/LRK_joint.urdf.xacro (robot description, xacro)
@@ -9,4 +9,5 @@
                effort="${K_effort}"
                velocity="${K_velocity}" />
+        <dynamics friction="${K_friction}" damping="${K_damping}" />
         <axis xyz="0 -1 0" />
     </joint>

File: src/meldog_description/description/joints/knee/RFK_joint.urdf.xacro (robot description, xacro)
@@ -9,4 +9,5 @@
                effort="${K_effort}"
                velocity="${K_velocity}" />
+        <dynamics friction="${K_friction}" damping="${K_damping}" />
         <axis xyz="0 -1 0" />
     </joint>

File: src/meldog_description/description/joints/knee/RRK_joint.urdf.xacro (robot description, xacro)
@@ -9,4 +9,5 @@
                effort="${K_effort}"
                velocity="${K_velocity}" />
+        <dynamics friction="${K_friction}" damping="${K_damping}" />
         <axis xyz="0 -1 0" />
     </joint>

File: src/meldog_description/description/joints/properties/H_joint_properties.urdf.xacro (robot description, xacro)
@@ -13,4 +13,4 @@
     <!-- Hip joint friction and damping -->
     <xacro:property name="H_damping" value="0"/>
-    <xacro:property name="H_friction" value="0"/>
+    <xacro:property name="H_friction" value="0.0312"/>
 </robot>

File: src/meldog_description/description/joints/properties/K_joint_properties.urdf.xacro (robot description, xacro)
@@ -9,4 +9,4 @@
     <!-- Knee joint friction and damping -->
     <xacro:property name="K_damping" value="0"/>
-    <xacro:property name="K_friction" value="0"/>
+    <xacro:property name="K_friction" value="0.0312"/>
 </robot>

File: src/meldog_description/description/joints/properties/T_joint_properties.urdf.xacro (robot description, xacro)
@@ -9,4 +9,4 @@
     <!-- Trunk joint friction and damping -->
     <xacro:property name="T_damping" value="0"/>
-    <xacro:property name="T_friction" value="0"/>
+    <xacro:property name="T_friction" value="0.0312"/>
 </robot>

File: src/meldog_description/description/joints/trunk/LFT_joint.urdf.xacro (robot description, xacro)
@@ -9,4 +9,5 @@
                effort="${T_effort}"
                velocity="${T_velocity}" />
+        <dynamics friction="${T_friction}" damping="${T_damping}" />
         <axis xyz="1 0 0" />
     </joint>

File: src/meldog_description/description/joints/trunk/LRT_joint.urdf.xacro (robot description, xacro)
@@ -9,4 +9,5 @@
                effort="${T_effort}"
                velocity="${T_velocity}" />
+        <dynamics friction="${T_friction}" damping="${T_damping}" />
         <axis xyz="1 0 0" />
     </joint>

File: src/meldog_description/description/joints/trunk/RFT_joint.urdf.xacro (robot description, xacro)
@@ -9,4 +9,5 @@
                effort="${T_effort}"
                velocity="${T_velocity}" />
+        <dynamics friction="${T_friction}" damping="${T_damping}" />
         <axis xyz="-1 0 0" />
     </joint>

File: src/meldog_description/description/joints/trunk/RRT_joint.urdf.xacro (robot description, xacro)
@@ -9,4 +9,5 @@
                effort="${T_effort}"
                velocity="${T_velocity}" />
+        <dynamics friction="${T_friction}" damping="${T_damping}" />
         <axis xyz="-1 0 0" />
     </joint>
