Commit message: Added back joint controller

File: meldog_description/description/gazebo/imu_gazebo_setup.urdf.xacro (robot description, xacro)
@@ -13,8 +13,4 @@
   <gazebo reference="imu_link">
     <sensor name="imu_sensor" type="imu">
-      <plugin filename="libignition-gazebo-imu-system.so"
-              name="ignition::gazebo::systems::Imu">
-        <initial_orientation_as_reference>false</initial_orientation_as_reference>
-      </plugin>
       <always_on>true</always_on>
       <update_rate>1000</update_rate>  <!-- since controller manager runs on 1000Hz, the same goes with IMU-->

File: meldog_description/description/ros2_control/meldog_gazebo_ros2_control.urdf.xacro (robot description, xacro)
@@ -61,5 +61,5 @@
           <robot_param>robot_description</robot_param>
           <robot_param_node>robot_state_publisher</robot_param_node>
-          <parameters>$(find meldog_description)/controllers/meldog_controllers.yaml</parameters>
+          <parameters>$(find meldog_description)/controllers/meldog_joint_controllers.yaml</parameters>
           <hold_joints>true</hold_joints>
         </plugin>

File: meldog_description/description/ros2_control/ros2_control_macros.urdf.xacro (robot description, xacro)
@@ -2,22 +2,13 @@
 <robot xmlns:xacro="http://www.ros.org/wiki/xacro">
     <xacro:macro name="ros2_control_joint_macro" params="name pos_min pos_max vel_max eff_max">
-        <joint name="${name}_joint">
-          <!-- co jesli joint continuous? -->
-            <command_interface name="position">
-              <param name="min">${pos_min}</param>
-              <param name="max">${pos_max}</param>
-            </command_interface>
-            <!-- <command_interface name="velocity" >
-              <param name="min">${-vel_max}</param>
-              <param name="max">${vel_max}</param>
-            </command_interface>
-            <command_interface name="effort">
-              <param name="min">${-eff_max}</param>
-              <param name="max">${eff_max}</param>
-            </command_interface> -->
-            <state_interface name="position" />
-            <state_interface name="velocity"/>
-            <state_interface name="effort"/>
-          </joint>
+      <joint name="${name}_joint">
+        <command_interface name="effort">
+          <param name="min">${-eff_max}</param>
+          <param name="max">${eff_max}</param>
+        </command_interface>
+        <state_interface name="position"/>
+        <state_interface name="velocity"/>
+         <state_interface name="effort"/>
+      </joint>
     </xacro:macro>
     <xacro:macro name="simple_transmission" params="joint reduction offset">
