Commit message: Added gazebo changes

File: meldog_description/description/gazebo/gazebo_properties.urdf.xacro (robot description, xacro)
@@ -9,5 +9,5 @@
     <xacro:property name="springStiffness_value" value="0" />
     <xacro:property name="springReference_value" value="0" />
-    <xacro:property name="implicitSpringDamper_value" value="0" />
+    <!-- <xacro:property name="implicitSpringDamper_value" value="0" /> -->
     <xacro:property name="stopErp_value" value="0" />
     <xacro:property name="stopCfm_value" value="0" />
@@ -20,10 +20,21 @@
     <xacro:property name="dampingFactor_value" value="0" />
     <!-- Gazebo link parameters for feet -->
-    <xacro:property name="mu1_value_foot" value="0" />
-    <xacro:property name="mu2_value_foot" value="0" />
-    <xacro:property name="kp_value_foot" value="0" />
-    <xacro:property name="kd_value_foot" value="0" />
-    <xacro:property name="maxVel_value_foot" value="0" />
-    <xacro:property name="dampingFactor_value_foot" value="0" />
+    <xacro:property name="mu1_value_foot" value="1.0" />
+    <xacro:property name="mu2_value_foot" value="1.0" />
+    <xacro:property name="kp_value_foot" value="100000.0" />
+    <xacro:property name="kd_value_foot" value="5000.0" />
+    <xacro:property name="maxVel_value_foot" value="0.01" />
+    <xacro:property name="minDepth_value_foot" value="0.001" />
+    <xacro:property name="dampingFactor_value_foot" value="0.25" />
+    <!-- <xacro:property name="mu1_value_foot" value="2.0" />
+    <xacro:property name="mu2_value_foot" value="2.0" />
+    <xacro:property name="kp_value_foot" value="1000000.0" />
+    <xacro:property name="kd_value_foot" value="1000.0" />
+    <xacro:property name="maxVel_value_foot" value="0.0" />
+    <xacro:property name="dampingFactor_value_foot" value="0.1" /> -->
+    <!-- <xacro:property name="kp_value_foot" value="10000.0"/>
+    <xacro:property name="kd_value_foot" value="10000.0"/>
+    <xacro:property name="maxVel_value_foot" value="0.0"/>
+    <xacro:property name="dampingFactor_value_foot" value="10.1"/> -->
     <!--      GAZEBO IMU NOICE PARAMETERS      -->
         <!-- Angular velocity noise parameters -->

File: meldog_description/description/gazebo/meldog_gazebo.urdf.xacro (robot description, xacro)
@@ -14,4 +14,5 @@
             <maxVel value="${maxVel}"/>
             <dampingFactor value="${dampingFactor}"/>
+            <minDepth value="0.0002"/>
         </gazebo>
     </xacro:macro>

File: meldog_description/description/joints/properties/H_joint_properties.urdf.xacro (robot description, xacro)
@@ -12,5 +12,5 @@
     <xacro:property name="H_velocity" value="${motor_max_vel*pi/30.0/actuator_reduction}" />
     <!-- Hip joint friction and damping -->
-    <xacro:property name="H_damping" value="0"/>
-    <xacro:property name="H_friction" value="0.0312"/>
+    <xacro:property name="H_damping" value="0.2"/>
+    <xacro:property name="H_friction" value="0.1312"/>
 </robot>

File: meldog_description/description/joints/properties/K_joint_properties.urdf.xacro (robot description, xacro)
@@ -8,5 +8,5 @@
     <xacro:property name="K_velocity" value="${motor_max_vel*pi/30.0/actuator_reduction}" />
     <!-- Knee joint friction and damping -->
-    <xacro:property name="K_damping" value="0"/>
-    <xacro:property name="K_friction" value="0.0312"/>
+    <xacro:property name="K_damping" value="0.2"/>
+    <xacro:property name="K_friction" value="0.1312"/>
 </robot>

File: meldog_description/description/joints/properties/T_joint_properties.urdf.xacro (robot description, xacro)
@@ -8,5 +8,5 @@
     <xacro:property name="T_velocity" value="${motor_max_vel*pi/30.0/actuator_reduction}" />
     <!-- Trunk joint friction and damping -->
-    <xacro:property name="T_damping" value="0"/>
-    <xacro:property name="T_friction" value="0.0312"/>
+    <xacro:property name="T_damping" value="0.2"/>
+    <xacro:property name="T_friction" value="0.1312"/>
 </robot>

File: meldog_description/description/meldog_core.urdf.xacro (robot description, xacro)
@@ -20,6 +20,6 @@
     <xacro:include filename="ros2_control/meldog_gazebo_ros2_control.urdf.xacro"/>
     <!-- LINKS -->
-        <!-- Base link -->
-        <link name="base_link" />
+        <!-- Base link
+        <link name="base_link" /> -->
         <!-- Trunk link -->
         <xacro:include filename="links/trunk.urdf.xacro" />
@@ -63,9 +63,9 @@
             <xacro:include filename="links/foot/RRF_link.urdf.xacro"/>
     <!-- JOINTS -->
-        <joint name="base_joint" type="fixed">
+        <!-- <joint name="base_joint" type="fixed">
             <parent link="base_link" />
             <child link="trunk_link" />
             <origin xyz="0 0 0.55" rpy="0 0 0" />
-        </joint>
+        </joint> -->
         <!-- IMU joint -->
         <xacro:include filename="joints/sensors/imu_joint.urdf.xacro"/>

File: meldog_description/description/meldog_real.urdf.xacro (robot description, xacro)
@@ -15,6 +15,6 @@
     <xacro:include filename="ros2_control/meldog_real_ros2_control.urdf.xacro"/>
     <!-- LINKS -->
-        <!-- Base link -->
-        <link name="base_link" />
+        <!-- Base link
+        <link name="base_link" /> -->
         <!-- Trunk link -->
         <xacro:include filename="links/trunk.urdf.xacro" />
@@ -58,9 +58,9 @@
             <xacro:include filename="links/foot/RRF_link.urdf.xacro"/>
     <!-- JOINTS -->
-        <joint name="base_joint" type="fixed">
+        <!-- <joint name="base_joint" type="fixed">
             <parent link="base_link" />
             <child link="trunk_link" />
             <origin xyz="0 0 0.55" rpy="0 0 0" />
-        </joint>
+        </joint> -->
         <!-- IMU joint -->
         <xacro:include filename="joints/sensors/imu_joint.urdf.xacro"/>

File: meldog_description/description/ros2_control/hardware_properties.urdf.xacro (robot description, xacro)
@@ -1,5 +1,5 @@
 <?xml version="1.0"?>
 <robot xmlns:xacro="http://www.ros.org/wiki/xacro">
-    <xacro:property name="motor_max_eff" value="3.5" />
+    <xacro:property name="motor_max_eff" value="2.0" />
     <xacro:property name="motor_max_vel" value="1800" />
     <xacro:property name="actuator_reduction" value="9.97" />

File: meldog_description/description/ros2_control/meldog_gazebo_ros2_control.urdf.xacro (robot description, xacro)
@@ -57,4 +57,13 @@
     </ros2_control>
     <gazebo>
+      <plugin
+          filename="libBaseTransformTwistPublisher.so"
+          name="gazebo_plugins::BaseTransformTwistPublisher">
+        <base_frame_name>trunk_link</base_frame_name>
+        <reference_frame_name>world</reference_frame_name>
+        <max_publish_frequency>200</max_publish_frequency>
+      </plugin>
+    </gazebo>
+    <gazebo>
         <plugin filename="gz_ros2_control-system"
           name="gz_ros2_control::GazeboSimROS2ControlPlugin">
