Commit message: Deleted sensors links and joints

File: meldog_description/description/meldog_core.urdf.xacro (robot description, xacro)
@@ -8,5 +8,4 @@
     <xacro:include filename="links/properties/LL_properties.urdf.xacro"/>
     <xacro:include filename="links/properties/UL_properties.urdf.xacro"/>
-    <xacro:include filename="links/properties/S_properties.urdf.xacro"/>
     <!-- Joint properties -->
     <xacro:include filename="joints/properties/T_joint_properties.urdf.xacro"/>
@@ -18,4 +17,6 @@
     <!-- IMU gazebo setup -->
     <xacro:include filename="gazebo/imu_gazebo_setup.urdf.xacro"/>
+    <!-- Contact sensors setup -->
+    <xacro:include filename="gazebo/contact_gazebo_setup.urdf.xacro"/>
     <!-- ROS2 Control -->
     <xacro:include filename="ros2_control/meldog_gazebo_ros2_control.urdf.xacro"/>
@@ -36,6 +37,4 @@
             <!-- Left front foot link -->
             <xacro:include filename="links/foot/LFF_link.urdf.xacro"/>
-            <!-- Left front sensor link -->
-            <xacro:include filename="links/sensors/LFS_link.urdf.xacro"/>
         <!-- Right front leg links -->
             <!-- Right front hip link -->
@@ -47,6 +46,4 @@
             <!-- Right front foot link -->
             <xacro:include filename="links/foot/RFF_link.urdf.xacro"/>
-            <!-- Right front sensor link -->
-            <xacro:include filename="links/sensors/RFS_link.urdf.xacro"/>
         <!-- Left rear leg links -->
             <!-- Left rear hip link -->
@@ -58,6 +55,4 @@
             <!-- Left rear foot link -->
             <xacro:include filename="links/foot/LRF_link.urdf.xacro"/>
-            <!-- Left rear sensor link -->
-            <xacro:include filename="links/sensors/LRS_link.urdf.xacro"/>
         <!-- Right rear leg links -->
             <!-- Right rear hip link -->
@@ -69,11 +64,9 @@
             <!-- Right rear foot link -->
             <xacro:include filename="links/foot/RRF_link.urdf.xacro"/>
-            <!-- Right rear sensor link -->
-            <xacro:include filename="links/sensors/RRS_link.urdf.xacro"/>
     <!-- JOINTS -->
         <joint name="base_joint" type="fixed">
             <parent link="base_link" />
             <child link="trunk_link" />
-            <origin xyz="0 0 0.55" rpy="0 0 0" />
+            <origin xyz="0 0 500.55" rpy="0 0 0" />
         </joint>
         <!-- IMU joint -->
@@ -88,6 +81,4 @@
             <!-- Left front foot joint -->
             <xacro:include filename="joints/foot/LFF_joint.urdf.xacro"/>
-            <!-- Left front sensor joint -->
-            <xacro:include filename="joints/sensors/LFS_joint.urdf.xacro"/>
         <!-- Right front leg joints -->
             <!-- Right front trunk joint -->
@@ -99,6 +90,4 @@
             <!-- Right front foot joint -->
             <xacro:include filename="joints/foot/RFF_joint.urdf.xacro"/>
-            <!-- Right front sensor joint -->
-            <xacro:include filename="joints/sensors/RFS_joint.urdf.xacro"/>
         <!-- Left rear leg joints -->
             <!-- Left rear trunk joint -->
@@ -110,6 +99,4 @@
             <!-- Left rear foot joint -->
             <xacro:include filename="joints/foot/LRF_joint.urdf.xacro"/>
-            <!-- Left rear sensor joint -->
-            <xacro:include filename="joints/sensors/LRS_joint.urdf.xacro"/>
         <!-- Right rear leg joints -->
             <!-- Right rear trunk joint -->
@@ -121,5 +108,3 @@
             <!-- Right rear foot joint -->
             <xacro:include filename="joints/foot/RRF_joint.urdf.xacro"/>
-            <!-- Right rear sensor joint -->
-            <xacro:include filename="joints/sensors/RRS_joint.urdf.xacro"/>
 </robot>

Commit message: Reverted origin of robot

File: meldog_description/description/meldog_core.urdf.xacro (robot description, xacro)
@@ -68,5 +68,5 @@
             <parent link="base_link" />
             <child link="trunk_link" />
-            <origin xyz="0 0 500.55" rpy="0 0 0" />
+            <origin xyz="0 0 0.55" rpy="0 0 0" />
         </joint>
         <!-- IMU joint -->
