Commit message: adapt model to CAD  geometry

File: meldog_description/description/joints/trunk/LFT_joint.urdf.xacro (robot description, xacro)
@@ -4,5 +4,6 @@
         <parent link="trunk_link" />
         <child link="LFH_link" />
-        <origin xyz="${trunk_actuators_length/2.0} ${(trunk_base_width+trunk_actuators_width)/2.0} 0" rpy="0 0 0" />
+        <!-- ADD LEG PLACEMENT AS PARAMETERS-->
+        <origin xyz="0.084 0.1101 0" rpy="0 0 0" />
         <limit lower="${T_lower_limit/180.0*pi}"
                upper="${T_upper_limit/180.0*pi}"

File: meldog_description/description/joints/trunk/LRT_joint.urdf.xacro (robot description, xacro)
@@ -4,5 +4,6 @@
         <parent link="trunk_link" />
         <child link="LRH_link" />
-        <origin xyz="${-trunk_actuators_length/2.0} ${(trunk_base_width+trunk_actuators_width)/2.0} 0" rpy="0 0 0" />
+        <!-- ADD LEG PLACEMENT AS PARAMETERS-->
+        <origin xyz="-0.084 0.1101 0" rpy="0 0 0" />
         <limit lower="${T_lower_limit/180.0*pi}"
                upper="${T_upper_limit/180.0*pi}"

File: meldog_description/description/joints/trunk/RFT_joint.urdf.xacro (robot description, xacro)
@@ -4,5 +4,6 @@
         <parent link="trunk_link" />
         <child link="RFH_link" />
-        <origin xyz="${trunk_actuators_length/2.0} ${-(trunk_base_width+trunk_actuators_width)/2.0} 0" rpy="0 0 0" />
+        <!-- ADD LEG PLACEMENT AS PARAMETERS-->
+        <origin xyz="0.084 -0.1101 0" rpy="0 0 0" />
         <limit lower="${T_lower_limit/180.0*pi}"
                upper="${T_upper_limit/180.0*pi}"

File: meldog_description/description/joints/trunk/RRT_joint.urdf.xacro (robot description, xacro)
@@ -4,5 +4,6 @@
         <parent link="trunk_link" />
         <child link="RRH_link" />
-        <origin xyz="${-trunk_actuators_length/2.0} ${-(trunk_base_width+trunk_actuators_width)/2.0} 0" rpy="0 0 0" />
+        <!-- ADD LEG PLACEMENT AS PARAMETERS-->
+        <origin xyz="-0.084 -0.1101 0" rpy="0 0 0" />
         <limit lower="${T_lower_limit/180.0*pi}"
                upper="${T_upper_limit/180.0*pi}"

File: meldog_description/description/links/trunk.urdf.xacro (robot description, xacro)
@@ -7,13 +7,16 @@
 <xacro:property name="trunk_actuators_width" value="0.15" />
 <xacro:property name="trunk_actuators_height" value="0.1" />
-<xacro:property name="trunk_mass" value="8.0"/>
+<xacro:property name="trunk_mass" value="10.0"/>
 <link name="trunk_link">
         <inertial>
-            <origin xyz="0.0 0.0 0.0" rpy="0.0 0.0 0.0"/>
+        <!--ADD PARAMETRIZATION TRUNK FIX
+            current CAD model is broken, STL center is shifted relative to geometric center by 19,774mm
+         -->
+            <origin xyz="0.019774 0.0 0.0" rpy="0.0 0.0 0.0"/>
             <mass value="${trunk_mass}"/>
             <inertia ixx="${1/12*trunk_mass*(trunk_base_width*trunk_base_width + trunk_base_height*trunk_base_height)}" ixy="0.0" ixz="0.0" iyy="${1/12*trunk_mass*(trunk_base_length*trunk_base_length + trunk_base_height*trunk_base_height)}" iyz=".0" izz="${1/12*trunk_mass*(trunk_base_length*trunk_base_length + trunk_base_width*trunk_base_width)}"/>
         </inertial>
         <visual>
-            <origin xyz="0 0 0" rpy="${pi/2} 0 ${pi/2}"/>
+            <origin xyz="0.019774 0 0" rpy="${pi/2} 0 ${pi/2}"/>
             <geometry>
                 <mesh filename="package://meldog_description/meshes/visual/trunk.stl"
@@ -22,5 +25,5 @@
         </visual>
         <collision>
-            <origin xyz="0 0 0" rpy="0 0 0"/>
+            <origin xyz="0.019774 0 0" rpy="${pi/2} 0 ${pi/2}"/>
             <geometry>
                 <mesh filename="package://meldog_description/meshes/collision/trunk_collision.stl"
