Commit message: fix joint limits

File: meldog_description/description/joints/hip/LFH_joint.urdf.xacro (robot description, xacro)
@@ -6,6 +6,7 @@
         <origin xyz="${H_x}
                      ${H_y}
-                     ${H_z}" rpy="0 0 0" />
-        <limit lower="${H_lower_limit}" upper="${H_upper_limit}"
+                     ${H_z}"
+                rpy="0 0 0" />
+        <limit lower="${H_lower_limit/180.0*pi}" upper="${H_upper_limit/180.0*pi}"
                effort="${H_effort}" velocity="${H_velocity}" />
         <dynamics friction="${H_friction}" damping="${H_damping}" />

File: meldog_description/description/joints/properties/H_joint_properties.urdf.xacro (robot description, xacro)
@@ -6,6 +6,6 @@
     <xacro:property name="H_z" value="0"/>
     <!-- Hip upper limb joint movement limits -->
-    <xacro:property name="H_lower_limit" value="-120" />
-    <xacro:property name="H_upper_limit" value="120" />
+    <xacro:property name="H_lower_limit" value="-360" /> <!-- degrees-->
+    <xacro:property name="H_upper_limit" value="360" /> <!-- degrees-->
     <!-- Hip joint effort and velocity limits -->
     <xacro:property name="H_effort" value="${motor_max_eff*actuator_reduction}" />

File: meldog_description/description/joints/properties/K_joint_properties.urdf.xacro (robot description, xacro)
@@ -2,6 +2,6 @@
 <robot xmlns:xacro="http://www.ros.org/wiki/xacro">
     <!-- Knee joint movement limits -->
-    <xacro:property name="K_lower_limit" value="-160" />
-    <xacro:property name="K_upper_limit" value="160" />
+    <xacro:property name="K_lower_limit" value="-160" /> <!-- degrees-->
+    <xacro:property name="K_upper_limit" value="160" /> <!-- degrees-->
     <!-- Knee joint effort and velocity limits -->
     <xacro:property name="K_effort" value="${motor_max_eff*actuator_reduction}" />

File: meldog_description/description/joints/properties/T_joint_properties.urdf.xacro (robot description, xacro)
@@ -2,6 +2,6 @@
 <robot xmlns:xacro="http://www.ros.org/wiki/xacro">
     <!-- Trunk joint movement limits -->
-    <xacro:property name="T_lower_limit" value="-45" />
-    <xacro:property name="T_upper_limit" value="45" />
+    <xacro:property name="T_lower_limit" value="-60" /> <!-- degrees-->
+    <xacro:property name="T_upper_limit" value="60" /> <!-- degrees-->
     <!-- Trunk joint effort and velocity limits -->
     <xacro:property name="T_effort" value="${motor_max_eff*actuator_reduction}" />
