Commit message: fix trunk parametrization

File: meldog_description/description/joints/properties/H_joint_properties.urdf.xacro (robot description, xacro)
@@ -2,7 +2,7 @@
 <robot xmlns:xacro="http://www.ros.org/wiki/xacro">
     <!-- Hip joint origin -->
-    <xacro:property name="H_x" value="0.174"/>
-    <xacro:property name="H_y" value="0.0925"/>
-    <xacro:property name="H_z" value="0"/>
+    <xacro:property name="H_x" value="0.174"/> <!--meters-->
+    <xacro:property name="H_y" value="0.0925"/> <!--meters-->
+    <xacro:property name="H_z" value="0"/> <!--meters-->
     <!-- Hip upper limb joint movement limits -->
     <xacro:property name="H_lower_limit" value="-360" /> <!-- degrees-->

File: meldog_description/description/joints/properties/T_joint_properties.urdf.xacro (robot description, xacro)
@@ -1,4 +1,8 @@
 <?xml version="1.0"?>
 <robot xmlns:xacro="http://www.ros.org/wiki/xacro">
+    <!-- Trunk joint origin -->
+    <xacro:property name="T_x" value="0.084" /> <!--meters-->
+    <xacro:property name="T_y" value="0.1101"/> <!--meters-->
+    <xacro:property name="T_z" value="0"/> <!--meters-->
     <!-- Trunk joint movement limits -->
     <xacro:property name="T_lower_limit" value="-60" /> <!-- degrees-->

File: meldog_description/description/joints/trunk/LFT_joint.urdf.xacro (robot description, xacro)
@@ -5,5 +5,8 @@
         <child link="LFH_link" />
         <!-- ADD LEG PLACEMENT AS PARAMETERS-->
-        <origin xyz="0.084 0.1101 0" rpy="0 0 0" />
+                <origin xyz="${T_x}
+                        ${T_y}
+                        ${T_z}"
+                    rpy="0 0 0" />
         <limit lower="${T_lower_limit/180.0*pi}"
                upper="${T_upper_limit/180.0*pi}"

File: meldog_description/description/joints/trunk/LRT_joint.urdf.xacro (robot description, xacro)
@@ -5,5 +5,8 @@
         <child link="LRH_link" />
         <!-- ADD LEG PLACEMENT AS PARAMETERS-->
-        <origin xyz="-0.084 0.1101 0" rpy="0 0 0" />
+                <origin xyz="${-T_x}
+                        ${T_y}
+                        ${T_z}"
+                    rpy="0 0 0" />
         <limit lower="${T_lower_limit/180.0*pi}"
                upper="${T_upper_limit/180.0*pi}"

File: meldog_description/description/joints/trunk/RFT_joint.urdf.xacro (robot description, xacro)
@@ -5,5 +5,8 @@
         <child link="RFH_link" />
         <!-- ADD LEG PLACEMENT AS PARAMETERS-->
-        <origin xyz="0.084 -0.1101 0" rpy="0 0 0" />
+                <origin xyz="${T_x}
+                        ${-T_y}
+                        ${T_z}"
+                    rpy="0 0 0" />
         <limit lower="${T_lower_limit/180.0*pi}"
                upper="${T_upper_limit/180.0*pi}"

File: meldog_description/description/joints/trunk/RRT_joint.urdf.xacro (robot description, xacro)
@@ -5,5 +5,8 @@
         <child link="RRH_link" />
         <!-- ADD LEG PLACEMENT AS PARAMETERS-->
-        <origin xyz="-0.084 -0.1101 0" rpy="0 0 0" />
+                <origin xyz="${-T_x}
+                        ${-T_y}
+                        ${T_z}"
+                    rpy="0 0 0" />
         <limit lower="${T_lower_limit/180.0*pi}"
                upper="${T_upper_limit/180.0*pi}"
