Commit message: Dodano nowe parametry symulacji i controller'y

File: meldog_description/description/joints/properties/H_joint_properties.urdf.xacro (robot description, xacro)
@@ -12,5 +12,5 @@
     <xacro:property name="H_velocity" value="${motor_max_vel*pi/30.0/actuator_reduction}" />
     <!-- Hip joint friction and damping -->
-    <xacro:property name="H_damping" value="0"/>
-    <xacro:property name="H_friction" value="0.0312"/>
+    <xacro:property name="H_damping" value="0.05"/>
+    <xacro:property name="H_friction" value="0.1312"/>
 </robot>

File: meldog_description/description/joints/properties/K_joint_properties.urdf.xacro (robot description, xacro)
@@ -10,5 +10,5 @@
     <xacro:property name="K_velocity" value="${motor_max_vel*pi/30.0/actuator_reduction}" />
     <!-- Knee joint friction and damping -->
-    <xacro:property name="K_damping" value="0"/>
-    <xacro:property name="K_friction" value="0.0312"/>
+    <xacro:property name="K_damping" value="0.05"/>
+    <xacro:property name="K_friction" value="0.1312"/>
 </robot>

File: meldog_description/description/joints/properties/T_joint_properties.urdf.xacro (robot description, xacro)
@@ -12,5 +12,5 @@
     <xacro:property name="T_velocity" value="${motor_max_vel*pi/30.0/actuator_reduction}" />
     <!-- Trunk joint friction and damping -->
-    <xacro:property name="T_damping" value="0"/>
-    <xacro:property name="T_friction" value="0.0312"/>
+    <xacro:property name="T_damping" value="0.05"/>
+    <xacro:property name="T_friction" value="0.1312"/>
 </robot>

File: meldog_description/description/meldog_core.urdf.xacro (robot description, xacro)
@@ -23,6 +23,4 @@
     <xacro:include filename="ros2_control/meldog_gazebo_ros2_control.urdf.xacro"/>
     <!-- LINKS -->
-        <!-- Base link -->
-        <link name="base_link" />
         <!-- Trunk link -->
         <xacro:include filename="links/trunk.urdf.xacro" />
@@ -66,9 +64,4 @@
             <xacro:include filename="links/foot/RRF_link.urdf.xacro"/>
     <!-- JOINTS -->
-        <joint name="base_joint" type="fixed">
-            <parent link="base_link" />
-            <child link="trunk_link" />
-            <origin xyz="0 0 0.55" rpy="0 0 0" />
-        </joint>
         <!-- IMU joint -->
         <xacro:include filename="joints/sensors/imu_joint.urdf.xacro"/>
