Commit message: fix naming, add initial mesh loading

File: meldog_description/description/links/trunk.urdf.xacro (robot description, xacro)
@@ -1,5 +1,34 @@
 <?xml version="1.0"?>
 <robot xmlns:xacro="http://www.ros.org/wiki/xacro">
+<xacro:property name="trunk_base_length" value="0.8" />
+<xacro:property name="trunk_base_width" value="0.2" />
+<xacro:property name="trunk_base_height" value="0.1" />
+<xacro:property name="trunk_actuators_length" value="0.3" />
+<xacro:property name="trunk_actuators_width" value="0.15" />
+<xacro:property name="trunk_actuators_height" value="0.1" />
+<xacro:property name="trunk_mass" value="8.0"/>
+<link name="trunk_link">
+        <inertial>
+            <origin xyz="0.0 0.0 0.0" rpy="0.0 0.0 0.0"/>
+            <mass value="${trunk_mass}"/>
+            <inertia ixx="${1/12*trunk_mass*(trunk_base_width*trunk_base_width + trunk_base_height*trunk_base_height)}" ixy="0.0" ixz="0.0" iyy="${1/12*trunk_mass*(trunk_base_length*trunk_base_length + trunk_base_height*trunk_base_height)}" iyz=".0" izz="${1/12*trunk_mass*(trunk_base_length*trunk_base_length + trunk_base_width*trunk_base_width)}"/>
+        </inertial>
+        <visual>
+            <origin xyz="0 0 0" rpy="${pi/2} 0 ${pi/2}"/>
+            <geometry>
+                <mesh filename="package://meldog_description/meshes/visual/trunk.stl"
+                      scale="0.001 0.001 0.001" />
+                </geometry>
+        </visual>
+        <collision>
+            <origin xyz="0 0 0" rpy="0 0 0"/>
+            <geometry>
+                <mesh filename="package://meldog_description/meshes/collision/trunk_collision.stl"
+                      scale="0.001 0.001 0.001" />
+                </geometry>
+        </collision>
+    </link>
     <!-- Meldog trunk (3 simple boxes) -->
+    <!--
     <xacro:property name="trunk_base_length" value="0.8" />
     <xacro:property name="trunk_base_width" value="0.2" />
@@ -52,3 +81,4 @@
         </collision>
     </link>
+    -->
 </robot>

Commit message: improve link macro

File: meldog_description/description/links/trunk.urdf.xacro (robot description, xacro)
@@ -4,84 +4,21 @@
 <xacro:property name="trunk_base_width" value="0.2" />
 <xacro:property name="trunk_base_height" value="0.1" />
-<xacro:property name="trunk_actuators_length" value="0.3" />
-<xacro:property name="trunk_actuators_width" value="0.15" />
-<xacro:property name="trunk_actuators_height" value="0.1" />
-<xacro:property name="trunk_mass" value="10.0"/>
-<link name="trunk_link">
-        <inertial>
-        <!--ADD PARAMETRIZATION TRUNK FIX
-            current CAD model is broken, STL center is shifted relative to geometric center by 19,774mm
-         -->
-            <origin xyz="0.019774 0.0 0.0" rpy="0.0 0.0 0.0"/>
-            <mass value="${trunk_mass}"/>
-            <inertia ixx="${1/12*trunk_mass*(trunk_base_width*trunk_base_width + trunk_base_height*trunk_base_height)}" ixy="0.0" ixz="0.0" iyy="${1/12*trunk_mass*(trunk_base_length*trunk_base_length + trunk_base_height*trunk_base_height)}" iyz=".0" izz="${1/12*trunk_mass*(trunk_base_length*trunk_base_length + trunk_base_width*trunk_base_width)}"/>
-        </inertial>
-        <visual>
-            <origin xyz="0.019774 0 0" rpy="${pi/2} 0 ${pi/2}"/>
-            <geometry>
-                <mesh filename="package://meldog_description/meshes/visual/trunk.stl"
-                      scale="0.001 0.001 0.001" />
-                </geometry>
-        </visual>
-        <collision>
-            <origin xyz="0.019774 0 0" rpy="${pi/2} 0 ${pi/2}"/>
-            <geometry>
-                <mesh filename="package://meldog_description/meshes/collision/trunk_collision.stl"
-                      scale="0.001 0.001 0.001" />
-                </geometry>
-        </collision>
-    </link>
-    <!-- Meldog trunk (3 simple boxes) -->
-    <!--
-    <xacro:property name="trunk_base_length" value="0.8" />
-    <xacro:property name="trunk_base_width" value="0.2" />
-    <xacro:property name="trunk_base_height" value="0.1" />
-    <xacro:property name="trunk_actuators_length" value="0.3" />
-    <xacro:property name="trunk_actuators_width" value="0.15" />
-    <xacro:property name="trunk_actuators_height" value="0.1" />
-    <xacro:property name="trunk_mass" value="8.0"/>
-    <link name="trunk_link">
-        <inertial>
-            <origin xyz="0.0 0.0 0.0" rpy="0.0 0.0 0.0"/>
-            <mass value="${trunk_mass}"/>
-            <inertia ixx="${1/12*trunk_mass*(trunk_base_width*trunk_base_width + trunk_base_height*trunk_base_height)}" ixy="0.0" ixz="0.0" iyy="${1/12*trunk_mass*(trunk_base_length*trunk_base_length + trunk_base_height*trunk_base_height)}" iyz=".0" izz="${1/12*trunk_mass*(trunk_base_length*trunk_base_length + trunk_base_width*trunk_base_width)}"/>
-        </inertial>
-        <visual name="trunk_base_visual">
-            <origin xyz="0.0 0.0 0.0" rpy="0.0 0.0 0.0"/>
-            <geometry>
-                <box size="${trunk_base_length} ${trunk_base_width} ${trunk_base_height}"/>
-            </geometry>
-        </visual>
-        <visual name="trunk_actuators_left_visual">
-            <origin xyz="0.0 ${trunk_base_width/2 + trunk_actuators_width/2} 0.0" rpy="0.0 0.0 0.0"/>
-            <geometry>
-                <box size="${trunk_actuators_length} ${trunk_actuators_width} ${trunk_actuators_height}"/>
-            </geometry>
-        </visual>
-        <visual name="trunk_actuators_right_visual">
-            <origin xyz="0.0 ${-trunk_base_width/2 - trunk_actuators_width/2} 0.0" rpy="0.0 0.0 0.0"/>
-            <geometry>
-                <box size="${trunk_actuators_length} ${trunk_actuators_width} ${trunk_actuators_height}"/>
-            </geometry>
-        </visual>
-         <collision name="trunk_base_collision">
-            <origin xyz="0.0 0.0 0.0" rpy="0.0 0.0 0.0"/>
-            <geometry>
-                <box size="${trunk_base_length} ${trunk_base_width} ${trunk_base_height}"/>
-            </geometry>
-        </collision>
-        <collision name="trunk_actuators_left_collision">
-            <origin xyz="0.0 ${trunk_base_width/2 + trunk_actuators_width/2} 0.0" rpy="0.0 0.0 0.0"/>
-            <geometry>
-                <box size="${trunk_actuators_length} ${trunk_actuators_width} ${trunk_actuators_height}"/>
-            </geometry>
-        </collision>
-        <collision name="trunk_actuators_right_collision">
-            <origin xyz="0.0 ${-trunk_base_width/2 - trunk_actuators_width/2} 0.0" rpy="0.0 0.0 0.0"/>
-            <geometry>
-                <box size="${trunk_actuators_length} ${trunk_actuators_width} ${trunk_actuators_height}"/>
-            </geometry>
-        </collision>
-    </link>
-    -->
+<!-- visual and collision STL have wrong orientation and position
+ (CAD model was broken at the time of export), its fixed here-->
+    <xacro:link_macro
+        name="trunk_link"
+        is_foot="0"
+        vis_name="${trunk_vis_stl_name}"
+        coll_name="${trunk_coll_stl_name}"
+        vis_rpy="${pi/2} 0.0 ${pi/2}"
+        vis_xyz="0.019774 0.0 0.0"
+        coll_rpy="${pi/2} 0.0 ${pi/2}"
+        coll_xyz="0.019774 0.0 0.0"
+        m="${trunk_mass}"
+        cm_x="${trunk_cm_x}"
+        cm_y="${trunk_cm_y}"
+        cm_z="${trunk_cm_z}"
+        ixx="${trunk_ixx}" ixy="${trunk_ixy}" ixz="${trunk_ixz}"
+                                iyy="${trunk_iyy}" iyz="${trunk_iyz}"
+                                                        izz="${trunk_izz}"/>
 </robot>

File: meldog_description/description/macros/link_macro.urdf.xacro (robot description, xacro)
@@ -1,8 +1,7 @@
 <?xml version="1.0"?>
 <robot xmlns:xacro="http://www.ros.org/wiki/xacro">
-    <!-- Macro for defining a link, please ensure that
-    the visual and collision models coordinate
-    systems are placed in joints -->
-    <xacro:macro name="link_macro" params="name is_foot vis_name coll_name m cm_x cm_y cm_z ixx ixy ixz iyy iyz izz">
+    <xacro:macro name="link_macro" params="name is_foot vis_name coll_name m cm_x cm_y cm_z ixx ixy ixz iyy iyz izz
+                                            vis_xyz:='0.0 0.0 0.0' vis_rpy:='0.0 0.0 0.0'
+                                            coll_xyz:='0.0 0.0 0.0' coll_rpy:='0.0 0.0 0.0'">
         <link name="${name}">
             <visual>
@@ -11,5 +10,5 @@
                           scale="0.001 0.001 0.001" />
                 </geometry>
-                <origin xyz="0 0 0" rpy="0 0 0"/>
+                <origin xyz="${vis_xyz}" rpy="${vis_rpy}"/>
             </visual>
             <xacro:if value="${is_foot == 1}">
@@ -18,5 +17,5 @@
                         <sphere radius="${foot_radius}" />
                     </geometry>
-                    <origin xyz="0 0 0" rpy="0 0 0" />
+                    <origin xyz="${coll_xyz}" rpy="0 0 0" />
                 </collision>
             </xacro:if>
@@ -27,5 +26,5 @@
                             scale="0.001 0.001 0.001" />
                     </geometry>
-                    <origin xyz="0 0 0" rpy="0 0 0" />
+                    <origin xyz="${coll_xyz}" rpy="${coll_rpy}" />
                 </collision>
             </xacro:if>
