Commit message: First fix of properties dimensions

File: meldog_description/description/links/properties/H_properties.urdf.xacro (robot description, xacro)
@@ -2,6 +2,6 @@
 <robot xmlns:xacro="http://www.ros.org/wiki/xacro">
     <!-- simple collision shape properties  -->
-    <xacro:property name="hip_col_length" value="0.2"/>
-    <xacro:property name="hip_col_radius" value="0.125"/>
+    <xacro:property name="hip_col_length" value="0.23"/>
+    <xacro:property name="hip_col_radius" value="0.12"/>
     <!-- meshes -->
     <xacro:property name="hip_vis_stl_name" value="hip_test.stl" />

File: meldog_description/description/links/properties/LL_properties.urdf.xacro (robot description, xacro)
@@ -3,5 +3,5 @@
     <!-- simple collision shape dimensions  -->
     <xacro:property name="lower_limb_col_length" value="0.25"/>
-    <xacro:property name="lower_limb_col_radius" value="0.125"/>
+    <xacro:property name="lower_limb_col_radius" value="0.0275"/>
     <!-- meshes -->
     <xacro:property name="lower_limb_vis_stl_name" value="LL_vis_v2.stl" />

File: meldog_description/description/links/properties/UL_properties.urdf.xacro (robot description, xacro)
@@ -3,5 +3,5 @@
     <!-- simple collision shape properties  -->
     <xacro:property name="upper_limb_col_length" value="0.25"/>
-    <xacro:property name="upper_limb_col_radius" value="0.125"/>
+    <xacro:property name="upper_limb_col_radius" value="0.025"/>
     <!-- meshes -->
     <xacro:property name="upper_limb_vis_stl_name" value="upper_limb_test.stl" />
