Commit message: Updating mass parameters

File: meldog_description/description/links/properties/F_properties.urdf.xacro (robot description, xacro)
@@ -10,15 +10,15 @@
     <!-- inertial properties -->
         <!-- mass -->
-        <xacro:property name="foot_mass" value="0.037"/>
+        <xacro:property name="foot_mass" value="0.0"/>
         <!-- center of mass -->
         <xacro:property name="foot_cm_x" value="0.0"/>
         <xacro:property name="foot_cm_y" value="0.0"/>
-        <xacro:property name="foot_cm_z" value="-8.417"/>
+        <xacro:property name="foot_cm_z" value="0.0"/>
         <!-- tensor of inertia -->
-        <xacro:property name="foot_ixx" value="14.919"/>
+        <xacro:property name="foot_ixx" value="0.0"/>
         <xacro:property name="foot_ixy" value="0.0"/>
         <xacro:property name="foot_ixz" value="0.0"/>
-        <xacro:property name="foot_iyy" value="25.291"/>
+        <xacro:property name="foot_iyy" value="0.0"/>
         <xacro:property name="foot_iyz" value="0.0"/>
-        <xacro:property name="foot_izz" value="23.390"/>
+        <xacro:property name="foot_izz" value="0.0"/>
 </robot>

File: meldog_description/description/links/properties/H_properties.urdf.xacro (robot description, xacro)
@@ -10,15 +10,15 @@
     <!-- inertial properties -->
         <!-- mass -->
-        <xacro:property name="hip_mass" value="2.276"/>
+        <xacro:property name="hip_mass" value="2.210"/>
         <!-- center of mass -->
-        <xacro:property name="hip_cm_x" value="126.369"/>
-        <xacro:property name="hip_cm_y" value="14.729"/>
-        <xacro:property name="hip_cm_z" value="0.160"/>
+        <xacro:property name="hip_cm_x" value="126.318"/>
+        <xacro:property name="hip_cm_y" value="12.309"/>
+        <xacro:property name="hip_cm_z" value="0.112"/>
         <!-- tensor of inertia -->
-        <xacro:property name="hip_ixx" value="3609.753"/>
-        <xacro:property name="hip_ixy" value="-371.167"/>
-        <xacro:property name="hip_ixz" value="0.550"/>
-        <xacro:property name="hip_iyy" value="8775.172"/>
-        <xacro:property name="hip_iyz" value="17.541"/>
-        <xacro:property name="hip_izz" value="9362.116"/>
+        <xacro:property name="hip_ixx" value="3658.000"/>
+        <xacro:property name="hip_ixy" value="-334.100"/>
+        <xacro:property name="hip_ixz" value="0.218"/>
+        <xacro:property name="hip_iyy" value="8851.000"/>
+        <xacro:property name="hip_iyz" value="12.221"/>
+        <xacro:property name="hip_izz" value="9241.000"/>
 </robot>

File: meldog_description/description/links/properties/LL_properties.urdf.xacro (robot description, xacro)
@@ -12,15 +12,15 @@
     <!-- inertial properties -->
         <!-- mass -->
-        <xacro:property name="lower_limb_mass" value="0.079"/>
+        <xacro:property name="lower_limb_mass" value="0.226"/>
         <!-- center of mass -->
-        <xacro:property name="lower_limb_cm_x" value="0.801"/>
+        <xacro:property name="lower_limb_cm_x" value="0.048"/>
         <xacro:property name="lower_limb_cm_y" value="0"/>
-        <xacro:property name="lower_limb_cm_z" value="-139.836"/>
+        <xacro:property name="lower_limb_cm_z" value="-182.98"/>
         <!-- moments of inertia -->
-        <xacro:property name="lower_limb_ixx" value="598.222"/>
+        <xacro:property name="lower_limb_ixx" value="1811.000"/>
         <xacro:property name="lower_limb_ixy" value="0.0"/>
-        <xacro:property name="lower_limb_ixz" value="-2.447"/>
-        <xacro:property name="lower_limb_iyy" value="603.088"/>
+        <xacro:property name="lower_limb_ixz" value="-3.618"/>
+        <xacro:property name="lower_limb_iyy" value="1838.000"/>
         <xacro:property name="lower_limb_iyz" value="0.0"/>
-        <xacro:property name="lower_limb_izz" value="13.771"/>
+        <xacro:property name="lower_limb_izz" value="83.423"/>
 </robot>

File: meldog_description/description/links/properties/UL_properties.urdf.xacro (robot description, xacro)
@@ -12,15 +12,15 @@
     <!-- inertial properties -->
         <!-- mass -->
-        <xacro:property name="upper_limb_mass" value="0.474"/>
+        <xacro:property name="upper_limb_mass" value="0.398"/>
         <!-- center of mass -->
-        <xacro:property name="upper_limb_cm_x" value="-1.185"/>
-        <xacro:property name="upper_limb_cm_y" value="-4.308"/>
-        <xacro:property name="upper_limb_cm_z" value="-94.203"/>
+        <xacro:property name="upper_limb_cm_x" value="-0.467"/>
+        <xacro:property name="upper_limb_cm_y" value="0.271"/>
+        <xacro:property name="upper_limb_cm_z" value="-105.160"/>
         <!-- moments of inertia -->
-        <xacro:property name="upper_limb_ixx" value="4064.505"/>
-        <xacro:property name="upper_limb_ixy" value="1.241"/>
-        <xacro:property name="upper_limb_ixz" value="19.989"/>
-        <xacro:property name="upper_limb_iyy" value="4150.05"/>
-        <xacro:property name="upper_limb_iyz" value="235.648"/>
-        <xacro:property name="upper_limb_izz" value="424.555"/>
+        <xacro:property name="upper_limb_ixx" value="3553.000"/>
+        <xacro:property name="upper_limb_ixy" value="0.288"/>
+        <xacro:property name="upper_limb_ixz" value="3.222"/>
+        <xacro:property name="upper_limb_iyy" value="3648.05"/>
+        <xacro:property name="upper_limb_iyz" value="29.960"/>
+        <xacro:property name="upper_limb_izz" value="309.300"/>
 </robot>
