Commit message: Adding an option for choosing simple collision model, didn't set proper dimensions

File: meldog_description/description/links/foot/LFF_link.urdf.xacro (robot description, xacro)
@@ -3,5 +3,6 @@
     <xacro:link_macro
         name="LFF_link"
-        is_foot="1"
+        sc_length="${foot_col_length}"
+        sc_radius="${foot_col_radius}"
         vis_name="${foot_vis_stl_name}"
         coll_name="empty"

File: meldog_description/description/links/foot/LRF_link.urdf.xacro (robot description, xacro)
@@ -3,5 +3,6 @@
     <xacro:link_macro
         name="LRF_link"
-        is_foot="1"
+        sc_length="${foot_col_length}"
+        sc_radius="${foot_col_radius}"
         vis_name="${foot_vis_stl_name}"
         coll_name="empty"

File: meldog_description/description/links/foot/RFF_link.urdf.xacro (robot description, xacro)
@@ -3,5 +3,6 @@
     <xacro:link_macro
         name="RFF_link"
-        is_foot="1"
+        sc_length="${foot_col_length}"
+        sc_radius="${foot_col_radius}"
         vis_name="${foot_vis_stl_name}"
         coll_name="empty"

File: meldog_description/description/links/foot/RRF_link.urdf.xacro (robot description, xacro)
@@ -3,5 +3,6 @@
     <xacro:link_macro
         name="RRF_link"
-        is_foot="1"
+        sc_length="${foot_col_length}"
+        sc_radius="${foot_col_radius}"
         vis_name="${foot_vis_stl_name}"
         coll_name="empty"

File: meldog_description/description/links/hip/LFH_link.urdf.xacro (robot description, xacro)
@@ -3,5 +3,6 @@
     <xacro:link_macro
         name="LFH_link"
-        is_foot="0"
+        sc_length="${hip_col_length}"
+        sc_radius="${hip_col_radius}"
         vis_name="${hip_vis_stl_name}"
         coll_name="${hip_coll_stl_name}"

File: meldog_description/description/links/hip/LRH_link.urdf.xacro (robot description, xacro)
@@ -3,5 +3,6 @@
     <xacro:link_macro
         name="LRH_link"
-        is_foot="0"
+        sc_length="${hip_col_length}"
+        sc_radius="${hip_col_radius}"
         vis_name="rear_left_hip.stl"
         coll_name="rear_left_hip_collision.stl"

File: meldog_description/description/links/hip/RFH_link.urdf.xacro (robot description, xacro)
@@ -3,5 +3,6 @@
     <xacro:link_macro
         name="RFH_link"
-        is_foot="0"
+        vis_name="${hip_vis_stl_name}"
+        coll_name="${hip_coll_stl_name}"
         vis_name="front_right_hip.stl"
         coll_name="front_right_hip_collision.stl"

File: meldog_description/description/links/hip/RRH_link.urdf.xacro (robot description, xacro)
@@ -3,5 +3,6 @@
     <xacro:link_macro
         name="RRH_link"
-        is_foot="0"
+        sc_length="${hip_col_length}"
+        sc_radius="${hip_col_radius}"
         vis_name="rear_right_hip.stl"
         coll_name="rear_right_hip_collision.stl"

File: meldog_description/description/links/lower_limb/LFLL_link.urdf.xacro (robot description, xacro)
@@ -3,5 +3,6 @@
     <xacro:link_macro
         name="LFLL_link"
-        is_foot="0"
+        sc_length="${lower_limb_col_length}"
+        sc_radius="${lower_limb_col_radius}"
         vis_name="${lower_limb_vis_stl_name}"
         coll_name="${lower_limb_coll_stl_name}"

File: meldog_description/description/links/lower_limb/LRLL_link.urdf.xacro (robot description, xacro)
@@ -3,5 +3,6 @@
     <xacro:link_macro
         name="LRLL_link"
-        is_foot="0"
+        sc_length="${lower_limb_col_length}"
+        sc_radius="${fower_limb_col_radius}"
         vis_name="${lower_limb_vis_stl_name}"
         coll_name="${lower_limb_coll_stl_name}"

File: meldog_description/description/links/lower_limb/RFLL_link.urdf.xacro (robot description, xacro)
@@ -3,5 +3,6 @@
     <xacro:link_macro
         name="RFLL_link"
-        is_foot="0"
+        sc_length="${lower_limb_col_length}"
+        sc_radius="${lower_limb_col_radius}"
         vis_name="${lower_limb_vis_stl_name}"
         coll_name="${lower_limb_coll_stl_name}"

File: meldog_description/description/links/lower_limb/RRLL_link.urdf.xacro (robot description, xacro)
@@ -3,5 +3,6 @@
     <xacro:link_macro
         name="RRLL_link"
-        is_foot="0"
+        sc_length="${lower_limb_col_length}"
+        sc_radius="${lower_limb_col_radius}"
         vis_name="${lower_limb_vis_stl_name}"
         coll_name="${lower_limb_coll_stl_name}"

File: meldog_description/description/links/properties/F_properties.urdf.xacro (robot description, xacro)
@@ -1,6 +1,7 @@
 <?xml version="1.0"?>
 <robot xmlns:xacro="http://www.ros.org/wiki/xacro">
-    <!-- foot radius -->
-    <xacro:property name="foot_radius" value="0.035" />
+    <!-- simple collision shape properties  -->
+    <xacro:property name="foot_col_length" value="0"/>
+    <xacro:property name="foot_col_radius" value="0.035"/>
     <!-- meshes -->
     <xacro:property name="foot_vis_stl_name" value="foot_vis.stl" />

File: meldog_description/description/links/properties/H_properties.urdf.xacro (robot description, xacro)
@@ -1,4 +1,7 @@
 <?xml version="1.0"?>
 <robot xmlns:xacro="http://www.ros.org/wiki/xacro">
+    <!-- simple collision shape properties  -->
+    <xacro:property name="hip_col_length" value="0.2"/>
+    <xacro:property name="hip_col_radius" value="0.125"/>
     <!-- meshes -->
     <xacro:property name="hip_vis_stl_name" value="hip_test.stl" />

File: meldog_description/description/links/properties/LL_properties.urdf.xacro (robot description, xacro)
@@ -1,4 +1,7 @@
 <?xml version="1.0"?>
 <robot xmlns:xacro="http://www.ros.org/wiki/xacro">
+    <!-- simple collision shape dimensions  -->
+    <xacro:property name="lower_limb_col_length" value="0.25"/>
+    <xacro:property name="lower_limb_col_radius" value="0.125"/>
     <!-- meshes -->
     <xacro:property name="lower_limb_vis_stl_name" value="LL_vis_v2.stl" />

File: meldog_description/description/links/properties/UL_properties.urdf.xacro (robot description, xacro)
@@ -1,4 +1,7 @@
 <?xml version="1.0"?>
 <robot xmlns:xacro="http://www.ros.org/wiki/xacro">
+    <!-- simple collision shape properties  -->
+    <xacro:property name="upper_limb_col_length" value="0.25"/>
+    <xacro:property name="upper_limb_col_radius" value="0.125"/>
     <!-- meshes -->
     <xacro:property name="upper_limb_vis_stl_name" value="upper_limb_test.stl" />

File: meldog_description/description/links/upper_limb/LFUL_link.urdf.xacro (robot description, xacro)
@@ -3,5 +3,6 @@
     <xacro:link_macro
         name="LFUL_link"
-        is_foot="0"
+        sc_length="${upper_limb_col_length}"
+        sc_radius="${upper_limb_col_radius}"
         vis_name="${upper_limb_vis_stl_name}"
         coll_name="${upper_limb_coll_stl_name}"

File: meldog_description/description/links/upper_limb/LRUL_link.urdf.xacro (robot description, xacro)
@@ -3,5 +3,6 @@
     <xacro:link_macro
         name="LRUL_link"
-        is_foot="0"
+        sc_length="${upper_limb_col_length}"
+        sc_radius="${upper_limb_col_radius}"
         vis_name="upper_limb_test.stl"
         coll_name="upper_limb_collision.stl"

File: meldog_description/description/links/upper_limb/RFUL_link.urdf.xacro (robot description, xacro)
@@ -3,5 +3,6 @@
     <xacro:link_macro
         name="RFUL_link"
-        is_foot="0"
+        sc_length="${upper_limb_col_length}"
+        sc_radius="${upper_limb_col_radius}"
         vis_name="r_upper_limb_vis.stl"
         coll_name="upper_limb_collision.stl"

File: meldog_description/description/links/upper_limb/RRUL_link.urdf.xacro (robot description, xacro)
@@ -3,5 +3,6 @@
     <xacro:link_macro
         name="RRUL_link"
-        is_foot="0"
+        sc_length="${upper_limb_col_length}"
+        sc_radius="${upper_limb_col_radius}"
         vis_name="r_upper_limb_vis.stl"
         coll_name="upper_limb_collision.stl"
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
Commit message: Fixing up URDF files, trying geometry

File: meldog_description/description/links/foot/LFF_link.urdf.xacro (robot description, xacro)
@@ -3,5 +3,5 @@
     <xacro:link_macro
         name="LFF_link"
-        has_sc = 1
+        has_sc="1"
         sc_length="${foot_col_length}"
         sc_radius="${foot_col_radius}"

File: meldog_description/description/links/foot/LRF_link.urdf.xacro (robot description, xacro)
@@ -3,5 +3,5 @@
     <xacro:link_macro
         name="LRF_link"
-        has_sc = 1
+        has_sc="1"
         sc_length="${foot_col_length}"
         sc_radius="${foot_col_radius}"

File: meldog_description/description/links/foot/RFF_link.urdf.xacro (robot description, xacro)
@@ -3,5 +3,5 @@
     <xacro:link_macro
         name="RFF_link"
-        has_sc = 1
+        has_sc="1"
         sc_length="${foot_col_length}"
         sc_radius="${foot_col_radius}"

File: meldog_description/description/links/foot/RRF_link.urdf.xacro (robot description, xacro)
@@ -3,5 +3,5 @@
     <xacro:link_macro
         name="RRF_link"
-        has_sc = 1
+        has_sc="1"
         sc_length="${foot_col_length}"
         sc_radius="${foot_col_radius}"

File: meldog_description/description/links/hip/LFH_link.urdf.xacro (robot description, xacro)
@@ -3,5 +3,5 @@
     <xacro:link_macro
         name="LFH_link"
-        has_sc = 1
+        has_sc="0"
         sc_length="${hip_col_length}"
         sc_radius="${hip_col_radius}"

File: meldog_description/description/links/hip/LRH_link.urdf.xacro (robot description, xacro)
@@ -3,5 +3,5 @@
     <xacro:link_macro
         name="LRH_link"
-        has_sc = 1
+        has_sc="0"
         sc_length="${hip_col_length}"
         sc_radius="${hip_col_radius}"

File: meldog_description/description/links/hip/RFH_link.urdf.xacro (robot description, xacro)
@@ -3,7 +3,7 @@
     <xacro:link_macro
         name="RFH_link"
-        has_sc = 1
-        vis_name="${hip_vis_stl_name}"
-        coll_name="${hip_coll_stl_name}"
+        has_sc="0"
+        sc_length="${hip_col_length}"
+        sc_radius="${hip_col_radius}"
         vis_name="front_right_hip.stl"
         coll_name="front_right_hip_collision.stl"

File: meldog_description/description/links/hip/RRH_link.urdf.xacro (robot description, xacro)
@@ -3,5 +3,5 @@
     <xacro:link_macro
         name="RRH_link"
-        has_sc = 1
+        has_sc="0"
         sc_length="${hip_col_length}"
         sc_radius="${hip_col_radius}"

File: meldog_description/description/links/lower_limb/LFLL_link.urdf.xacro (robot description, xacro)
@@ -3,5 +3,5 @@
     <xacro:link_macro
         name="LFLL_link"
-        has_sc = 1
+        has_sc="1"
         sc_length="${lower_limb_col_length}"
         sc_radius="${lower_limb_col_radius}"

File: meldog_description/description/links/lower_limb/LRLL_link.urdf.xacro (robot description, xacro)
@@ -3,7 +3,7 @@
     <xacro:link_macro
         name="LRLL_link"
-        has_sc = 1
+        has_sc="1"
         sc_length="${lower_limb_col_length}"
-        sc_radius="${fower_limb_col_radius}"
+        sc_radius="${lower_limb_col_radius}"
         vis_name="${lower_limb_vis_stl_name}"
         coll_name="${lower_limb_coll_stl_name}"

File: meldog_description/description/links/lower_limb/RFLL_link.urdf.xacro (robot description, xacro)
@@ -3,5 +3,5 @@
     <xacro:link_macro
         name="RFLL_link"
-        has_sc = 1
+        has_sc="1"
         sc_length="${lower_limb_col_length}"
         sc_radius="${lower_limb_col_radius}"

File: meldog_description/description/links/lower_limb/RRLL_link.urdf.xacro (robot description, xacro)
@@ -3,5 +3,5 @@
     <xacro:link_macro
         name="RRLL_link"
-        has_sc = 1
+        has_sc="1"
         sc_length="${lower_limb_col_length}"
         sc_radius="${lower_limb_col_radius}"

File: meldog_description/description/links/properties/H_properties.urdf.xacro (robot description, xacro)
@@ -2,5 +2,5 @@
 <robot xmlns:xacro="http://www.ros.org/wiki/xacro">
     <!-- simple collision shape properties  -->
-    <xacro:property name="hip_col_length" value="0.23"/>
+    <xacro:property name="hip_col_length" value="0.023"/>
     <xacro:property name="hip_col_radius" value="0.12"/>
     <!-- meshes -->

File: meldog_description/description/links/properties/UL_properties.urdf.xacro (robot description, xacro)
@@ -3,5 +3,5 @@
     <!-- simple collision shape properties  -->
     <xacro:property name="upper_limb_col_length" value="0.25"/>
-    <xacro:property name="upper_limb_col_radius" value="0.025"/>
+    <xacro:property name="upper_limb_col_radius" value="0.05"/>
     <!-- meshes -->
     <xacro:property name="upper_limb_vis_stl_name" value="upper_limb_test.stl" />

File: meldog_description/description/links/upper_limb/LFUL_link.urdf.xacro (robot description, xacro)
@@ -3,5 +3,5 @@
     <xacro:link_macro
         name="LFUL_link"
-        has_sc = 1
+        has_sc="1"
         sc_length="${upper_limb_col_length}"
         sc_radius="${upper_limb_col_radius}"

File: meldog_description/description/links/upper_limb/LRUL_link.urdf.xacro (robot description, xacro)
@@ -3,5 +3,5 @@
     <xacro:link_macro
         name="LRUL_link"
-        has_sc = 1
+        has_sc="1"
         sc_length="${upper_limb_col_length}"
         sc_radius="${upper_limb_col_radius}"

File: meldog_description/description/links/upper_limb/RFUL_link.urdf.xacro (robot description, xacro)
@@ -3,5 +3,5 @@
     <xacro:link_macro
         name="RFUL_link"
-        has_sc = 1
+        has_sc="1"
         sc_length="${upper_limb_col_length}"
         sc_radius="${upper_limb_col_radius}"

File: meldog_description/description/links/upper_limb/RRUL_link.urdf.xacro (robot description, xacro)
@@ -3,5 +3,5 @@
     <xacro:link_macro
         name="RRUL_link"
-        has_sc = 1
+        has_sc="1"
         sc_length="${upper_limb_col_length}"
         sc_radius="${upper_limb_col_radius}"

File: meldog_description/description/macros/link_macro.urdf.xacro (robot description, xacro)
@@ -14,5 +14,5 @@
                 <origin xyz="0 0 0" rpy="0 0 0"/>
             </visual>
-            <xacro:if value="${has_simple_collision == 1}">
+            <xacro:if value="${has_sc == 1}">
                 <collision name="collision">
                     <geometry>
@@ -21,10 +21,11 @@
                         </xacro:if>
                         <xacro:if value="${sc_length != 0}">
-                            <cyllinder length="${sc_length}" radius="${sc_radius}"/>
+                            <cylinder length="${sc_length}" radius="${sc_radius}"/>
                         </xacro:if>
                     </geometry>
-                    <origin xyz="0 0 0" rpy="0 0 0" />
+                    <origin xyz="0 0 -${sc_length/2}" rpy="0 0 0" />
                 </collision>
-            <xacro:if value="${has_simple_collision == 0}">
+            </xacro:if>
+            <xacro:if value="${has_sc == 0}">
                 <collision>
                     <geometry>

Commit message: Hip model problem not solving

File: meldog_description/description/links/foot/LFF_link.urdf.xacro (robot description, xacro)
@@ -3,5 +3,5 @@
     <xacro:link_macro
         name="LFF_link"
-        has_sc="1"
+        has_sc="${foot_has_sc}"
         sc_length="${foot_col_length}"
         sc_radius="${foot_col_radius}"

File: meldog_description/description/links/foot/LRF_link.urdf.xacro (robot description, xacro)
@@ -3,5 +3,5 @@
     <xacro:link_macro
         name="LRF_link"
-        has_sc="1"
+        has_sc="${foot_has_sc}"
         sc_length="${foot_col_length}"
         sc_radius="${foot_col_radius}"

File: meldog_description/description/links/foot/RFF_link.urdf.xacro (robot description, xacro)
@@ -3,5 +3,5 @@
     <xacro:link_macro
         name="RFF_link"
-        has_sc="1"
+        has_sc="${foot_has_sc}"
         sc_length="${foot_col_length}"
         sc_radius="${foot_col_radius}"

File: meldog_description/description/links/foot/RRF_link.urdf.xacro (robot description, xacro)
@@ -3,5 +3,5 @@
     <xacro:link_macro
         name="RRF_link"
-        has_sc="1"
+        has_sc="${foot_has_sc}"
         sc_length="${foot_col_length}"
         sc_radius="${foot_col_radius}"

File: meldog_description/description/links/hip/LFH_link.urdf.xacro (robot description, xacro)
@@ -3,9 +3,9 @@
     <xacro:link_macro
         name="LFH_link"
-        has_sc="0"
+        has_sc="${hip_has_sc}"
         sc_length="${hip_col_length}"
         sc_radius="${hip_col_radius}"
         vis_name="${hip_vis_stl_name}"
-        coll_name="${hip_coll_stl_name}"
+        coll_name="hip_collision.stl"
         m="${hip_mass}"
         cm_x="${hip_cm_x}"

File: meldog_description/description/links/hip/LRH_link.urdf.xacro (robot description, xacro)
@@ -3,8 +3,8 @@
     <xacro:link_macro
         name="LRH_link"
-        has_sc="0"
+        has_sc="${hip_has_sc}"
         sc_length="${hip_col_length}"
         sc_radius="${hip_col_radius}"
-        vis_name="rear_left_hip.stl"
+        vis_name="${hip_vis_stl_name}"
         coll_name="rear_left_hip_collision.stl"
         m="${hip_mass}"

File: meldog_description/description/links/hip/RFH_link.urdf.xacro (robot description, xacro)
@@ -3,9 +3,9 @@
     <xacro:link_macro
         name="RFH_link"
-        has_sc="0"
+        has_sc="${hip_has_sc}"
         sc_length="${hip_col_length}"
         sc_radius="${hip_col_radius}"
-        vis_name="front_right_hip.stl"
-        coll_name="front_right_hip_collision.stl"
+        vis_name="${hip_vis_stl_name}"
+        coll_name="forward_right_hip_collision.stl"
         m="${hip_mass}"
         cm_x="${hip_cm_x}"

File: meldog_description/description/links/hip/RRH_link.urdf.xacro (robot description, xacro)
@@ -3,8 +3,8 @@
     <xacro:link_macro
         name="RRH_link"
-        has_sc="0"
+        has_sc="${hip_has_sc}"
         sc_length="${hip_col_length}"
         sc_radius="${hip_col_radius}"
-        vis_name="rear_right_hip.stl"
+        vis_name="${hip_vis_stl_name}"
         coll_name="rear_right_hip_collision.stl"
         m="${hip_mass}"

File: meldog_description/description/links/lower_limb/LFLL_link.urdf.xacro (robot description, xacro)
@@ -3,5 +3,5 @@
     <xacro:link_macro
         name="LFLL_link"
-        has_sc="1"
+        has_sc="${lower_limb_has_sc}"
         sc_length="${lower_limb_col_length}"
         sc_radius="${lower_limb_col_radius}"

File: meldog_description/description/links/lower_limb/LRLL_link.urdf.xacro (robot description, xacro)
@@ -3,5 +3,5 @@
     <xacro:link_macro
         name="LRLL_link"
-        has_sc="1"
+        has_sc="${lower_limb_has_sc}"
         sc_length="${lower_limb_col_length}"
         sc_radius="${lower_limb_col_radius}"

File: meldog_description/description/links/lower_limb/RFLL_link.urdf.xacro (robot description, xacro)
@@ -3,5 +3,5 @@
     <xacro:link_macro
         name="RFLL_link"
-        has_sc="1"
+        has_sc="${lower_limb_has_sc}"
         sc_length="${lower_limb_col_length}"
         sc_radius="${lower_limb_col_radius}"

File: meldog_description/description/links/lower_limb/RRLL_link.urdf.xacro (robot description, xacro)
@@ -3,5 +3,5 @@
     <xacro:link_macro
         name="RRLL_link"
-        has_sc="1"
+        has_sc= "${lower_limb_has_sc}"
         sc_length="${lower_limb_col_length}"
         sc_radius="${lower_limb_col_radius}"

File: meldog_description/description/links/properties/F_properties.urdf.xacro (robot description, xacro)
@@ -2,4 +2,5 @@
 <robot xmlns:xacro="http://www.ros.org/wiki/xacro">
     <!-- simple collision shape properties  -->
+    <xacro:property name="foot_has_sc" value="0"/>
     <xacro:property name="foot_col_length" value="0"/>
     <xacro:property name="foot_col_radius" value="0.035"/>

File: meldog_description/description/links/properties/H_properties.urdf.xacro (robot description, xacro)
@@ -2,4 +2,5 @@
 <robot xmlns:xacro="http://www.ros.org/wiki/xacro">
     <!-- simple collision shape properties  -->
+    <xacro:property name="hip_has_sc" value="1"/>
     <xacro:property name="hip_col_length" value="0.023"/>
     <xacro:property name="hip_col_radius" value="0.12"/>

File: meldog_description/description/links/properties/LL_properties.urdf.xacro (robot description, xacro)
@@ -2,4 +2,5 @@
 <robot xmlns:xacro="http://www.ros.org/wiki/xacro">
     <!-- simple collision shape dimensions  -->
+    <xacro:property name="lower_limb_has_sc" value="0"/>
     <xacro:property name="lower_limb_col_length" value="0.25"/>
     <xacro:property name="lower_limb_col_radius" value="0.0275"/>

File: meldog_description/description/links/properties/UL_properties.urdf.xacro (robot description, xacro)
@@ -2,4 +2,5 @@
 <robot xmlns:xacro="http://www.ros.org/wiki/xacro">
     <!-- simple collision shape properties  -->
+    <xacro:property name="upper_limb_has_sc" value="0"/>
     <xacro:property name="upper_limb_col_length" value="0.25"/>
     <xacro:property name="upper_limb_col_radius" value="0.05"/>

File: meldog_description/description/links/upper_limb/LFUL_link.urdf.xacro (robot description, xacro)
@@ -3,5 +3,5 @@
     <xacro:link_macro
         name="LFUL_link"
-        has_sc="1"
+        has_sc="${upper_limb_has_sc}"
         sc_length="${upper_limb_col_length}"
         sc_radius="${upper_limb_col_radius}"

File: meldog_description/description/links/upper_limb/LRUL_link.urdf.xacro (robot description, xacro)
@@ -3,5 +3,5 @@
     <xacro:link_macro
         name="LRUL_link"
-        has_sc="1"
+        has_sc="${upper_limb_has_sc}"
         sc_length="${upper_limb_col_length}"
         sc_radius="${upper_limb_col_radius}"

File: meldog_description/description/links/upper_limb/RFUL_link.urdf.xacro (robot description, xacro)
@@ -3,5 +3,5 @@
     <xacro:link_macro
         name="RFUL_link"
-        has_sc="1"
+        has_sc="${upper_limb_has_sc}"
         sc_length="${upper_limb_col_length}"
         sc_radius="${upper_limb_col_radius}"

File: meldog_description/description/links/upper_limb/RRUL_link.urdf.xacro (robot description, xacro)
@@ -3,5 +3,5 @@
     <xacro:link_macro
         name="RRUL_link"
-        has_sc="1"
+        has_sc="${upper_limb_has_sc}"
         sc_length="${upper_limb_col_length}"
         sc_radius="${upper_limb_col_radius}"
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