Commit message: New simple collision model implementation

File: meldog_description/description/links/lower_limb/LFLL_link.urdf.xacro (robot description, xacro)
@@ -3,5 +3,7 @@
     <xacro:link_macro
         name="LFLL_link"
-        is_foot="0"
+        has_sc="${lower_limb_has_sc}"
+        sc_length="${lower_limb_col_length}"
+        sc_radius="${lower_limb_col_radius}"
         vis_name="${lower_limb_vis_stl_name}"
         coll_name="${lower_limb_coll_stl_name}"

File: meldog_description/description/links/lower_limb/LRLL_link.urdf.xacro (robot description, xacro)
@@ -3,5 +3,7 @@
     <xacro:link_macro
         name="LRLL_link"
-        is_foot="0"
+        has_sc="${lower_limb_has_sc}"
+        sc_length="${lower_limb_col_length}"
+        sc_radius="${lower_limb_col_radius}"
         vis_name="${lower_limb_vis_stl_name}"
         coll_name="${lower_limb_coll_stl_name}"

File: meldog_description/description/links/lower_limb/RFLL_link.urdf.xacro (robot description, xacro)
@@ -3,5 +3,7 @@
     <xacro:link_macro
         name="RFLL_link"
-        is_foot="0"
+        has_sc="${lower_limb_has_sc}"
+        sc_length="${lower_limb_col_length}"
+        sc_radius="${lower_limb_col_radius}"
         vis_name="${lower_limb_vis_stl_name}"
         coll_name="${lower_limb_coll_stl_name}"

File: meldog_description/description/links/lower_limb/RRLL_link.urdf.xacro (robot description, xacro)
@@ -3,5 +3,7 @@
     <xacro:link_macro
         name="RRLL_link"
-        is_foot="0"
+        has_sc= "${lower_limb_has_sc}"
+        sc_length="${lower_limb_col_length}"
+        sc_radius="${lower_limb_col_radius}"
         vis_name="${lower_limb_vis_stl_name}"
         coll_name="${lower_limb_coll_stl_name}"

File: meldog_description/description/links/properties/F_properties.urdf.xacro (robot description, xacro)
@@ -1,6 +1,8 @@
 <?xml version="1.0"?>
 <robot xmlns:xacro="http://www.ros.org/wiki/xacro">
-    <!-- foot radius -->
-    <xacro:property name="foot_radius" value="0.035" />
+    <!-- simple collision shape properties  -->
+    <xacro:property name="foot_has_sc" value="0"/>
+    <xacro:property name="foot_col_length" value="0"/>
+    <xacro:property name="foot_col_radius" value="0.035"/>
     <!-- meshes -->
     <xacro:property name="foot_vis_stl_name" value="foot_vis.stl" />

File: meldog_description/description/links/properties/H_properties.urdf.xacro (robot description, xacro)
@@ -1,4 +1,8 @@
 <?xml version="1.0"?>
 <robot xmlns:xacro="http://www.ros.org/wiki/xacro">
+    <!-- simple collision shape properties  -->
+    <xacro:property name="hip_has_sc" value="1"/>
+    <xacro:property name="hip_col_length" value="0.023"/>
+    <xacro:property name="hip_col_radius" value="0.12"/>
     <!-- meshes -->
     <xacro:property name="hip_vis_stl_name" value="hip_test.stl" />

File: meldog_description/description/links/properties/LL_properties.urdf.xacro (robot description, xacro)
@@ -1,4 +1,8 @@
 <?xml version="1.0"?>
 <robot xmlns:xacro="http://www.ros.org/wiki/xacro">
+    <!-- simple collision shape dimensions  -->
+    <xacro:property name="lower_limb_has_sc" value="0"/>
+    <xacro:property name="lower_limb_col_length" value="0.25"/>
+    <xacro:property name="lower_limb_col_radius" value="0.0275"/>
     <!-- meshes -->
     <xacro:property name="lower_limb_vis_stl_name" value="LL_vis_v2.stl" />

File: meldog_description/description/links/properties/T_properties.urdf.xacro (robot description, xacro)
@@ -1,4 +1,8 @@
 <?xml version="1.0"?>
 <robot xmlns:xacro="http://www.ros.org/wiki/xacro">
+    <!-- simple collision shape properties  -->
+    <xacro:property name="trunk_col_length" value="0.8"/>
+    <xacro:property name="trunk_has_sc" value="1"/>
+    <xacro:property name="trunk_col_radius" value="0.2"/>
     <!-- meshes -->
     <xacro:property name="trunk_vis_stl_name" value="trunk.stl" />

File: meldog_description/description/links/properties/UL_properties.urdf.xacro (robot description, xacro)
@@ -1,4 +1,8 @@
 <?xml version="1.0"?>
 <robot xmlns:xacro="http://www.ros.org/wiki/xacro">
+    <!-- simple collision shape properties  -->
+    <xacro:property name="upper_limb_has_sc" value="0"/>
+    <xacro:property name="upper_limb_col_length" value="0.25"/>
+    <xacro:property name="upper_limb_col_radius" value="0.05"/>
     <!-- meshes -->
     <xacro:property name="upper_limb_vis_stl_name" value="upper_limb_test.stl" />

File: meldog_description/description/links/trunk.urdf.xacro (robot description, xacro)
@@ -8,5 +8,7 @@
     <xacro:link_macro
         name="trunk_link"
-        is_foot="0"
+        has_sc= "${trunk_has_sc}"
+        sc_length="${trunk_col_length}"
+        sc_radius="${trunk_col_radius}"
         vis_name="${trunk_vis_stl_name}"
         coll_name="${trunk_coll_stl_name}"

File: meldog_description/description/links/upper_limb/LFUL_link.urdf.xacro (robot description, xacro)
@@ -3,5 +3,7 @@
     <xacro:link_macro
         name="LFUL_link"
-        is_foot="0"
+        has_sc="${upper_limb_has_sc}"
+        sc_length="${upper_limb_col_length}"
+        sc_radius="${upper_limb_col_radius}"
         vis_name="${upper_limb_vis_stl_name}"
         coll_name="${upper_limb_coll_stl_name}"

File: meldog_description/description/links/upper_limb/LRUL_link.urdf.xacro (robot description, xacro)
@@ -3,5 +3,7 @@
     <xacro:link_macro
         name="LRUL_link"
-        is_foot="0"
+        has_sc="${upper_limb_has_sc}"
+        sc_length="${upper_limb_col_length}"
+        sc_radius="${upper_limb_col_radius}"
         vis_name="upper_limb_test.stl"
         coll_name="upper_limb_collision.stl"

File: meldog_description/description/links/upper_limb/RFUL_link.urdf.xacro (robot description, xacro)
@@ -3,5 +3,7 @@
     <xacro:link_macro
         name="RFUL_link"
-        is_foot="0"
+        has_sc="${upper_limb_has_sc}"
+        sc_length="${upper_limb_col_length}"
+        sc_radius="${upper_limb_col_radius}"
         vis_name="r_upper_limb_vis.stl"
         coll_name="upper_limb_collision.stl"

File: meldog_description/description/links/upper_limb/RRUL_link.urdf.xacro (robot description, xacro)
@@ -3,5 +3,7 @@
     <xacro:link_macro
         name="RRUL_link"
-        is_foot="0"
+        has_sc="${upper_limb_has_sc}"
+        sc_length="${upper_limb_col_length}"
+        sc_radius="${upper_limb_col_radius}"
         vis_name="r_upper_limb_vis.stl"
         coll_name="upper_limb_collision.stl"

File: meldog_description/description/macros/link_macro.urdf.xacro (robot description, xacro)
@@ -1,5 +1,9 @@
 <?xml version="1.0"?>
 <robot xmlns:xacro="http://www.ros.org/wiki/xacro">
-    <xacro:macro name="link_macro" params="name is_foot vis_name coll_name m cm_x cm_y cm_z ixx ixy ixz iyy iyz izz
+    <!-- Macro for defining a link, please ensure that
+    the visual and collision models coordinate
+    systems are placed in joints -->
+    <!-- sc abbreviates simple collision -->
+    <xacro:macro name="link_macro" params="name has_sc sc_length sc_radius vis_name coll_name m cm_x cm_y cm_z ixx ixy ixz iyy iyz izz
                                             vis_xyz:='0.0 0.0 0.0' vis_rpy:='0.0 0.0 0.0'
                                             coll_xyz:='0.0 0.0 0.0' coll_rpy:='0.0 0.0 0.0'">
@@ -12,13 +16,18 @@
                 <origin xyz="${vis_xyz}" rpy="${vis_rpy}"/>
             </visual>
-            <xacro:if value="${is_foot == 1}">
+            <xacro:if value="${has_sc == 0}">
                 <collision name="collision">
                     <geometry>
-                        <sphere radius="${foot_radius}" />
+                        <xacro:if value="${sc_length == 0}">
+                            <sphere radius="${sc_radius}" />
+                        </xacro:if>
+                        <xacro:if value="${sc_length != 0}">
+                            <cylinder length="${sc_length}" radius="${sc_radius}"/>
+                        </xacro:if>
                     </geometry>
-                    <origin xyz="${coll_xyz}" rpy="0 0 0" />
+                    <origin xyz="${coll_xyz}" rpy="${coll_rpy}" />
                 </collision>
             </xacro:if>
-            <xacro:if value="${is_foot == 0}">
+            <xacro:if value="${has_sc == 1}">
                 <collision>
                     <geometry>
