Commit message: Changed name of collisions

File: meldog_description/description/macros/link_macro.urdf.xacro (robot description, xacro)
@@ -14,5 +14,5 @@
             </visual>
             <xacro:if value="${is_foot == 1}">
-                <collision>
+                <collision name="collision">
                     <geometry>
                         <sphere radius="${foot_radius}" />

Commit message: Accepting changes which had to be accepted after merging

File: meldog_description/description/macros/link_macro.urdf.xacro (robot description, xacro)
@@ -5,11 +5,7 @@
     systems are placed in joints -->
     <!-- sc abbreviates simple collision -->
-<<<<<<< HEAD
-    <xacro:macro name="link_macro" params="name has_sc sc_length sc_radius vis_name coll_name m cm_x cm_y cm_z ixx ixy ixz iyy iyz izz">
-=======
     <xacro:macro name="link_macro" params="name has_sc sc_length sc_radius vis_name coll_name m cm_x cm_y cm_z ixx ixy ixz iyy iyz izz
                                             vis_xyz:='0.0 0.0 0.0' vis_rpy:='0.0 0.0 0.0'
                                             coll_xyz:='0.0 0.0 0.0' coll_rpy:='0.0 0.0 0.0'">
->>>>>>> meldog-urdf-fix
         <link name="${name}">
             <visual>
@@ -30,9 +26,5 @@
                         </xacro:if>
                     </geometry>
-<<<<<<< HEAD
-                    <origin xyz="0 0 -${sc_length/2}" rpy="0 0 0" />
-=======
                     <origin xyz="${coll_xyz}" rpy="${coll_rpy}" />
->>>>>>> meldog-urdf-fix
                 </collision>
             </xacro:if>
